File: stepstick-bc2/stepstick-bc2.sch (KiCad schematic (older format))
At the start: 18 parts, among them P1 CONN_8, P2 CONN_8, U1 A4985-LP

Commit message: stepstick-bc2 v2
Parts:
- added TP1: VREF, symbol TEST_POINT_RMC
Connections:
- net at RV1.2, U1.12 (VREF): now also TP1.1
Other:
- note added: "Can also use A4982, A4987"
- note added: "MS3 is not used"
- moved on the sheet: C1, P1, P2, R2, R7
