File: sango-bob/sango-bob.sch (KiCad schematic (older format))
At the start: 0 parts

Commit message: Sango-bc v0.2
Other:
- note added: "TODO:\n\n"
- note removed: "TODO:\n\nSD card (SPI)\nUART conn (ISP)\nSWD\nUSB"
Changed lines of the file:
@@
-EESchema Schematic File Version 2  date 29/09/2012 12:59:23
+EESchema Schematic File Version 2  date 03/01/2013 13:12:05
 LIBS:power
 LIBS:device
@@
 $Descr A4 11700 8267
 encoding utf-8
-Sheet 1 5
-Title ""
-Date "29 sep 2012"
-Rev ""
+Sheet 1 9
+Title "Sango-bc"
+Date "2 jan 2013"
+Rev "0.2"
 Comp ""
 Comment1 ""
@@
 $EndDescr
 $Sheet
+S 1000 2900 1400 900
+U 5071C6A3
+F0 "Stepper-X" 60
+F1 "stepper-x.sch" 60
+$EndSheet
+$Sheet
 S 3000 1000 1500 1000
 U 5048EA8E
@@
 $EndSheet
 Text Notes 1400 5550 0    60   ~ 0
-TODO:\n\nSD card (SPI)\nUART conn (ISP)\nSWD\nUSB
+TODO:\n\n
 $Sheet
 S 5000 1000 1500 1000
@@
 F1 "sango-steppers.sch" 60
 $EndSheet
+$Sheet
+S 3000 2900 1500 900
+U 50E20F62
+F0 "Stepper-Y" 60
+F1 "stepper-y.sch" 60
+$EndSheet
+$Sheet
+S 5000 2900 1500 900
+U 50E238E5
+F0 "Stepper-Z" 60
+F1 "stepper-z.sch" 60
+$EndSheet
+$Sheet
+S 7000 2900 1500 900
+U 50E23918
+F0 "Stepper-E1" 60
+F1 "stepper-e1.sch" 60
+$EndSheet
 $EndSCHEMATC
