File: sango-bob/sango-conn.sch (KiCad schematic (older format))
At the start: 20 parts, among them K1 CONN_3, K2 CONN_3, K3 CONN_3, K4 CONN_3, P10 CONN_4, P20 CONN_6, P4 CONN_2, P5 CONN_2, P6 CONN_4, P7 CONN_2, P8 CONN_2, Q1 MOSFET_N_RMC, Q2 MOSFET_N_RMC, U9 CONN_MICROSD

Commit message: Sango-bc printer controller version 0.1
Parts:
- added C301: 100nF, symbol C
Connections:
- net labels added: +12V, GNDPWR
- wire segments 70 -> 68
Other:
- moved on the sheet: R5, R6

Commit message: Sango-bc v0.2
Parts:
- removed K4: CONN_3, symbol CONN_3
- removed P10, P6: CONN_4, symbol CONN_4
- added JP401: V_SEL, symbol JUMP_MINI_3
- added P404, P408: HEATER_1, symbol CONN_2
- added P407: HEATER_2, symbol CONN_2
- added Q401, Q402, Q405: 2N7002, symbol MOSFET_N_RMC
- added R404: 10k, symbol R
- K401: renamed from K1; value CONN_3 -> X_STOP
- K403: renamed from K2; value CONN_3 -> Y_STOP
- K404: renamed from K3; value CONN_3 -> Z_STOP
- P401: renamed from P7; value CONN_2 -> AUXPWR1
- P402: renamed from P8; value CONN_2 -> AUXPWR2
- P403: renamed from P20; value CONN_6 -> SERIAL
- P405: renamed from P4; value CONN_2 -> THERM_1
- P406: renamed from P5; value CONN_2 -> THERM_2
- Q403: renamed from Q1; value MOSFET_N_RMC -> IRLB8743
- Q404: renamed from Q2; value MOSFET_N_RMC -> IRLB8743
- R401: renamed from R3; value 4k7 -> 330R
- R403: renamed from R4; value 4k7 -> 10k
- renumbered C7 to C401, C8 to C402, C301 to C403, R5 to R402, R6 to R405, U9 to U401
Connections:
- net labels added: AUX_1, AUX_2, HEATER_1, HEATER_2, SD_DETECT
- net labels removed: FET_1, FET_2
- wire segments 68 -> 70
Other:
- note added: "3.3V TTL-serial connector\n(FTDI compatible)"
- note added: "Endstops\nselectable voltage"
- note added: "Extruder - thermistor input"
- note added: "Extruder heater"
- note added: "Heated bed"
- note added: "Heated bed - thermistor input"
- note added: "Micro SD card (option)"
- moved on the sheet: C403, P401, P402, P403, Q403, Q404, R402, R405
