File: sango-bob/sango-cpu.sch (KiCad schematic (older format))
At the start: 17 parts, among them SW1 RST, U7 STM32F100_48, U8 CONN_CORTEX_DEBUG, X1 8MHz

Commit message: Sango-bc printer controller version 0.1
Parts:
- added P201, P202, P203, P204, P205, P206, P207, P208: TST, symbol TST
Connections:
- net at U7.11 (PA1): now also P204.1
- net at U7.12 (PA2): now also P205.1
- net at U7.13 (PA3): now also P206.1
- net at U7.2 (PC13-TAMPER-RTC): now also P201.1
- net at U7.29 (PA8): now also P207.1
- net at U7.3 (PC14-OSC32_IN): now also P202.1
- net at U7.38 (PA15): now also P208.1
- net at U7.4 (PC15-OSC32_OUT): now also P203.1
- no-connect marks 11 -> 3

Commit message: Sango-bc v0.2
Parts:
- removed P201, P202, P203, P204, P205, P206, P207, P208: TST, symbol TST
- added C309: 100nF, symbol C
- added C310: 4n7, symbol C
- added D301: LED, symbol LED
- added P301: CONN_6X2, symbol CONN_6X2
- added Q301: BSS84, symbol MOSFET_P_OPENDOUS
- added Q302: 2N7002, symbol MOSFET_N_RMC
- added R305, R306, R311: 0R, symbol R
- added R307: 1M, symbol R
- added R308, R309: 4k7, symbol R
- added R310: 1k, symbol R
- added R312: 10k, symbol R
- added R313: 22k, symbol R
- added R314, R315, R316: NF, symbol R
- added U301: 24C08, symbol 24C512
- added U304: USBUF01W6, symbol USBUFXXW6
- added U305: USBCONN, symbol USBCONN
- renumbered C1 to C301, C2 to C302, C12 to C303, C13 to C304, C14 to C305, C15 to C306, C16 to C307, C17 to C308, JP13 to JP301, R10 to R301, R12 to R302, R11 to R303, R13 to R304, SW1 to SW301, U8 to U302, U7 to U303, X1 to X301
Connections:
- net labels added: +5V, AUX_1, AUX_2, DM, DP, EEP_SCL, EEP_SDA, GND_USB, HEATER_1, HEATER_2, SPARE1, SPARE2, SPARE3, SPARE4, USB_PU_EN, VBUS_DET
- net labels removed: FET_1, FET_2
- wire segments 84 -> 155
- no-connect marks 3 -> 4
Other:
- note added: "External IO"
- note added: "JTAG-SWD (option)"
- note added: "R305, R306:\nSTM32F051 NF\nSTM32F1xx 0R"
- note added: "Reset/boot control"
- note added: "Serial EEPROM (option)"
- note added: "Status LED"
- note added: "TODO:\n\n"
- note added: "USB (option)"
- note removed: "TODO:\n\nSD card (SPI)\nUART conn (ISP)\nSWD\nUSB"
- moved on the sheet: C301, C302, C303, C304, C305, C306, C307, C308, JP301, R301, R302, R303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

Commit message: Updates to symbols and fix some ERC errors
Other:
- moved on the sheet: U305
