File: sango-bob/sango-steppers.sch (KiCad schematic (older format))
At the start: 28 parts, among them P15 MOT_Z, P16 MOT_E1, P2 MOT_X, P3 MOT_Y, U2 POLOLU-X, U3 POLOLU-Y, U5 POLOLU-Z, U6 POLOLU-E1

Commit message: Sango-bc printer controller version 0.1
Connections:
- net GND: no longer C10.2, C11.2, C5.2, C6.2, U2.15 (GNDMOT), U3.15 (GNDMOT), U5.15 (GNDMOT), U6.15 (GNDMOT)
- net X_1B: now reaches U2.11 (MOT-1B)
- net X_1B: now also P2.1 (P1); no longer P2.4 (P4)
- net X_1A: now reaches U2.12 (MOT-1A)
- net X_1A: now also P2.2 (P2); no longer P2.3 (P3)
- net X_2A: now reaches U2.13 (MOT-2A)
- net X_2A: now also P2.3 (P3); no longer P2.2 (P2)
- net X_2B: now reaches U2.14 (MOT-2B)
- net X_2B: now also P2.4 (P4); no longer P2.1 (P1)
- net Y_1B: now reaches P3.1 (P1)
- net Y_1B: now also U3.11 (MOT-1B); no longer U3.14 (MOT-2B)
- net Y_1A: now reaches P3.2 (P2)
- net Y_1A: now also U3.12 (MOT-1A); no longer U3.13 (MOT-2A)
- net Y_2A: now reaches P3.3 (P3)
- net Y_2A: now also U3.13 (MOT-2A); no longer U3.12 (MOT-1A)
- net Y_2B: now reaches P3.4 (P4)
- net Y_2B: now also U3.14 (MOT-2B); no longer U3.11 (MOT-1B)
- net Z_1B: now reaches U5.11 (MOT-1B)
- net Z_1B: now also P15.1 (P1); no longer P15.4 (P4)
- net Z_1A: now reaches U5.12 (MOT-1A)
- net Z_1A: now also P15.2 (P2); no longer P15.3 (P3)
- net Z_2A: now reaches U5.13 (MOT-2A)
- net Z_2A: now also P15.3 (P3); no longer P15.2 (P2)
- net Z_2B: now reaches U5.14 (MOT-2B)
- net Z_2B: now also P15.4 (P4); no longer P15.1 (P1)
- net E1_1B: now reaches P16.1 (P1)
- net E1_1B: now also U6.11 (MOT-1B); no longer U6.14 (MOT-2B)
- net E1_1A: now reaches P16.2 (P2)
- net E1_1A: now also U6.12 (MOT-1A); no longer U6.13 (MOT-2A)
- net E1_2A: now reaches P16.3 (P3)
- net E1_2A: now also U6.13 (MOT-2A); no longer U6.12 (MOT-1A)
- net E1_2B: now reaches P16.4 (P4)
- net E1_2B: now also U6.14 (MOT-2B); no longer U6.11 (MOT-1B)
- new net GNDPWR: C10.2, C11.2, C5.2, C6.2, U2.15 (GNDMOT), U3.15 (GNDMOT), U5.15 (GNDMOT), U6.15 (GNDMOT)
Other:
- moved on the sheet: C5, C6, JP4, JP5, JP6, P15, P16, P2, P3, R2, U3

Commit message: Sango-bc v0.2
Parts:
- removed C10, C11, C5, C6: 100uF, symbol CP1
- removed JP1, JP10, JP11, JP12, JP2, JP3, JP4, JP5, JP6, JP7, JP8, JP9: JUMP_MINI, symbol JUMP_MINI
- removed P15: MOT_Z, symbol CONN_4
- removed P16: MOT_E1, symbol CONN_4
- removed P2: MOT_X, symbol CONN_4
- removed P3: MOT_Y, symbol CONN_4
- removed R1, R2, R8, R9: 100k, symbol R
- removed U2: POLOLU-X, symbol POLOLU
- removed U3: POLOLU-Y, symbol POLOLU
- removed U5: POLOLU-Z, symbol POLOLU
- removed U6: POLOLU-E1, symbol POLOLU

Commit message: Updates to symbols and fix some ERC errors
Other:
- note added: "This sheet not used."
Changed lines of the file:
@@
-EESchema Schematic File Version 2  date 03/01/2013 13:12:05
+EESchema Schematic File Version 2  date 22/01/2013 21:21:55
 LIBS:power
 LIBS:device
@@
 Sheet 6 9
 Title "Sango-bc"
-Date "2 jan 2013"
+Date "22 jan 2013"
 Rev "0.2"
 Comp ""
@@
 Comment4 ""
 $EndDescr
+Text Notes 2000 2050 0    60   ~ 0
+This sheet not used.
 $EndSCHEMATC
