File: RAMPS-FD/RIB_interface.sch (KiCad schematic (older format))
At the start: 9 parts, among them U1 ZXGD3005E6, U2 ZXGD3005E6, U3 ZXGD3005E6, U4 TXS0108

Commit message: First version of RAMPS-FD, RIB
Other:
- moved on the sheet: R1, R2, R3, U1, U2, U3
Changed lines of the file:
@@
-EESchema Schematic File Version 2  date 02/02/2013 16:51:34
+EESchema Schematic File Version 2  date 16/02/2013 15:19:28
 LIBS:power
 LIBS:device
@@
 Sheet 2 2
 Title ""
-Date "2 feb 2013"
+Date "16 feb 2013"
 Rev ""
 Comp ""
@@
 Text Notes 2000 3950 0    50   ~ 0
 3.3V/5V Level Translation
-Text GLabel 5300 3050 0    60   Input ~ 0
+Text GLabel 5350 3300 0    60   Input ~ 0
 FET3
-Text GLabel 5300 2300 0    60   Input ~ 0
+Text GLabel 5350 2400 0    60   Input ~ 0
 FET2
-Text GLabel 5300 1450 0    60   Input ~ 0
+Text GLabel 5350 1400 0    60   Input ~ 0
 FET1
-Text GLabel 7400 3050 2    60   Output ~ 0
+Text GLabel 7450 3300 2    60   Output ~ 0
 RAMPS_FET3
-Text GLabel 7400 2300 2    60   Output ~ 0
+Text GLabel 7450 2400 2    60   Output ~ 0
 RAMPS_FET2
-Text GLabel 7400 1450 2    60   Output ~ 0
+Text GLabel 7450 1400 2    60   Output ~ 0
 RAMPS_FET1
 Text GLabel 3450 2800 2    60   Input ~ 0
@@
 Text GLabel 3450 2100 2    60   Input ~ 0
 RAMPS_X_MIN
-Text Notes 6350 3900 0    60   ~ 0
+Text Notes 6350 4100 0    60   ~ 0
 Gate drivers
 $Comp
 L ZXGD3005E6 U1
 U 1 1 510D250C
-P 6600 1450
-F 0 "U1" H 6400 1650 60  0000 C CNN
-F 1 "ZXGD3005E6" H 6600 1150 60  0000 C CNN
-F 2 "SOT26" H 6750 1650 60  0001 C CNN
-	1    6600 1450
+P 6650 1400
+F 0 "U1" H 6450 1600 60  0000 C CNN
+F 1 "ZXGD3005E6" H 6650 1100 60  0000 C CNN
+F 2 "SOT26" H 6800 1600 60  0001 C CNN
+	1    6650 1400
 	1    0    0    -1
 $EndComp
@@
 L R R1
 U 1 1 510D250B
-P 5800 1450
-F 0 "R1" V 5880 1450 50  0000 C CNN
-F 1 "1k" V 5800 1450 50  0000 C CNN
-	1    5800 1450
+P 5850 1400
+F 0 "R1" V 5930 1400 50  0000 C CNN
+F 1 "1k" V 5850 1400 50  0000 C CNN
+	1    5850 1400
 	0    -1   -1   0
 $EndComp
@@
 L +12V #PWR019
 U 1 1 510D250A
-P 5950 1200
-F 0 "#PWR019" H 5950 1150 20  0001 C CNN
-F 1 "+12V" H 5950 1300 30  0000 C CNN
-	1    5950 1200
+P 6000 1150
+F 0 "#PWR019" H 6000 1100 20  0001 C CNN
+F 1 "+12V" H 6000 1250 30  0000 C CNN
+	1    6000 1150
 	1    0    0    -1
 $EndComp
@@
 L GND #PWR020
 U 1 1 510D2509
-P 5950 1750
-F 0 "#PWR020" H 5950 1750 30  0001 C CNN
-F 1 "GND" H 5950 1680 30  0001 C CNN
-	1    5950 1750
+P 6000 1700
+F 0 "#PWR020" H 6000 1700 30  0001 C CNN
+F 1 "GND" H 6000 1630 30  0001 C CNN
+	1    6000 1700
 	1    0    0    -1
 $EndComp
@@
 L GND #PWR021
 U 1 1 510D2508
-P 5950 2600
-F 0 "#PWR021" H 5950 2600 30  0001 C CNN
-F 1 "GND" H 5950 2530 30  0001 C CNN
-	1    5950 2600
+P 6000 2700
+F 0 "#PWR021" H 6000 2700 30  0001 C CNN
+F 1 "GND" H 6000 2630 30  0001 C CNN
+	1    6000 2700
 	1    0    0    -1
 $EndComp
@@
 L +12V #PWR022
 U 1 1 510D2507
-P 5950 2050
-F 0 "#PWR022" H 5950 2000 20  0001 C CNN
-F 1 "+12V" H 5950 2150 30  0000 C CNN
-	1    5950 2050
+P 6000 2150
+F 0 "#PWR022" H 6000 2100 20  0001 C CNN
+F 1 "+12V" H 6000 2250 30  0000 C CNN
+	1    6000 2150
 	1    0    0    -1
 $EndComp
@@
 L R R2
 U 1 1 510D2506
-P 5800 2300
-F 0 "R2" V 5880 2300 50  0000 C CNN
-F 1 "1k" V 5800 2300 50  0000 C CNN
-	1    5800 2300
+P 5850 2400
+F 0 "R2" V 5930 2400 50  0000 C CNN
+F 1 "1k" V 5850 2400 50  0000 C CNN
+	1    5850 2400
 	0    -1   -1   0
 $EndComp
@@
 L ZXGD3005E6 U2
 U 1 1 510D2505
-P 6600 2300
-F 0 "U2" H 6400 2500 60  0000 C CNN
-F 1 "ZXGD3005E6" H 6600 2000 60  0000 C CNN
-F 2 "SOT26" H 6750 2500 60  0001 C CNN
-	1    6600 2300
+P 6650 2400
+F 0 "U2" H 6450 2600 60  0000 C CNN
+F 1 "ZXGD3005E6" H 6650 2100 60  0000 C CNN
+F 2 "SOT26" H 6800 2600 60  0001 C CNN
+	1    6650 2400
 	1    0    0    -1
 $EndComp
@@
 L ZXGD3005E6 U3
 U 1 1 510D2504
-P 6600 3050
-F 0 "U3" H 6400 3250 60  0000 C CNN
-F 1 "ZXGD3005E6" H 6600 2750 60  0000 C CNN
-F 2 "SOT26" H 6750 3250 60  0001 C CNN
-	1    6600 3050
+P 6650 3300
+F 0 "U3" H 6450 3500 60  0000 C CNN
+F 1 "ZXGD3005E6" H 6650 3000 60  0000 C CNN
+F 2 "SOT26" H 6800 3500 60  0001 C CNN
+	1    6650 3300
 	1    0    0    -1
 $EndComp
@@
 L R R3
 U 1 1 510D2503
-P 5800 3050
-F 0 "R3" V 5880 3050 50  0000 C CNN
-F 1 "1k" V 5800 3050 50  0000 C CNN
-	1    5800 3050
+P 5850 3300
+F 0 "R3" V 5930 3300 50  0000 C CNN
+F 1 "1k" V 5850 3300 50  0000 C CNN
+	1    5850 3300
 	0    -1   -1   0
 $EndComp
@@
 L +12V #PWR023
 U 1 1 510D2502
-P 5950 2800
-F 0 "#PWR023" H 5950 2750 20  0001 C CNN
-F 1 "+12V" H 5950 2900 30  0000 C CNN
-	1    5950 2800
+P 6000 3050
+F 0 "#PWR023" H 6000 3000 20  0001 C CNN
+F 1 "+12V" H 6000 3150 30  0000 C CNN
+	1    6000 3050
 	1    0    0    -1
 $EndComp
@@
 L GND #PWR024
 U 1 1 510D2501
-P 5950 3350
-F 0 "#PWR024" H 5950 3350 30  0001 C CNN
-F 1 "GND" H 5950 3280 30  0001 C CNN
-	1    5950 3350
-	1    0    0    -1
-$EndComp
-Wire Wire Line
-	5300 3050 5550 3050
-Wire Wire Line
-	5950 2050 5950 2200
-Wire Wire Line
-	5950 2200 6100 2200
-Wire Wire Line
-	7100 2200 7250 2200
-Wire Wire Line
-	7250 2200 7250 2400
-Wire Wire Line
-	7250 2400 7100 2400
-Wire Wire Line
-	6050 2300 6100 2300
-Wire Wire Line
-	7400 2300 7250 2300
-Connection ~ 7250 2300
-Wire Wire Line
-	6100 2400 5950 2400
-Wire Wire Line
-	5950 2400 5950 2600
-Wire Wire Line
-	5950 1750 5950 1550
-Wire Wire Line
-	5950 1550 6100 1550
-Connection ~ 7250 1450
-Wire Wire Line
-	7400 1450 7250 1450
-Wire Wire Line
-	6050 1450 6100 1450
-Wire Wire Line
-	5300 1450 5550 1450
-Wire Wire Line
-	7100 1550 7250 1550
-Wire Wire Line
-	7250 1550 7250 1350
-Wire Wire Line
-	7250 1350 7100 1350
-Wire Wire Line
-	6100 1350 5950 1350
-Wire Wire Line
-	5950 1350 5950 1200
-Wire Wire Line
-	5300 2300 5550 2300
-Wire Wire Line
-	5950 3350 5950 3150
-Wire Wire Line
-	5950 3150 6100 3150
-Connection ~ 7250 3050
-Wire Wire Line
-	7400 3050 7250 3050
-Wire Wire Line
-	6050 3050 6100 3050
-Wire Wire Line
-	7100 3150 7250 3150
-Wire Wire Line
-	7250 3150 7250 2950
-Wire Wire Line
-	7250 2950 7100 2950
-Wire Wire Line
-	6100 2950 5950 2950
-Wire Wire Line
-	5950 2950 5950 2800
+P 6000 3600
+F 0 "#PWR024" H 6000 3600 30  0001 C CNN
+F 1 "GND" H 6000 3530 30  0001 C CNN
+	1    6000 3600
+	1    0    0    -1
+$EndComp
+Wire Wire Line
+	5350 3300 5600 3300
+Wire Wire Line
+	6000 2150 6000 2300
+Wire Wire Line
+	6000 2300 6150 2300
+Wire Wire Line
+	7150 2300 7300 2300
+Wire Wire Line
+	7300 2300 7300 2500
+Wire Wire Line
+	7300 2500 7150 2500
+Wire Wire Line
+	6100 2400 6150 2400
+Wire Wire Line
+	7450 2400 7300 2400
+Connection ~ 7300 2400
+Wire Wire Line
+	6150 2500 6000 2500
+Wire Wire Line
+	6000 2500 6000 2700
+Wire Wire Line
+	6000 1700 6000 1500
+Wire Wire Line
+	6000 1500 6150 1500
+Connection ~ 7300 1400
+Wire Wire Line
+	7450 1400 7300 1400
+Wire Wire Line
+	6100 1400 6150 1400
+Wire Wire Line
+	5350 1400 5600 1400
+Wire Wire Line
+	7150 1500 7300 1500
+Wire Wire Line
+	7300 1500 7300 1300
+Wire Wire Line
+	7300 1300 7150 1300
+Wire Wire Line
+	6150 1300 6000 1300
+Wire Wire Line
+	6000 1300 6000 1150
+Wire Wire Line
+	5350 2400 5600 2400
+Wire Wire Line
+	6000 3600 6000 3400
+Wire Wire Line
+	6000 3400 6150 3400
+Connection ~ 7300 3300
+Wire Wire Line
+	7450 3300 7300 3300
+Wire Wire Line
+	6100 3300 6150 3300
+Wire Wire Line
+	7150 3400 7300 3400
+Wire Wire Line
+	7300 3400 7300 3200
+Wire Wire Line
+	7300 3200 7150 3200
+Wire Wire Line
+	6150 3200 6000 3200
+Wire Wire Line
+	6000 3200 6000 3050
 Text GLabel 1550 2200 0    60   Output ~ 0
 X-MAX
