File: RAMPS-FD/RAMPS-FD.sch (KiCad schematic (older format))
At the start: 16 parts, among them P101 CONN_4, P102 VCC, P103 PS-ON, P104 5V, P105 12V-AUX, P106 CONN_3X2, SW101 SW_PUSH

Commit message: RAMPS-FD update
Parts:
- added M101: LOGO_OSHW, OSHW_logo_2, symbol LOGO_OSHW
- C101: value CP1 -> 100u
- C102: value C -> 100n
- D101: value LED -> LED GRN
Other:
- moved on the sheet: C101, C102, D102, D103, P103, P104

Commit message: First version of RAMPS-FD, RIB
Parts:
- removed P101: CONN_4, symbol CONN_4
- added F103: FUSE 10A, symbol FUSE
- added J101, J103: NET-TIE, TIE-1MM, symbol NET-TIE
- added JP101: VSEL, symbol JUMP_MINI_3
- added P101: HB_IN, symbol CONN_2
- added P107: MOT_IN, symbol CONN_2
- added P108: POWER_IN, symbol CONN_2
- F101: value MFR1100 -> FUSE 15A
- F102: value MFR500 -> FUSE 10A
Connections:
- net labels added: +V_HEATBED, +V_LOGIC, +V_MOTOR, +V_POWER, /ESTOP, A6, A7, D51, E2_DIR, E2_EN, E2_STEP, FET4, GNDPWR, HB_GND, HB_IN, MOT_GND, MOT_IN, P_IN, SERVO1, SERVO2, SERVO3, SERVO4, THERM3, UART_RX_LVC, UART_TX_LVC, VCC
- net labels removed: +12P, +12V, A10, A11, A12, A3, A9, D11, D12, D16, D17, D32, D4, D40, D42, D44, D5, D6, SER1, SER2, SER3, SER4, UART_RX, UART_TX
- wire segments 133 -> 150
- no-connect marks 10 -> 11
Other:
- note added: "5V standby?"
- note added: "Extruder heaters, fans,\nDue/Mega input\n9-15V"
- note added: "Heatbed Only: 12-24V, 15A"
- note added: "Motors only, 12-24V"
- note added: "Note: On R3 compatible Arduinos, IOREF \nwill supply 3.3V (Due), or 5V (Mega).\n\nIf IOREF is not provided (non-R3) then it \nmust be a 5V Arduino so set VSEL to 5V.\n\nIf not 5V then need to get 3.3V from somewhere ..."
- note added: "VSEL - Select logic voltage\n1-2 = Autoselect by IOREF\n2-3 = 5V"
- note added: "X/Y/Z pins \non one port"
- moved on the sheet: C101, C102, D101, D102, D103, F101, F102, M101, P102, P103, P104, P105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

Commit message: RAMPS-FD update
Parts:
- removed C101: 100u, symbol CP1
- removed C102: 100n, symbol C
- removed D102, D103: 1N4004, symbol DIODE
- removed F101: FUSE 15A, symbol FUSE
- removed F102, F103: FUSE 10A, symbol FUSE
- removed J101, J103: NET-TIE, TIE-1MM, symbol NET-TIE
- removed JP101: VSEL, symbol JUMP_MINI_3
- removed P101: HB_IN, symbol CONN_2
- removed P102: VCC, symbol CONN_1
- removed P103: PS-ON, symbol CONN_1
- removed P104: 5V, symbol CONN_1
- removed P105: 12V-AUX, symbol CONN_2
- removed P107: MOT_IN, symbol CONN_2
- removed P108: POWER_IN, symbol CONN_2
- R101: value 1k -> 56R
Connections:
- net AUX_UART_TX_LV: now reaches SHIELD101.18 (D18-TX1)
- net AUX_UART_RX_LV: now reaches SHIELD101.19 (D19-RX1)
- net D42: now reaches SHIELD101.42 (D42)
- net D50: now reaches SHIELD101.50 (D50-MISO)
- net D52: now reaches SHIELD101.52 (D52-SCK)
- net AD14: now reaches SHIELD101.AD14 (AD14-CANRX)
- net AD15: now reaches SHIELD101.AD15 (AD15-CANTX)
- net SCL1: now reaches SHIELD101.SCL1
- net SDA1: now reaches SHIELD101.SDA1
- net UART_RX_LVC renamed UART_RX_LV
- net UART_TX_LVC renamed UART_TX_LV
- no-connect marks 11 -> 2
Other:
- note added: "Also used by\nProgramming USB port"
- note removed: "5V standby?"
- note removed: "Extruder heaters, fans,\nDue/Mega input\n9-15V"
- note removed: "Heatbed Only: 12-24V, 15A"
- note removed: "Motors only, 12-24V"
- note removed: "Note: On R3 compatible Arduinos, IOREF \nwill supply 3.3V (Due), or 5V (Mega).\n\nIf IOREF is not provided (non-R3) then it \nmust be a 5V Arduino so set VSEL to 5V.\n\nIf not 5V then need to get 3.3V from somewhere ..."
- note removed: "Or 3V3?"
- note removed: "Power"
- note removed: "VSEL - Select logic voltage\n1-2 = Autoselect by IOREF\n2-3 = 5V"
- moved on the sheet: D101, M101, P106, R101, SHIELD101, SW101

Commit message: Updates to RAMPS-FD
Parts:
- added M102: PCB_GREEN_RMC, symbol PCB_GREEN_RMC
Connections:
- net D42 is gone; now on net E0_EN: SHIELD101.42 (D42)
- net E2_DIR is gone; now on net E0_STEP: SHIELD101.36 (D36)
- net E2_EN is gone; now on net E0_DIR: SHIELD101.28 (D28)
- net E2_STEP is gone; now on net PS-ON: SHIELD101.38 (D38)
- net E0_DIR: no longer SHIELD101.2 (D2)
- net E0_EN: no longer SHIELD101.14 (D14-TX3)
- net E0_STEP: no longer SHIELD101.3 (D3)
- net PS-ON: no longer SHIELD101.12 (D12)
- net SERVO4: now also SHIELD101.3 (D3); no longer SHIELD101.4 (D4)
- net /ESTOP renamed ESTOP
- net AUX_UART_RX_LV renamed UART1_RX_LV
- net AUX_UART_TX_LV renamed UART1_TX_LV
- net D50 renamed D50-MISO
- net D51 renamed D51-MOSI
- net D52 renamed D52-SCK
- net D53 renamed D53-SS
- net E1_DIR renamed UART3_RX_LV
- net E1_EN renamed UART2_RX_LV
- net E1_STEP renamed UART2_TX_LV
- net UART_RX_LV renamed UART0_RX_LV
- net UART_TX_LV renamed UART0_TX_LV
- new net D11-FET5: SHIELD101.12 (D12)
- new net D2-FET6: SHIELD101.2 (D2)
- new net SPI_CS1: SHIELD101.4 (D4)
- new net UART3_TX_LV: SHIELD101.14 (D14-TX3)
Other:
- note added: "Fit P106 on Due version only, not compatible with Mega"
- note added: "X/Y/Z pins are\non single port for both\nMega and Due"
- note removed: "X/Y/Z pins \non one port"
Changed lines of the file:
@@
-EESchema Schematic File Version 2  date 19/09/2013 22:01:21
+EESchema Schematic File Version 2
 LIBS:power
 LIBS:device
@@
 LIBS:opendous
 LIBS:RAMPS-FD-cache
-EELAYER 25  0
+EELAYER 27 0
 EELAYER END
-$Descr A4 11700 8267
+$Descr A4 11693 8268
 encoding utf-8
-Sheet 1 8
+Sheet 1 9
 Title "RAMPS-FD (RAMPS for Arduino Due)"
-Date "19 sep 2013"
+Date "22 sep 2013"
 Rev "0.2"
 Comp ""
@@
 Text GLabel 900  4150 0    50   Input ~ 0
 AD15
-Text GLabel 1000 4750 0    50   BiDi ~ 0
-D52
-Text GLabel 1000 4950 0    50   BiDi ~ 0
-D50
-Text GLabel 1000 5800 0    50   BiDi ~ 0
-D42
+Text GLabel 1450 4750 0    50   BiDi ~ 0
+D52-SCK
+Text GLabel 1450 4950 0    50   BiDi ~ 0
+D50-MISO
 Text GLabel 4350 1250 2    50   BiDi ~ 0
 SDA1
@@
 Also used by\nProgramming USB port
 Text GLabel 4750 3750 2    50   Input ~ 0
-AUX_UART_RX_LV
+UART1_RX_LV
 Text GLabel 4750 3650 2    50   Output ~ 0
-AUX_UART_TX_LV
+UART1_TX_LV
 Text GLabel 2000 1650 0    50   Output ~ 0
 IOREF
@@
 	1450 3850 2200 3850
 Wire Wire Line
-	1000 5800 2200 5800
+	1450 5800 2200 5800
 Connection ~ 1050 2050
 Wire Wire Line
@@
 	4100 6250 4350 6250
 Wire Wire Line
-	4350 5850 4100 5850
-Wire Wire Line
-	4350 5650 4100 5650
-Wire Wire Line
-	4100 5200 4350 5200
-Wire Wire Line
-	4350 4800 4100 4800
+	4100 5850 5400 5850
+Wire Wire Line
+	4100 5650 5400 5650
+Wire Wire Line
+	4100 5200 5400 5200
+Wire Wire Line
+	4100 4800 5400 4800
 Wire Wire Line
 	1850 5950 2200 5950
@@
 	4750 3250 4100 3250
 Wire Wire Line
-	4750 2850 4100 2850
+	4100 2850 5100 2850
 Wire Wire Line
 	4750 2150 4100 2150
@@
 	1450 5400 2200 5400
 Wire Wire Line
-	2200 1950 1350 1950
+	1350 1950 2200 1950
 Wire Wire Line
 	4100 6150 4800 6150
@@
 	4200 4500 4100 4500
 Wire Wire Line
-	2200 4500 1600 4500
+	1600 4500 2200 4500
 Wire Wire Line
 	1600 4500 1600 4550
@@
 	4800 5100 4100 5100
 Wire Wire Line
-	1000 4750 2200 4750
-Wire Wire Line
-	1000 4950 2200 4950
-Wire Wire Line
-	1850 4850 2200 4850
+	1450 4750 2200 4750
+Wire Wire Line
+	1450 4950 2200 4950
+Wire Wire Line
+	1450 4850 2200 4850
 Wire Wire Line
 	2200 1650 2000 1650
@@
 	4750 2050 4100 2050
 Wire Wire Line
-	5150 1750 4100 1750
+	5100 1750 4100 1750
 Wire Wire Line
 	4750 2750 4100 2750
@@
 	2200 5600 1450 5600
 Wire Wire Line
-	1850 4650 2200 4650
+	1450 4650 2200 4650
 Wire Wire Line
 	4100 3550 4750 3550
@@
 	2200 6150 1850 6150
 Wire Wire Line
-	4350 5000 4100 5000
-Wire Wire Line
-	4350 5400 4100 5400
+	4100 5000 5400 5000
+Wire Wire Line
+	4100 5400 5400 5400
 Wire Wire Line
 	4100 5750 4800 5750
@@
 	900  3400 1100 3400
 Text GLabel 1450 6050 0    50   Input ~ 0
-/ESTOP
+ESTOP
 $Sheet
 S 8150 850  950  400
@@
 F1 "steppers2.sch" 60
 $EndSheet
-Text Notes 400  3550 0    50   ~ 0
-X/Y/Z pins \non one port
+Text Notes 500  3150 0    50   ~ 0
+X/Y/Z pins are\non single port for both\nMega and Due
 $Comp
 L ARDUINO_DUE_SHIELD SHIELD101
@@
 F 0 "SHIELD101" H 2800 6650 60  0000 C CNN
 F 1 "ARDUINO_DUE_SHIELD" H 3100 1100 60  0000 C CNN
+F 2 "" H 3200 3800 60  0001 C CNN
+F 3 "" H 3200 3800 60  0001 C CNN
 	1    3200 3800
 	1    0    0    -1
 $EndComp
-Text GLabel 1850 4850 0    50   BiDi ~ 0
-D51
-Text GLabel 5150 1750 2    50   Output ~ 0
+Text GLabel 1450 4850 0    50   BiDi ~ 0
+D51-MOSI
+Text GLabel 1450 6250 0    50   Output ~ 0
 PS-ON
 Text GLabel 1800 3250 0    50   Input ~ 0
@@
 F1 "con_misc.sch" 60
 $EndSheet
-Text GLabel 1450 6250 0    50   Output ~ 0
+Text GLabel 5400 5650 2    50   Output ~ 0
 E2_STEP
-Text GLabel 4800 6150 2    50   Output ~ 0
+Text GLabel 5400 5400 2    50   Output ~ 0
 E2_DIR
-Text GLabel 4800 5300 2    50   Output ~ 0
+Text GLabel 5400 5850 2    50   Output ~ 0
 E2_EN
 $Sheet
@@
 F 1 "LOGO_OSHW" H 10700 5900 60  0000 C CNN
 F 2 "OSHW_logo_2" H 10600 6050 60  0000 C CNN
+F 3 "" H 10700 6000 60  0001 C CNN
 	1    10700 6000
 	1    0    0    -1
@@
 Text GLabel 1850 5300 0    50   BiDi ~ 0
 D47
-Text GLabel 1850 4650 0    50   BiDi ~ 0
-D53
+Text GLabel 1450 4650 0    50   BiDi ~ 0
+D53-SS
 Text GLabel 1850 5100 0    50   BiDi ~ 0
 D49
@@
 F 0 "#PWR01" H 3700 7450 30  0001 C CNN
 F 1 "GND" H 3700 7380 30  0001 C CNN
+F 2 "" H 3700 7450 60  0001 C CNN
+F 3 "" H 3700 7450 60  0001 C CNN
 	1    3700 7450
 	1    0    0    -1
@@
 F 0 "#PWR02" H 3750 7140 20  0001 C CNN
 F 1 "+5V" H 3750 7140 30  0000 C CNN
+F 2 "" H 3750 7050 60  0001 C CNN
+F 3 "" H 3750 7050 60  0001 C CNN
 	1    3750 7050
 	1    0    0    -1
@@
 F 0 "P106" H 3100 7500 50  0000 C CNN
 F 1 "CONN_3X2" V 3100 7300 40  0000 C CNN
+F 2 "" H 3100 7250 60  0001 C CNN
+F 3 "" H 3100 7250 60  0001 C CNN
 	1    3100 7250
 	1    0    0    -1
@@
 A4
 Text GLabel 4750 3050 2    50   Input ~ 0
-UART_RX_LV
+UART0_RX_LV
 Text GLabel 4750 2950 2    50   Output ~ 0
-UART_TX_LV
+UART0_TX_LV
 Text GLabel 4750 3950 2    50   Output ~ 0
 SCL
@@
 Text GLabel 4750 2550 2    50   Output ~ 0
 SERVO3
-Text GLabel 4750 2650 2    50   Output ~ 0
+Text GLabel 4750 2750 2    50   Output ~ 0
 SERVO4
 $Sheet
@@
 F 0 "#FLG03" H 1350 2045 30  0001 C CNN
 F 1 "PWR_FLAG" H 1350 2130 30  0000 C CNN
+F 2 "" H 1350 1950 60  0001 C CNN
+F 3 "" H 1350 1950 60  0001 C CNN
 	1    1350 1950
 	1    0    0    -1
@@
 F 0 "#FLG04" H 900 2145 30  0001 C CNN
 F 1 "PWR_FLAG" H 900 2230 30  0000 C CNN
+F 2 "" H 900 2050 60  0001 C CNN
+F 3 "" H 900 2050 60  0001 C CNN
 	1    900  2050
 	1    0    0    -1
 $EndComp
 NoConn ~ 4100 1450
-Text GLabel 4750 3450 2    50   Output ~ 0
+Text GLabel 5400 5000 2    50   Output ~ 0
 E1_STEP
 Text GLabel 1450 5200 0    50   Output ~ 0
 X_EN
-Text GLabel 4750 3350 2    50   Output ~ 0
+Text GLabel 5400 4800 2    50   Output ~ 0
 E1_DIR
-Text GLabel 4750 3550 2    50   Output ~ 0
+Text GLabel 5400 5200 2    50   Output ~ 0
 E1_EN
-Text GLabel 4750 2850 2    50   Output ~ 0
+Text GLabel 4800 5300 2    50   Output ~ 0
 E0_DIR
-Text GLabel 4750 2750 2    50   Output ~ 0
+Text GLabel 4800 6150 2    50   Output ~ 0
 E0_STEP
-Text GLabel 4750 3250 2    50   Output ~ 0
+Text GLabel 1450 5800 0    50   Output ~ 0
 E0_EN
 Text GLabel 1450 2750 0    50   Input ~ 0
@@
 F 0 "#PWR05" H 8650 5800 30  0001 C CNN
 F 1 "GND" H 8650 5730 30  0001 C CNN
+F 2 "" H 8650 5800 60  0001 C CNN
+F 3 "" H 8650 5800 60  0001 C CNN
 	1    8650 5800
 	1    0    0    -1
@@
 F 0 "SW101" H 8800 5210 50  0000 C CNN
 F 1 "SW_PUSH" H 8650 5020 50  0000 C CNN
+F 2 "" H 8650 5100 60  0001 C CNN
+F 3 "" H 8650 5100 60  0001 C CNN
 	1    8650 5100
 	0    1    1    0
@@
 F 0 "#PWR06" H 7750 5800 30  0001 C CNN
 F 1 "GND" H 7750 5730 30  0001 C CNN
+F 2 "" H 7750 5800 60  0001 C CNN
+F 3 "" H 7750 5800 60  0001 C CNN
 	1    7750 5800
 	1    0    0    -1
@@
 F 0 "D101" H 7750 5500 50  0000 C CNN
 F 1 "LED GRN" H 7750 5300 50  0000 C CNN
+F 2 "" H 7750 5400 60  0001 C CNN
+F 3 "" H 7750 5400 60  0001 C CNN
 	1    7750 5400
 	0    1    1    0
@@
 F 0 "R101" V 7830 4850 50  0000 C CNN
 F 1 "56R" V 7750 4850 50  0000 C CNN
+F 2 "" H 7750 4850 60  0001 C CNN
+F 3 "" H 7750 4850 60  0001 C CNN
 	1    7750 4850
 	1    0    0    -1
@@
 F 0 "#PWR07" H 1550 1660 30  0001 C CNN
 F 1 "+3.3V" H 1550 1810 30  0000 C CNN
+F 2 "" H 1550 1700 60  0001 C CNN
+F 3 "" H 1550 1700 60  0001 C CNN
 	1    1550 1700
 	1    0    0    -1
@@
 F 0 "#PWR08" H 1400 2350 30  0001 C CNN
 F 1 "GND" H 1400 2280 30  0001 C CNN
+F 2 "" H 1400 2350 60  0001 C CNN
+F 3 "" H 1400 2350 60  0001 C CNN
 	1    1400 2350
 	1    0    0    -1
@@
 F 0 "#PWR09" H 1050 1790 20  0001 C CNN
 F 1 "+5V" H 1050 1790 30  0000 C CNN
+F 2 "" H 1050 1700 60  0001 C CNN
+F 3 "" H 1050 1700 60  0001 C CNN
 	1    1050 1700
 	1    0    0    -1
@@
 F 0 "#PWR010" H 4650 1600 30  0001 C CNN
 F 1 "GND" H 4650 1530 30  0001 C CNN
+F 2 "" H 4650 1600 60  0001 C CNN
+F 3 "" H 4650 1600 60  0001 C CNN
 	1    4650 1600
 	1    0    0    -1
@@
 F 0 "#PWR011" H 1600 4550 30  0001 C CNN
 F 1 "GND" H 1600 4480 30  0001 C CNN
+F 2 "" H 1600 4550 60  0001 C CNN
+F 3 "" H 1600 4550 60  0001 C CNN
 	1    1600 4550
 	1    0    0    -1
@@
 F 0 "#PWR012" H 4350 4440 20  0001 C CNN
 F 1 "+5V" H 4350 4440 30  0000 C CNN
+F 2 "" H 4350 4350 60  0001 C CNN
+F 3 "" H 4350 4350 60  0001 C CNN
 	1    4350 4350
 	1    0    0    -1
 $EndComp
+$Comp
+L PCB_GREEN_RMC M102
+U 1 1 523E4D4E
+P 10700 5200
+F 0 "M102" H 10700 5350 60  0000 C CNN
+F 1 "PCB_GREEN_RMC" H 10700 5100 60  0000 C CNN
+F 2 "" H 10700 5200 60  0000 C CNN
+F 3 "" H 10700 5200 60  0000 C CNN
+	1    10700 5200
+	1    0    0    -1
+$EndComp
+Text GLabel 4750 2650 2    50   Output ~ 0
+SPI_CS1
+Text GLabel 4750 3350 2    50   Input ~ 0
+UART3_RX_LV
+Text GLabel 4750 3250 2    50   Output ~ 0
+UART3_TX_LV
+Text GLabel 4750 3550 2    50   Input ~ 0
+UART2_RX_LV
+Text GLabel 4750 3450 2    50   Output ~ 0
+UART2_TX_LV
+Wire Notes Line
+	5650 1650 5900 1650
+Text GLabel 5100 1750 2    50   Output ~ 0
+D11-FET5
+Text GLabel 5100 2850 2    50   Output ~ 0
+D2-FET6
+$Sheet
+S 8150 2950 950  400
+U 523E5F7E
+F0 "Extra MOSFETs" 50
+F1 "Extra_Mosfets.sch" 50
+$EndSheet
+Wire Notes Line
+	900  3700 700  3700
+Wire Notes Line
+	700  3700 700  3350
+Text Notes 2050 7650 0    50   ~ 0
+Fit P106 on Due version only, not compatible with Mega
 $EndSCHEMATC

Commit message: RAMPS-FD latest updates
Parts:
- R101: value 56R -> 150R
Connections:
- net D11-FET5 renamed D12-FET5
- net FET4 renamed D11-FET4
Other:
- note removed: "Fit P106 on Due version only, not compatible with Mega"
Changed lines of the file:
@@
 Sheet 1 9
 Title "RAMPS-FD (RAMPS for Arduino Due)"
-Date "22 sep 2013"
+Date "23 sep 2013"
 Rev "0.2"
 Comp ""
@@
 	4750 3250 4100 3250
 Wire Wire Line
-	4100 2850 5100 2850
+	4100 2850 4750 2850
 Wire Wire Line
 	4750 2150 4100 2150
@@
 	4750 2050 4100 2050
 Wire Wire Line
-	5100 1750 4100 1750
+	4750 1750 4100 1750
 Wire Wire Line
 	4750 2750 4100 2750
@@
 $EndSheet
 Text GLabel 4750 1850 2    50   Output ~ 0
-FET4
+D11-FET4
 $Comp
 L LOGO_OSHW M101
@@
 P 7750 4850
 F 0 "R101" V 7830 4850 50  0000 C CNN
-F 1 "56R" V 7750 4850 50  0000 C CNN
+F 1 "150R" V 7750 4850 50  0000 C CNN
 F 2 "" H 7750 4850 60  0001 C CNN
 F 3 "" H 7750 4850 60  0001 C CNN
@@
 Wire Notes Line
 	5650 1650 5900 1650
-Text GLabel 5100 1750 2    50   Output ~ 0
-D11-FET5
-Text GLabel 5100 2850 2    50   Output ~ 0
+Text GLabel 4750 1750 2    50   Output ~ 0
+D12-FET5
+Text GLabel 4750 2850 2    50   Output ~ 0
 D2-FET6
 $Sheet
@@
 Wire Notes Line
 	700  3700 700  3350
-Text Notes 2050 7650 0    50   ~ 0
-Fit P106 on Due version only, not compatible with Mega
 $EndSCHEMATC

Commit message: RAMPS-FD: latest update
Connections:
- net Y-MAX renamed D32
