File: RAMPS-FD/con_outputs.sch (KiCad schematic (older format))
At the start: 30 parts, among them K201 SER1, K202 SER2, K203 SER3, K204 SER4, P211 CONN_4, P212 CONN_6, P213 AUX-4, P214 AUX-2, P215 AUX-3, P216 SERIAL, P217 A-OUT, Q201 STP55NF06L, Q202 STP55NF06L, Q203 STP55NF06L

Commit message: RAMPS-FD update
Parts:
- removed Q201, Q202, Q203: STP55NF06L, symbol MOS_N
- removed R217: 10k, symbol R
- removed R218: 100k, symbol R
- added Q201, Q202, Q203: STP55NF06L, symbol MOSFET_N_RMC
- added Q301: 2N7002, symbol MOS_N
- added R304: 10k, symbol R
- D201, D202, D203: value LED -> LED RED
- gave numbers to parts that had none: 4
Connections:
- wire segments 138 -> 139
Other:
- note added: "NB: inverting driver"
- note removed: "NB: inverted driver"
- moved on the sheet: D201, D202, D203, P211, P212, Q204, R213, R214, R215, R216, R219, R220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

Commit message: First version of RAMPS-FD, RIB
Parts:
- removed K201: SER1, symbol CONN_3
- removed K202: SER2, symbol CONN_3
- removed K203: SER3, symbol CONN_3
- removed K204: SER4, symbol CONN_3
- removed P211: CONN_4, symbol CONN_4
- removed P212: CONN_6, symbol CONN_6
- removed P213: AUX-4, symbol CONN_18
- removed P214: AUX-2, symbol CONN_5X2
- removed P215: AUX-3, symbol CONN_4X2
- removed P216: SERIAL, symbol CONN_4
- removed P217: A-OUT, symbol CONN_4
- removed Q301: 2N7002, symbol MOS_N
- removed R211, R212: NF, symbol R
- removed R213: 1k, symbol R
- removed R216: 10, symbol R
- removed R304: 10k, symbol R
- removed U206: ZXGD3005E6, SOT26, symbol ZXGD3005E6
- added D204: LED RED, symbol LED
- added D401, D402, D403, D404: ES1F, symbol DIODE
- added J401, J402: NET-TIE, TIE-1MM, symbol NET-TIE
- added P218: AUX2, symbol CONN_2
- added P403: D9_EXT, symbol CONN_2
- added P404: D8_HB, symbol CONN_2
- added P405: D10_AUX, symbol CONN_2
- added Q205, Q501, Q502: 2N7002, symbol MOS_N
- added Q206: IRLB8743PBF, symbol MOSFET_N_RMC
- added R217, R508, R509: 10, symbol R
- added R218, R405, R406, R506, R507, R510, R511: 10k, symbol R
- added R222: 1k8, symbol R
- Q201, Q202, Q203: value STP55NF06L -> IRLB8743PBF
Connections:
- net labels added: +V_HEATBED, +V_LOGIC, +V_POWER, D10_OUT, D8_BUF, D8_OUT, D9_BUF, D9_OUT, FET4, FET4_OUT, GNDPWR, HB_GND, POWER_SIG
- net labels removed: +12P, +12V, +3.3V, +5V, A10, A11, A12, A3, A4, A5, A9, D11, D16, D17, D23, D25, D27, D29, D31, D32, D33, D35, D37, D39, D4, D40, D41, D42, D43, D44, D45, D47, D49, D5, D53, D6, D8, D9, MISO, MOSI, SCK, SCL, SDA, UART_RX, UART_TX
- wire segments 139 -> 78
- no-connect marks 1 -> 0
Other:
- note added: "D10 - Extruder 2 / Fan"
- note added: "D8 - Heatbed"
- note added: "D9 - Extruder 1"
- note added: "FET4 - Extruder 3 / Fan"
- note added: "MOSFET Outputs"
- note added: "NB: inverting drivers"
- note removed: "1k5 Pull ups on Due"
- note removed: "Aux connectors"
- note removed: "Aux-1"
- note removed: "Aux2"
- note removed: "Aux3-SPI"
- note removed: "Aux4"
- note removed: "Heaters and Fans"
- note removed: "I2C"
- note removed: "Must not have external pullups to 5V"
- note removed: "NB: inverting driver"
- note removed: "Need buffered outputs?"
- note removed: "Non-inverting gate driver"
- note removed: "Servos"
- note removed: "Should these be 5V?"
- note removed: "TTL-3V3 only"
- moved on the sheet: D201, D202, D203, Q201, Q202, Q203, Q204, R214, R215, R219, R220, R221

Commit message: RAMPS-FD update
Parts:
- removed J401, J402: NET-TIE, TIE-1MM, symbol NET-TIE
- removed R405, R406, R506, R507: 10k, symbol R
- removed R508, R509: 10, symbol R
- R215, R217: value 10 -> 10R
Connections:
- net POWER_SIG is gone; now on net V_GATE: R214.1, R218.1, R220.1, R221.1, R222.1, R511.1
- net V_GATE: now reaches R219.1, R510.1
- net /D9_BUF: now reaches Q502.G
- net /D8_BUF: now reaches Q501.G
- net D10 renamed /D10_BUF
- net FET4 renamed /FET4_BUF

Commit message: Updates to RAMPS-FD
Parts:
- P218: value AUX2 -> EXT3
- P405: value D10_AUX -> D10_EXT1
Changed lines of the file:
@@
-EESchema Schematic File Version 2  date 19/09/2013 22:01:21
+EESchema Schematic File Version 2
 LIBS:power
 LIBS:device
@@
 LIBS:opendous
 LIBS:RAMPS-FD-cache
-EELAYER 25  0
+EELAYER 27 0
 EELAYER END
-$Descr A4 11700 8267
+$Descr A4 11693 8268
 encoding utf-8
-Sheet 7 8
+Sheet 7 9
 Title ""
-Date "19 sep 2013"
+Date "22 sep 2013"
 Rev "0.2"
 Comp ""
@@
 Wire Wire Line
 	9600 1200 9600 650
-Connection ~ 9600 850
 Connection ~ 3650 850
 Wire Wire Line
@@
 F 0 "#PWR087" H 2150 3100 30  0001 C CNN
 F 1 "GND" H 2150 3030 30  0001 C CNN
+F 2 "" H 2150 3100 60  0001 C CNN
+F 3 "" H 2150 3100 60  0001 C CNN
 	1    2150 3100
 	1    0    0    -1
@@
 F 0 "R510" V 2230 1750 50  0000 C CNN
 F 1 "10k" V 2150 1750 50  0000 C CNN
+F 2 "" H 2150 1750 60  0001 C CNN
+F 3 "" H 2150 1750 60  0001 C CNN
 	1    2150 1750
 	1    0    0    -1
@@
 F 0 "Q501" H 2060 2920 60  0000 R CNN
 F 1 "2N7002" H 2500 2750 60  0000 R CNN
+F 2 "" H 2050 2750 60  0001 C CNN
+F 3 "" H 2050 2750 60  0001 C CNN
 	1    2050 2750
 	1    0    0    -1
@@
 F 0 "Q502" H 2110 6220 60  0000 R CNN
 F 1 "2N7002" H 2550 6050 60  0000 R CNN
+F 2 "" H 2100 6050 60  0001 C CNN
+F 3 "" H 2100 6050 60  0001 C CNN
 	1    2100 6050
 	1    0    0    -1
@@
 F 0 "R511" V 2280 5050 50  0000 C CNN
 F 1 "10k" V 2200 5050 50  0000 C CNN
+F 2 "" H 2200 5050 60  0001 C CNN
+F 3 "" H 2200 5050 60  0001 C CNN
 	1    2200 5050
 	1    0    0    -1
@@
 F 0 "#PWR088" H 2200 6400 30  0001 C CNN
 F 1 "GND" H 2200 6330 30  0001 C CNN
+F 2 "" H 2200 6400 60  0001 C CNN
+F 3 "" H 2200 6400 60  0001 C CNN
 	1    2200 6400
 	1    0    0    -1
@@
 F 0 "#PWR089" H 9300 3050 40  0001 C CNN
 F 1 "GNDPWR" H 9300 2920 40  0000 C CNN
+F 2 "" H 9300 3000 60  0001 C CNN
+F 3 "" H 9300 3000 60  0001 C CNN
 	1    9300 3000
 	1    0    0    -1
@@
 F 0 "#PWR090" H 8400 6600 30  0001 C CNN
 F 1 "GND" H 8400 6530 30  0001 C CNN
+F 2 "" H 8400 6600 60  0001 C CNN
+F 3 "" H 8400 6600 60  0001 C CNN
 	1    8400 6600
 	1    0    0    -1
@@
 F 0 "#PWR091" H 9450 6650 40  0001 C CNN
 F 1 "GNDPWR" H 9450 6520 40  0000 C CNN
+F 2 "" H 9450 6600 60  0001 C CNN
+F 3 "" H 9450 6600 60  0001 C CNN
 	1    9450 6600
 	1    0    0    -1
@@
 F 0 "#PWR092" H 3350 6600 40  0001 C CNN
 F 1 "GNDPWR" H 3350 6470 40  0000 C CNN
+F 2 "" H 3350 6550 60  0001 C CNN
+F 3 "" H 3350 6550 60  0001 C CNN
 	1    3350 6550
 	1    0    0    -1
@@
 P 10600 5550
 F 0 "P405" V 10550 5550 40  0000 C CNN
-F 1 "D10_AUX" V 10650 5550 40  0000 C CNN
+F 1 "D10_EXT1" V 10650 5550 40  0000 C CNN
+F 2 "" H 10600 5550 60  0001 C CNN
+F 3 "" H 10600 5550 60  0001 C CNN
 	1    10600 5550
 	1    0    0    -1
@@
 F 0 "P403" V 4650 5250 40  0000 C CNN
 F 1 "D9_EXT" V 4750 5250 40  0000 C CNN
+F 2 "" H 4700 5250 60  0001 C CNN
+F 3 "" H 4700 5250 60  0001 C CNN
 	1    4700 5250
 	1    0    0    -1
@@
 F 0 "P404" V 4800 1950 40  0000 C CNN
 F 1 "D8_HB" V 4900 1950 40  0000 C CNN
+F 2 "" H 4850 1950 60  0001 C CNN
+F 3 "" H 4850 1950 60  0001 C CNN
 	1    4850 1950
 	1    0    0    -1
@@
 F 0 "D404" H 3650 1600 40  0000 C CNN
 F 1 "ES1F" H 3650 1400 40  0000 C CNN
+F 2 "" H 3650 1500 60  0001 C CNN
+F 3 "" H 3650 1500 60  0001 C CNN
 	1    3650 1500
 	0    -1   -1   0
@@
 F 0 "D403" H 9600 1500 40  0000 C CNN
 F 1 "ES1F" H 9600 1300 40  0000 C CNN
+F 2 "" H 9600 1400 60  0001 C CNN
+F 3 "" H 9600 1400 60  0001 C CNN
 	1    9600 1400
 	0    -1   -1   0
@@
 F 0 "D401" H 3350 4900 40  0000 C CNN
 F 1 "ES1F" H 3350 4700 40  0000 C CNN
+F 2 "" H 3350 4800 60  0001 C CNN
+F 3 "" H 3350 4800 60  0001 C CNN
 	1    3350 4800
 	0    -1   -1   0
@@
 F 0 "D402" H 9450 5200 40  0000 C CNN
 F 1 "ES1F" H 9450 5000 40  0000 C CNN
+F 2 "" H 9450 5100 60  0001 C CNN
+F 3 "" H 9450 5100 60  0001 C CNN
 	1    9450 5100
 	0    -1   -1   0
@@
 P 10700 1850
 F 0 "P218" V 10650 1850 40  0000 C CNN
-F 1 "AUX2" V 10750 1850 40  0000 C CNN
+F 1 "EXT3" V 10750 1850 40  0000 C CNN
+F 2 "" H 10700 1850 60  0001 C CNN
+F 3 "" H 10700 1850 60  0001 C CNN
 	1    10700 1850
 	1    0    0    -1
@@
 F 0 "D204" H 8900 1800 50  0000 C CNN
 F 1 "LED RED" H 8900 1600 50  0000 C CNN
+F 2 "" H 8900 1700 60  0001 C CNN
+F 3 "" H 8900 1700 60  0001 C CNN
 	1    8900 1700
 	0    1    1    0
@@
 F 0 "R222" V 8980 1150 50  0000 C CNN
 F 1 "1k8" V 8900 1150 50  0000 C CNN
+F 2 "" H 8900 1150 60  0001 C CNN
+F 3 "" H 8900 1150 60  0001 C CNN
 	1    8900 1150
 	1    0    0    -1
@@
 F 0 "#PWR093" H 8250 3000 30  0001 C CNN
 F 1 "GND" H 8250 2930 30  0001 C CNN
+F 2 "" H 8250 3000 60  0001 C CNN
+F 3 "" H 8250 3000 60  0001 C CNN
 	1    8250 3000
 	1    0    0    -1
@@
 F 0 "R217" V 7580 2550 50  0000 C CNN
 F 1 "10R" V 7500 2550 50  0000 C CNN
+F 2 "" H 7500 2550 60  0001 C CNN
+F 3 "" H 7500 2550 60  0001 C CNN
 	1    7500 2550
 	0    -1   -1   0
@@
 F 0 "Q205" H 8160 2720 60  0000 R CNN
 F 1 "2N7002" H 8600 2550 60  0000 R CNN
+F 2 "" H 8150 2550 60  0001 C CNN
+F 3 "" H 8150 2550 60  0001 C CNN
 	1    8150 2550
 	1    0    0    -1
@@
 F 0 "R218" V 8330 1450 50  0000 C CNN
 F 1 "10k" V 8250 1450 50  0000 C CNN
+F 2 "" H 8250 1450 60  0001 C CNN
+F 3 "" H 8250 1450 60  0001 C CNN
 	1    8250 1450
 	1    0    0    -1
@@
 F 0 "Q206" H 9125 2500 60  0000 C CNN
 F 1 "IRLB8743PBF" H 9650 2150 60  0000 C CNN
+F 2 "" H 9250 2250 60  0001 C CNN
+F 3 "" H 9250 2250 60  0001 C CNN
 	1    9250 2250
 	1    0    0    -1
@@
 F 0 "#PWR094" H 9600 620 30  0001 C CNN
 F 1 "+V_POWER" H 9600 750 30  0000 C CNN
+F 2 "" H 9600 650 60  0001 C CNN
+F 3 "" H 9600 650 60  0001 C CNN
 	1    9600 650
 	1    0    0    -1
@@
 F 0 "Q201" H 3125 2700 60  0000 C CNN
 F 1 "IRLB8743PBF" H 3650 2350 60  0000 C CNN
+F 2 "" H 3250 2450 60  0001 C CNN
+F 3 "" H 3250 2450 60  0001 C CNN
 	1    3250 2450
 	1    0    0    -1
@@
 F 0 "#PWR095" H 3350 4120 30  0001 C CNN
 F 1 "+V_POWER" H 3350 4250 30  0000 C CNN
+F 2 "" H 3350 4150 60  0001 C CNN
+F 3 "" H 3350 4150 60  0001 C CNN
 	1    3350 4150
 	1    0    0    -1
@@
 F 0 "#PWR096" H 9450 4270 30  0001 C CNN
 F 1 "+V_POWER" H 9450 4400 30  0000 C CNN
+F 2 "" H 9450 4300 60  0001 C CNN
+F 3 "" H 9450 4300 60  0001 C CNN
 	1    9450 4300
 	1    0    0    -1
@@
 F 0 "#PWR097" H 3650 670 30  0001 C CNN
 F 1 "+V_HEATBED" H 3650 800 30  0000 C CNN
+F 2 "" H 3650 700 60  0001 C CNN
+F 3 "" H 3650 700 60  0001 C CNN
 	1    3650 700
 	1    0    0    -1
@@
 F 0 "Q203" H 3175 6000 60  0000 C CNN
 F 1 "IRLB8743PBF" H 3700 5650 60  0000 C CNN
+F 2 "" H 3300 5750 60  0001 C CNN
+F 3 "" H 3300 5750 60  0001 C CNN
 	1    3300 5750
 	1    0    0    -1
@@
 F 0 "Q202" H 9275 6200 60  0000 C CNN
 F 1 "IRLB8743PBF" H 9800 5850 60  0000 C CNN
+F 2 "" H 9400 5950 60  0001 C CNN
+F 3 "" H 9400 5950 60  0001 C CNN
 	1    9400 5950
 	1    0    0    -1
@@
 F 0 "R214" V 8480 5250 50  0000 C CNN
 F 1 "10k" V 8400 5250 50  0000 C CNN
+F 2 "" H 8400 5250 60  0001 C CNN
+F 3 "" H 8400 5250 60  0001 C CNN
 	1    8400 5250
 	1    0    0    -1
@@
 F 0 "Q204" H 8310 6420 60  0000 R CNN
 F 1 "2N7002" H 8750 6250 60  0000 R CNN
+F 2 "" H 8300 6250 60  0001 C CNN
+F 3 "" H 8300 6250 60  0001 C CNN
 	1    8300 6250
 	1    0    0    -1
@@
 F 0 "D203" H 2850 5200 50  0000 C CNN
 F 1 "LED RED" H 2850 5000 50  0000 C CNN
+F 2 "" H 2850 5100 60  0001 C CNN
+F 3 "" H 2850 5100 60  0001 C CNN
 	1    2850 5100
 	0    1    1    0
@@
 F 0 "R221" V 2930 4600 50  0000 C CNN
 F 1 "1k8" V 2850 4600 50  0000 C CNN
+F 2 "" H 2850 4600 60  0001 C CNN
+F 3 "" H 2850 4600 60  0001 C CNN
 	1    2850 4600
 	1    0    0    -1
@@
 F 0 "R215" V 7730 6250 50  0000 C CNN
 F 1 "10R" V 7650 6250 50  0000 C CNN
+F 2 "" H 7650 6250 60  0001 C CNN
+F 3 "" H 7650 6250 60  0001 C CNN
 	1    7650 6250
 	0    -1   -1   0
@@
 F 0 "R220" V 9080 4850 50  0000 C CNN
 F 1 "1k8" V 9000 4850 50  0000 C CNN
+F 2 "" H 9000 4850 60  0001 C CNN
+F 3 "" H 9000 4850 60  0001 C CNN
 	1    9000 4850
 	1    0    0    -1
@@
 F 0 "D202" H 9000 5500 50  0000 C CNN
 F 1 "LED RED" H 9000 5300 50  0000 C CNN
+F 2 "" H 9000 5400 60  0001 C CNN
+F 3 "" H 9000 5400 60  0001 C CNN
 	1    9000 5400
 	0    1    1    0
@@
 F 0 "D201" H 2700 1900 50  0000 C CNN
 F 1 "LED RED" H 2700 1700 50  0000 C CNN
+F 2 "" H 2700 1800 60  0001 C CNN
+F 3 "" H 2700 1800 60  0001 C CNN
 	1    2700 1800
 	0    1    1    0
@@
 F 0 "R219" V 2780 1250 50  0000 C CNN
 F 1 "1k8" V 2700 1250 50  0000 C CNN
+F 2 "" H 2700 1250 60  0001 C CNN
+F 3 "" H 2700 1250 60  0001 C CNN
 	1    2700 1250
 	1    0    0    -1

Commit message: RAMPS-FD latest updates
Parts:
- added R701, R702: 10R, symbol R
Connections:
- net /D8_BUF: now also R701.1; no longer Q501.G
- net /D9_BUF: now also R702.1; no longer Q502.G
- new net: Q502.G, R702.2
- new net: Q501.G, R701.2
Other:
- note added: "Or similar"
Changed lines of the file:
@@
 Sheet 7 9
 Title ""
-Date "22 sep 2013"
+Date "23 sep 2013"
 Rev "0.2"
 Comp ""
@@
 Wire Wire Line
 	3650 850  4100 850
-Wire Wire Line
-	1000 2750 1850 2750
 Connection ~ 2150 2500
 Wire Wire Line
@@
 Wire Wire Line
 	2150 2550 2150 2000
-Wire Wire Line
-	3000 2500 2150 2500
 Connection ~ 2200 4300
 Wire Wire Line
@@
 	2150 850  2150 1500
 Connection ~ 2150 850
-Wire Wire Line
-	1900 6050 1000 6050
 Wire Wire Line
 	3350 4600 3350 4150
@@
 V_GATE
 $Comp
-L GND #PWR087
+L GND #PWR088
 U 1 1 51B37840
 P 2150 3100
-F 0 "#PWR087" H 2150 3100 30  0001 C CNN
+F 0 "#PWR088" H 2150 3100 30  0001 C CNN
 F 1 "GND" H 2150 3030 30  0001 C CNN
 F 2 "" H 2150 3100 60  0001 C CNN
@@
 $EndComp
 $Comp
-L GND #PWR088
+L GND #PWR089
 U 1 1 51B377DD
 P 2200 6400
-F 0 "#PWR088" H 2200 6400 30  0001 C CNN
+F 0 "#PWR089" H 2200 6400 30  0001 C CNN
 F 1 "GND" H 2200 6330 30  0001 C CNN
 F 2 "" H 2200 6400 60  0001 C CNN
@@
 D8 - Heatbed
 $Comp
-L GNDPWR #PWR089
+L GNDPWR #PWR090
 U 1 1 51AA07E6
 P 9300 3000
-F 0 "#PWR089" H 9300 3050 40  0001 C CNN
+F 0 "#PWR090" H 9300 3050 40  0001 C CNN
 F 1 "GNDPWR" H 9300 2920 40  0000 C CNN
 F 2 "" H 9300 3000 60  0001 C CNN
@@
 $EndComp
 $Comp
-L GND #PWR090
+L GND #PWR091
 U 1 1 51AA071A
 P 8400 6600
-F 0 "#PWR090" H 8400 6600 30  0001 C CNN
+F 0 "#PWR091" H 8400 6600 30  0001 C CNN
 F 1 "GND" H 8400 6530 30  0001 C CNN
 F 2 "" H 8400 6600 60  0001 C CNN
@@
 $EndComp
 $Comp
-L GNDPWR #PWR091
+L GNDPWR #PWR092
 U 1 1 51AA0719
 P 9450 6600
-F 0 "#PWR091" H 9450 6650 40  0001 C CNN
+F 0 "#PWR092" H 9450 6650 40  0001 C CNN
 F 1 "GNDPWR" H 9450 6520 40  0000 C CNN
 F 2 "" H 9450 6600 60  0001 C CNN
@@
 HB_GND
 $Comp
-L GNDPWR #PWR092
+L GNDPWR #PWR093
 U 1 1 51AA06B9
 P 3350 6550
-F 0 "#PWR092" H 3350 6600 40  0001 C CNN
+F 0 "#PWR093" H 3350 6600 40  0001 C CNN
 F 1 "GNDPWR" H 3350 6470 40  0000 C CNN
 F 2 "" H 3350 6550 60  0001 C CNN
@@
 $EndComp
 $Comp
-L GND #PWR093
+L GND #PWR094
 U 1 1 51770EF7
 P 8250 3000
-F 0 "#PWR093" H 8250 3000 30  0001 C CNN
+F 0 "#PWR094" H 8250 3000 30  0001 C CNN
 F 1 "GND" H 8250 2930 30  0001 C CNN
 F 2 "" H 8250 3000 60  0001 C CNN
@@
 $EndComp
 $Comp
-L +V_POWER #PWR094
+L +V_POWER #PWR095
 U 1 1 51770EF2
 P 9600 650
-F 0 "#PWR094" H 9600 620 30  0001 C CNN
+F 0 "#PWR095" H 9600 620 30  0001 C CNN
 F 1 "+V_POWER" H 9600 750 30  0000 C CNN
 F 2 "" H 9600 650 60  0001 C CNN
@@
 D8_OUT
 $Comp
-L +V_POWER #PWR095
+L +V_POWER #PWR096
 U 1 1 5176EF23
 P 3350 4150
-F 0 "#PWR095" H 3350 4120 30  0001 C CNN
+F 0 "#PWR096" H 3350 4120 30  0001 C CNN
 F 1 "+V_POWER" H 3350 4250 30  0000 C CNN
 F 2 "" H 3350 4150 60  0001 C CNN
@@
 $EndComp
 $Comp
-L +V_POWER #PWR096
+L +V_POWER #PWR097
 U 1 1 5176EE9D
 P 9450 4300
-F 0 "#PWR096" H 9450 4270 30  0001 C CNN
+F 0 "#PWR097" H 9450 4270 30  0001 C CNN
 F 1 "+V_POWER" H 9450 4400 30  0000 C CNN
 F 2 "" H 9450 4300 60  0001 C CNN
@@
 $EndComp
 $Comp
-L +V_HEATBED #PWR097
+L +V_HEATBED #PWR098
 U 1 1 5176EDD7
 P 3650 700
-F 0 "#PWR097" H 3650 670 30  0001 C CNN
+F 0 "#PWR098" H 3650 670 30  0001 C CNN
 F 1 "+V_HEATBED" H 3650 800 30  0000 C CNN
 F 2 "" H 3650 700 60  0001 C CNN
@@
 Text GLabel 1000 2750 0    60   Input ~ 0
 /D8_BUF
+Text Notes 3900 1350 3    50   ~ 0
+Or similar
+$Comp
+L R R701
+U 1 1 52409A4A
+P 1450 2750
+F 0 "R701" V 1530 2750 50  0000 C CNN
+F 1 "10R" V 1450 2750 50  0000 C CNN
+F 2 "" H 1450 2750 60  0001 C CNN
+F 3 "" H 1450 2750 60  0001 C CNN
+	1    1450 2750
+	0    -1   -1   0
+$EndComp
+Wire Wire Line
+	3000 2500 2150 2500
+$Comp
+L R R702
+U 1 1 52409A65
+P 1450 6050
+F 0 "R702" V 1530 6050 50  0000 C CNN
+F 1 "10R" V 1450 6050 50  0000 C CNN
+F 2 "" H 1450 6050 60  0001 C CNN
+F 3 "" H 1450 6050 60  0001 C CNN
+	1    1450 6050
+	0    -1   -1   0
+$EndComp
+Wire Wire Line
+	1700 6050 1900 6050
+Wire Wire Line
+	1200 6050 1000 6050
+Wire Wire Line
+	1850 2750 1700 2750
+Wire Wire Line
+	1200 2750 1000 2750
 $EndSCHEMATC

Commit message: RAMPS-FD: latest update
Parts:
- removed R215, R217, R701, R702: 10R, symbol R
Connections:
- net /D10_BUF: now also Q204.G
- net /D8_BUF: now also Q501.G
- net /D9_BUF: now also Q502.G
- net /FET4_BUF: now also Q205.G
Changed lines of the file:
@@
 Sheet 7 9
 Title ""
-Date "23 sep 2013"
+Date "24 sep 2013"
 Rev "0.2"
 Comp ""
@@
 	2150 3100 2150 2950
 Wire Wire Line
-	2150 2550 2150 2000
+	2150 2000 2150 2550
 Connection ~ 2200 4300
 Wire Wire Line
@@
 	9800 5450 10250 5450
 Wire Wire Line
-	9450 5700 9450 5300
+	9450 5300 9450 5700
 Wire Wire Line
 	1550 4300 2850 4300
 Wire Wire Line
-	4350 5350 2850 5350
-Wire Wire Line
-	2700 1000 2700 850
+	2850 5350 4350 5350
+Wire Wire Line
+	2700 850  2700 1000
 Wire Wire Line
 	2850 5350 2850 5300
@@
 Wire Wire Line
 	9600 1600 9600 1950
-Connection ~ 7150 2550
-Connection ~ 7300 6250
 Wire Wire Line
 	4500 1850 4100 1850
@@
 	8400 5500 8400 6050
 Wire Wire Line
-	8100 6250 7900 6250
+	7000 6250 8100 6250
 Wire Wire Line
 	9000 5200 9000 5100
-Wire Wire Line
-	7000 6250 7400 6250
 Wire Wire Line
 	2700 1600 2700 1500
@@
 	8250 1200 8250 850
 Wire Wire Line
-	7050 2550 7250 2550
+	7050 2550 7950 2550
 Wire Wire Line
 	8900 1500 8900 1400
 Wire Wire Line
-	7950 2550 7750 2550
-Wire Wire Line
-	8250 2350 8250 1700
+	8250 1700 8250 2350
 Wire Wire Line
 	9000 2300 8250 2300
 Connection ~ 8250 2300
 Wire Wire Line
-	8900 900  8900 850
+	8900 850  8900 900
 Wire Wire Line
 	10350 1750 10000 1750
@@
 	10000 1750 10000 850
 Wire Wire Line
-	9600 1200 9600 650
+	9600 650  9600 1200
 Connection ~ 3650 850
 Wire Wire Line
@@
 	2850 4300 2850 4350
 Wire Wire Line
-	4500 2050 2700 2050
+	2700 2050 4500 2050
 Wire Wire Line
 	2700 2050 2700 2000
 Wire Wire Line
-	2700 850  1500 850
-Wire Wire Line
-	3650 1300 3650 700
+	1500 850  2700 850
+Wire Wire Line
+	3650 700  3650 1300
 Wire Wire Line
 	4350 5150 3750 5150
@@
 	9000 4550 9000 4600
 Wire Wire Line
-	10250 5650 9000 5650
+	9000 5650 10250 5650
 Wire Wire Line
 	9000 5650 9000 5600
 Wire Wire Line
-	10350 1950 8900 1950
+	8900 1950 10350 1950
 Wire Wire Line
 	8900 1950 8900 1900
 Wire Wire Line
-	8900 850  7800 850
+	7800 850  8900 850
 Connection ~ 8250 850
 Wire Wire Line
@@
 	3050 5800 2200 5800
 Wire Wire Line
-	2200 5850 2200 5300
+	2200 5300 2200 5850
 Wire Wire Line
 	2200 6400 2200 6250
@@
 Connection ~ 2150 850
 Wire Wire Line
-	3350 4600 3350 4150
+	3350 4150 3350 4600
 Text GLabel 1550 4300 0    40   Input ~ 0
 V_GATE
@@
 	1    0    0    -1
 $EndComp
-$Comp
-L R R217
-U 1 1 51770EF6
-P 7500 2550
-F 0 "R217" V 7580 2550 50  0000 C CNN
-F 1 "10R" V 7500 2550 50  0000 C CNN
-F 2 "" H 7500 2550 60  0001 C CNN
-F 3 "" H 7500 2550 60  0001 C CNN
-	1    7500 2550
-	0    -1   -1   0
-$EndComp
 Text GLabel 7050 2550 0    60   Input ~ 0
 /FET4_BUF
@@
 /D9_BUF
 $Comp
-L R R215
-U 1 1 510479B2
-P 7650 6250
-F 0 "R215" V 7730 6250 50  0000 C CNN
-F 1 "10R" V 7650 6250 50  0000 C CNN
-F 2 "" H 7650 6250 60  0001 C CNN
-F 3 "" H 7650 6250 60  0001 C CNN
-	1    7650 6250
-	0    -1   -1   0
-$EndComp
-$Comp
 L R R220
 U 1 1 510479AF
@@
 Text Notes 3900 1350 3    50   ~ 0
 Or similar
-$Comp
-L R R701
-U 1 1 52409A4A
-P 1450 2750
-F 0 "R701" V 1530 2750 50  0000 C CNN
-F 1 "10R" V 1450 2750 50  0000 C CNN
-F 2 "" H 1450 2750 60  0001 C CNN
-F 3 "" H 1450 2750 60  0001 C CNN
-	1    1450 2750
-	0    -1   -1   0
-$EndComp
 Wire Wire Line
 	3000 2500 2150 2500
-$Comp
-L R R702
-U 1 1 52409A65
-P 1450 6050
-F 0 "R702" V 1530 6050 50  0000 C CNN
-F 1 "10R" V 1450 6050 50  0000 C CNN
-F 2 "" H 1450 6050 60  0001 C CNN
-F 3 "" H 1450 6050 60  0001 C CNN
-	1    1450 6050
-	0    -1   -1   0
-$EndComp
-Wire Wire Line
-	1700 6050 1900 6050
-Wire Wire Line
-	1200 6050 1000 6050
-Wire Wire Line
-	1850 2750 1700 2750
-Wire Wire Line
-	1200 2750 1000 2750
+Wire Wire Line
+	1000 6050 1900 6050
+Wire Wire Line
+	1000 2750 1850 2750
 $EndSCHEMATC
