File: RAMPS-FD/steppers.sch (KiCad schematic (older format))
At the start: 31 parts, among them P201 CONN_3X2, P202 CONN_3X2, P203 CONN_3X2, P204 X-MOT, P205 Y-MOT, P206 Z-MOT, P207 CONN_3X2, P208 CONN_3X2, P209 E0-MOT, P210 E1-MOT, P401 Z-MOT1, U201 X, U202 Y, U203 Z, U204 E0, U205 E1

Commit message: First version of RAMPS-FD, RIB
Parts:
- removed C204, C205: 100u, symbol CP1
- removed P207, P208: CONN_3X2, symbol CONN_3X2
- removed P209: E0-MOT, symbol CONN_4
- removed P210: E1-MOT, symbol CONN_4
- removed P401: Z-MOT1, symbol CONN_4
- removed R207, R208: 100k, symbol R
- removed R209, R210: 10k, symbol R
- removed U204: E0, symbol POLOLU
- removed U205: E1, symbol POLOLU
- added D301: DIODE, symbol DIODE
- added P302: ESTOP, symbol CONN_2
- added R304: 100k, symbol R
- added R305: 4k7, symbol R
- added U302, U303: 74LS08, symbol 74LS08
Connections:
- net labels added: +V_LOGIC, +V_MOTOR, /ESTOP, D8, D8_BUF, D9, D9_BUF, E0_EN_BUF, E1_EN_BUF, E2_EN, E2_EN_BUF, MOT_GND, X-1A, X-1B, X-2A, X-2B, X_EN_BUF, Y-1A, Y-1B, Y-2A, Y-2B, Y_EN_BUF, Z-1A, Z-1B, Z-2A, Z-2B, Z_EN_BUF
- net labels removed: +12V, +3.3V, E0_DIR, E0_STEP, E1_DIR, E1_STEP
- wire segments 160 -> 129
Other:
- moved on the sheet: C201, C202, C203, P201, P202, P203, P204, P205, P206, R201, R202, R203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

Commit message: RAMPS-FD update
Parts:
- removed D301: DIODE, symbol DIODE
- removed P302: ESTOP, symbol CONN_2
- removed R204, R205, R206: 10k, symbol R
- removed R304: 100k, symbol R
- removed R305: 4k7, symbol R
- removed U302, U303: 74LS08, symbol 74LS08
- C201, C202, C203: value 100u -> 100u 25V
Connections:
- net labels added: /X_EN_BUF, /Y_EN_BUF, /Z_EN_BUF
- net labels removed: /ESTOP, D8, D8_BUF, D9, D9_BUF, E0_EN, E0_EN_BUF, E1_EN, E1_EN_BUF, E2_EN, E2_EN_BUF, X_EN, X_EN_BUF, Y_EN, Y_EN_BUF, Z_EN, Z_EN_BUF
- wire segments 129 -> 93
Other:
- moved on the sheet: C202, C203, P201, P202, P205, P206, R201, R203, U202, U203

Commit message: Updates to RAMPS-FD
Parts:
- C201, C202, C203: value 100u 25V -> 100u 35V
Connections:
- net +V_LOGIC: now also P201.1, P201.3, P201.5, P202.1, P202.3, P202.5, P203.1, P203.3, P203.5; no longer P201.2, P201.4, P201.6, P202.2, P202.4, P202.6, P203.2, P203.4, P203.6
- net at R202.1, U201.2 (MS1): now also P203.2; no longer P203.1
- net at U201.3 (MS2): now also P203.4; no longer P203.3
- net at U201.4 (MS3): now also P203.6; no longer P203.5
- net at R203.1, U202.2 (MS1): now also P201.2; no longer P201.1
- net at U202.3 (MS2): now also P201.4; no longer P201.3
- net at U202.4 (MS3): now also P201.6; no longer P201.5
- net at R201.1, U203.2 (MS1): now also P202.2; no longer P202.1
- net at U203.3 (MS2): now also P202.4; no longer P202.3
- net at U203.4 (MS3): now also P202.6; no longer P202.5
Changed lines of the file:
@@
-EESchema Schematic File Version 2  date 19/09/2013 22:01:21
+EESchema Schematic File Version 2
 LIBS:power
 LIBS:device
@@
 LIBS:opendous
 LIBS:RAMPS-FD-cache
-EELAYER 25  0
+EELAYER 27 0
 EELAYER END
-$Descr A4 11700 8267
+$Descr A4 11693 8268
 encoding utf-8
-Sheet 3 8
+Sheet 3 9
 Title "RAMPS-FS RAMPS for Due"
-Date "19 sep 2013"
+Date "22 sep 2013"
 Rev "0.2"
 Comp ""
@@
 F 0 "#PWR034" H 3850 6970 30  0001 C CNN
 F 1 "+V_LOGIC" H 3850 7100 30  0000 C CNN
+F 2 "" H 3850 7000 60  0001 C CNN
+F 3 "" H 3850 7000 60  0001 C CNN
 	1    3850 7000
 	1    0    0    -1
@@
 F 0 "#PWR035" H 3850 4620 30  0001 C CNN
 F 1 "+V_LOGIC" H 3850 4750 30  0000 C CNN
+F 2 "" H 3850 4650 60  0001 C CNN
+F 3 "" H 3850 4650 60  0001 C CNN
 	1    3850 4650
 	1    0    0    -1
@@
 F 0 "#PWR036" H 3750 2270 30  0001 C CNN
 F 1 "+V_LOGIC" H 3750 2400 30  0000 C CNN
+F 2 "" H 3750 2300 60  0001 C CNN
+F 3 "" H 3750 2300 60  0001 C CNN
 	1    3750 2300
 	1    0    0    -1
@@
 F 0 "#PWR037" H 3800 5420 30  0001 C CNN
 F 1 "+V_LOGIC" H 3800 5550 30  0000 C CNN
+F 2 "" H 3800 5450 60  0001 C CNN
+F 3 "" H 3800 5450 60  0001 C CNN
 	1    3800 5450
 	1    0    0    -1
@@
 F 0 "#PWR038" H 3800 3070 30  0001 C CNN
 F 1 "+V_LOGIC" H 3800 3200 30  0000 C CNN
+F 2 "" H 3800 3100 60  0001 C CNN
+F 3 "" H 3800 3100 60  0001 C CNN
 	1    3800 3100
 	1    0    0    -1
@@
 F 0 "#PWR039" H 3700 720 30  0001 C CNN
 F 1 "+V_LOGIC" H 3700 850 30  0000 C CNN
+F 2 "" H 3700 750 60  0001 C CNN
+F 3 "" H 3700 750 60  0001 C CNN
 	1    3700 750
 	1    0    0    -1
@@
 F 0 "#PWR040" H 5700 5870 30  0001 C CNN
 F 1 "+V_MOTOR" H 5700 6000 30  0000 C CNN
+F 2 "" H 5700 5900 60  0001 C CNN
+F 3 "" H 5700 5900 60  0001 C CNN
 	1    5700 5900
 	1    0    0    -1
@@
 F 0 "#PWR041" H 5700 3520 30  0001 C CNN
 F 1 "+V_MOTOR" H 5700 3650 30  0000 C CNN
+F 2 "" H 5700 3550 60  0001 C CNN
+F 3 "" H 5700 3550 60  0001 C CNN
 	1    5700 3550
 	1    0    0    -1
@@
 F 0 "#PWR042" H 5600 1170 30  0001 C CNN
 F 1 "+V_MOTOR" H 5600 1300 30  0000 C CNN
+F 2 "" H 5600 1200 60  0001 C CNN
+F 3 "" H 5600 1200 60  0001 C CNN
 	1    5600 1200
 	1    0    0    -1
@@
 F 0 "R201" V 3730 7250 50  0000 C CNN
 F 1 "100k" V 3650 7250 50  0000 C CNN
+F 2 "" H 3650 7250 60  0001 C CNN
+F 3 "" H 3650 7250 60  0001 C CNN
 	1    3650 7250
 	1    0    0    -1
@@
 F 0 "R203" V 3780 4900 50  0000 C CNN
 F 1 "100k" V 3700 4900 50  0000 C CNN
+F 2 "" H 3700 4900 60  0001 C CNN
+F 3 "" H 3700 4900 60  0001 C CNN
 	1    3700 4900
 	1    0    0    -1
@@
 F 0 "#PWR043" H 5750 5250 30  0001 C CNN
 F 1 "GND" H 5750 5180 30  0001 C CNN
+F 2 "" H 5750 5250 60  0001 C CNN
+F 3 "" H 5750 5250 60  0001 C CNN
 	1    5750 5250
 	1    0    0    -1
@@
 F 0 "#PWR044" H 5650 2800 30  0001 C CNN
 F 1 "GND" H 5650 2730 30  0001 C CNN
+F 2 "" H 5650 2800 60  0001 C CNN
+F 3 "" H 5650 2800 60  0001 C CNN
 	1    5650 2800
 	1    0    0    -1
@@
 F 0 "R202" V 3680 2450 50  0000 C CNN
 F 1 "100k" V 3600 2450 50  0000 C CNN
+F 2 "" H 3600 2450 60  0001 C CNN
+F 3 "" H 3600 2450 60  0001 C CNN
 	1    3600 2450
 	1    0    0    -1
@@
 P 6250 6550
 F 0 "C203" H 6300 6650 50  0000 L CNN
-F 1 "100u 25V" H 6300 6450 50  0000 L CNN
+F 1 "100u 35V" H 6300 6450 50  0000 L CNN
+F 2 "" H 6250 6550 60  0001 C CNN
+F 3 "" H 6250 6550 60  0001 C CNN
 	1    6250 6550
 	1    0    0    -1
@@
 P 6350 4200
 F 0 "C202" H 6400 4300 50  0000 L CNN
-F 1 "100u 25V" H 6400 4100 50  0000 L CNN
+F 1 "100u 35V" H 6400 4100 50  0000 L CNN
+F 2 "" H 6350 4200 60  0001 C CNN
+F 3 "" H 6350 4200 60  0001 C CNN
 	1    6350 4200
 	1    0    0    -1
@@
 P 6250 1850
 F 0 "C201" H 6300 1950 50  0000 L CNN
-F 1 "100u 25V" H 6300 1750 50  0000 L CNN
+F 1 "100u 35V" H 6300 1750 50  0000 L CNN
+F 2 "" H 6250 1850 60  0001 C CNN
+F 3 "" H 6250 1850 60  0001 C CNN
 	1    6250 1850
 	1    0    0    -1
@@
 F 0 "P202" H 3100 7000 50  0000 C CNN
 F 1 "CONN_3X2" V 3100 6800 40  0000 C CNN
+F 2 "" H 3100 6750 60  0001 C CNN
+F 3 "" H 3100 6750 60  0001 C CNN
 	1    3100 6750
-	-1   0    0    -1
+	1    0    0    -1
 $EndComp
 $Comp
@@
 F 0 "P206" V 5950 6550 50  0000 C CNN
 F 1 "Z-MOT" V 6050 6550 50  0000 C CNN
+F 2 "" H 6000 6550 60  0001 C CNN
+F 3 "" H 6000 6550 60  0001 C CNN
 	1    6000 6550
 	1    0    0    -1
@@
 F 0 "#PWR045" H 5750 7700 30  0001 C CNN
 F 1 "GND" H 5750 7630 30  0001 C CNN
+F 2 "" H 5750 7700 60  0001 C CNN
+F 3 "" H 5750 7700 60  0001 C CNN
 	1    5750 7700
 	1    0    0    -1
@@
 F 0 "P201" H 3100 4650 50  0000 C CNN
 F 1 "CONN_3X2" V 3100 4450 40  0000 C CNN
+F 2 "" H 3100 4400 60  0001 C CNN
+F 3 "" H 3100 4400 60  0001 C CNN
 	1    3100 4400
-	-1   0    0    -1
+	1    0    0    -1
 $EndComp
 Text GLabel 4100 4050 0    50   Input ~ 0
@@
 F 0 "P205" V 6050 4200 50  0000 C CNN
 F 1 "Y-MOT" V 6150 4200 50  0000 C CNN
+F 2 "" H 6100 4200 60  0001 C CNN
+F 3 "" H 6100 4200 60  0001 C CNN
 	1    6100 4200
 	1    0    0    -1
@@
 F 0 "P204" V 5950 1850 50  0000 C CNN
 F 1 "X-MOT" V 6050 1850 50  0000 C CNN
+F 2 "" H 6000 1850 60  0001 C CNN
+F 3 "" H 6000 1850 60  0001 C CNN
 	1    6000 1850
 	1    0    0    -1
@@
 F 0 "P203" H 3100 2300 50  0000 C CNN
 F 1 "CONN_3X2" V 3100 2100 40  0000 C CNN
+F 2 "" H 3100 2050 60  0001 C CNN
+F 3 "" H 3100 2050 60  0001 C CNN
 	1    3100 2050
-	-1   0    0    -1
+	1    0    0    -1
 $EndComp
 $Comp
@@
 F 0 "U203" H 4500 7200 60  0000 C CNN
 F 1 "Z" H 4600 5950 60  0000 C CNN
+F 2 "" H 4800 6600 60  0001 C CNN
+F 3 "" H 4800 6600 60  0001 C CNN
 	1    4800 6600
 	1    0    0    -1
@@
 F 0 "U202" H 4500 4850 60  0000 C CNN
 F 1 "Y" H 4600 3600 60  0000 C CNN
+F 2 "" H 4800 4250 60  0001 C CNN
+F 3 "" H 4800 4250 60  0001 C CNN
 	1    4800 4250
 	1    0    0    -1
@@
 F 0 "U201" H 4400 2500 60  0000 C CNN
 F 1 "X" H 4500 1250 60  0000 C CNN
+F 2 "" H 4700 1900 60  0001 C CNN
+F 3 "" H 4700 1900 60  0001 C CNN
 	1    4700 1900
 	1    0    0    -1
