File: RAMPS-FD/con_misc.sch (KiCad schematic (older format))
At the start: 11 parts, among them K201 SER1, K202 SER2, K203 SER3, K204 SER4, P211 I2C, P213 AUX-4, P214 AUX-2, P215 AUX-3, P216 SERIAL

Commit message: RAMPS-FD update
Parts:
- removed P215: AUX-3, symbol CONN_4X2
- removed P216: SERIAL, symbol CONN_4
- added P1: SERIAL2, symbol CONN_6
- added P2: I2C-1, symbol CONN_4
- added P215: AUX-2, symbol CONN_5X2
- added P216: SERIAL1, symbol CONN_6
- added R1, R2: NF, symbol R
- P211: value I2C -> I2C-0
Connections:
- net +V_LOGIC: now also P2.1 (P1), P215.1, R1.1, R2.1
- net D49: now also P213.5 (P5)
- net D51: now also P215.7; no longer P213.4 (P4)
- net D53: now also P215.9
- net GND: now also P1.1, P2.2 (P2), P215.2, P216.1
- net MISO: now also P215.3
- net MOSI: now also P215.4
- net SCK: now also P215.5
- net AD15: now reaches P213.3 (P3)
- new net AD14: P213.4 (P4)
- new net AUX_UART_RX_LV: P1.4
- new net AUX_UART_TX_LV: P1.5
- new net D42: P215.10
- new net D50: P215.6
- new net D52: P215.8
- new net SCL1: P2.4 (P4), R1.2
- new net SDA1: P2.3 (P3), R2.2
- new net UART_RX_LV: P216.4
- new net UART_TX_LV: P216.5
- no-connect marks 7 -> 10
Other:
- note added: "Serial"
- moved on the sheet: K201, K202, K203, K204, P211, P213, P214, R211, R212

Commit message: Updates to RAMPS-FD
Parts:
- P1: value SERIAL2 -> SERIAL1
- P215: value AUX-2 -> AUX-3
- P216: value SERIAL1 -> SERIAL0
Connections:
- net D51 is gone; now on net A6: P215.7
- net D52 is gone; now on net A7: P215.8
- net A4: now also P214.7; no longer P214.3
- net A5: now also P214.8; no longer P214.5
- net A6: no longer P214.7
- net A7: no longer P214.9
- net UART2_RX_LV: now reaches P214.10
- net D51-MOSI: now reaches P214.4
- net D53-SS: now reaches P214.6
- net AUX_UART_RX_LV renamed UART1_RX_LV
- net AUX_UART_TX_LV renamed UART1_TX_LV
- net D42 renamed UART3_RX_LV
- net D50 renamed SPI_CS1
- net D53 renamed UART3_TX_LV
- net UART_RX_LV renamed UART0_RX_LV
- net UART_TX_LV renamed UART0_TX_LV
- new net D50-MISO: P214.3
- new net D52-SCK: P214.5
- new net UART2_TX_LV: P214.9
- no-connect marks 10 -> 6
Other:
- note added: "Aux2"
- note added: "Aux3"
- note added: "NB: On Arduino Due: IOs on this page are not 5V tolerant. Do not exceed 3.3V."
- note added: "Note: this serial port is shared with\nUSB programming port"
- note added: "These are shared with E1 \nand E2 stepper signals"
- note removed: "Aux2 - spare ADC inputs"
- note removed: "Aux3-SPI"
- note removed: "Should these be 5V?"
- note removed: "TTL 3V3 or 5V\ncompatible"
- moved on the sheet: P1, P2, P211, P214, P215, P216, R1, R2, R211, R212

Commit message: RAMPS-FD latest updates
Connections:
- net A4: now also P214.3; no longer P214.7
- net A5: now also P214.4; no longer P214.8
- net A6: now also P214.5; no longer P215.7
- net A7: now also P214.6; no longer P215.8
- net AD14: now also P214.7; no longer P213.4 (P4)
- net AD15: now also P214.8; no longer P213.3 (P3)
- net D49: now also P215.7; no longer P213.5 (P5)
- net D50-MISO: now also P213.5 (P5); no longer P214.3
- net D51-MOSI: now also P213.4 (P4); no longer P214.4
- net D52-SCK: now also P213.3 (P3); no longer P214.5
- net D53-SS: now also P215.6; no longer P214.6
- net SPI_CS1: now also P215.8; no longer P215.6
Other:
- note added: "Mega only: same signals as \nMISO, MOSI & SCK on Aux3"
Changed lines of the file:
@@
 Sheet 6 9
 Title ""
-Date "22 sep 2013"
+Date "23 sep 2013"
 Rev "0.2"
 Comp ""
@@
 Comment4 ""
 $EndDescr
-Text GLabel 8250 6350 0    50   Input ~ 0
+Text GLabel 9600 2600 2    50   Input ~ 0
 AD15
-Text GLabel 8250 6250 0    50   Input ~ 0
+Text GLabel 8300 2600 0    50   Input ~ 0
 AD14
 Wire Wire Line
@@
 	8650 6250 8250 6250
 Wire Wire Line
-	8650 6550 7850 6550
-Wire Wire Line
-	7850 6550 7850 6450
+	8650 6550 7500 6550
+Wire Wire Line
+	7500 6550 7500 6450
 Wire Wire Line
 	9950 3750 9400 3750
@@
 	4950 4450 4950 4600
 Connection ~ 4950 4600
-Text GLabel 8300 2400 0    50   BiDi ~ 0
+Text GLabel 8250 6150 0    50   BiDi ~ 0
 D50-MISO
-Text GLabel 8300 2500 0    50   BiDi ~ 0
+Text GLabel 8250 6350 0    50   BiDi ~ 0
 D52-SCK
 $Comp
@@
 $EndComp
 $Comp
-L GND #PWR067
+L GND #PWR068
 U 1 1 523B601D
 P 5400 4800
-F 0 "#PWR067" H 5400 4800 30  0001 C CNN
+F 0 "#PWR068" H 5400 4800 30  0001 C CNN
 F 1 "GND" H 5400 4730 30  0001 C CNN
 F 2 "" H 5400 4800 60  0001 C CNN
@@
 SCL1
 $Comp
-L +V_LOGIC #PWR068
+L +V_LOGIC #PWR069
 U 1 1 523B601C
 P 4600 3800
-F 0 "#PWR068" H 4600 3770 30  0001 C CNN
+F 0 "#PWR069" H 4600 3770 30  0001 C CNN
 F 1 "+V_LOGIC" H 4600 3900 30  0000 C CNN
 F 2 "" H 4600 3800 60  0001 C CNN
@@
 UART1_TX_LV
 $Comp
-L GND #PWR069
+L GND #PWR070
 U 1 1 523B5AB9
 P 1950 3600
-F 0 "#PWR069" H 1950 3600 30  0001 C CNN
+F 0 "#PWR070" H 1950 3600 30  0001 C CNN
 F 1 "GND" H 1950 3530 30  0001 C CNN
 F 2 "" H 1950 3600 60  0001 C CNN
@@
 Text Notes 550  1950 0    50   ~ 0
 UART-TTL
-Text GLabel 8400 4050 0    50   Input ~ 0
+Text GLabel 8300 2500 0    50   Input ~ 0
 A6
-Text GLabel 9550 4050 2    50   Input ~ 0
+Text GLabel 9600 2500 2    50   Input ~ 0
 A7
-Text GLabel 9600 2600 2    50   Input ~ 0
+Text GLabel 9600 2400 2    50   Input ~ 0
 A5
-Text GLabel 8300 2600 0    50   Input ~ 0
+Text GLabel 8300 2400 0    50   Input ~ 0
 A4
-Text GLabel 9600 2400 2    50   BiDi ~ 0
+Text GLabel 8250 6250 0    50   BiDi ~ 0
 D51-MOSI
 $Comp
-L +V_LOGIC #PWR070
+L +V_LOGIC #PWR071
 U 1 1 517867DE
-P 7850 6450
-F 0 "#PWR070" H 7850 6420 30  0001 C CNN
-F 1 "+V_LOGIC" H 7850 6550 30  0000 C CNN
-F 2 "" H 7850 6450 60  0001 C CNN
-F 3 "" H 7850 6450 60  0001 C CNN
-	1    7850 6450
-	1    0    0    -1
-$EndComp
-$Comp
-L +V_LOGIC #PWR071
+P 7500 6450
+F 0 "#PWR071" H 7500 6420 30  0001 C CNN
+F 1 "+V_LOGIC" H 7500 6550 30  0000 C CNN
+F 2 "" H 7500 6450 60  0001 C CNN
+F 3 "" H 7500 6450 60  0001 C CNN
+	1    7500 6450
+	1    0    0    -1
+$EndComp
+$Comp
+L +V_LOGIC #PWR072
 U 1 1 517867DD
 P 8150 2200
-F 0 "#PWR071" H 8150 2170 30  0001 C CNN
+F 0 "#PWR072" H 8150 2170 30  0001 C CNN
 F 1 "+V_LOGIC" H 8150 2300 30  0000 C CNN
 F 2 "" H 8150 2200 60  0001 C CNN
@@
 $EndComp
 $Comp
-L +V_LOGIC #PWR072
+L +V_LOGIC #PWR073
 U 1 1 517867D0
 P 8100 3650
-F 0 "#PWR072" H 8100 3620 30  0001 C CNN
+F 0 "#PWR073" H 8100 3620 30  0001 C CNN
 F 1 "+V_LOGIC" H 8100 3750 30  0000 C CNN
 F 2 "" H 8100 3650 60  0001 C CNN
@@
 $EndComp
 $Comp
-L +V_LOGIC #PWR073
+L +V_LOGIC #PWR074
 U 1 1 517867C6
 P 4700 1600
-F 0 "#PWR073" H 4700 1570 30  0001 C CNN
+F 0 "#PWR074" H 4700 1570 30  0001 C CNN
 F 1 "+V_LOGIC" H 4700 1700 30  0000 C CNN
 F 2 "" H 4700 1600 60  0001 C CNN
@@
 $EndComp
 $Comp
-L GND #PWR074
+L GND #PWR075
 U 1 1 51084B2C
 P 8400 6500
-F 0 "#PWR074" H 8400 6500 30  0001 C CNN
+F 0 "#PWR075" H 8400 6500 30  0001 C CNN
 F 1 "GND" H 8400 6430 30  0001 C CNN
 F 2 "" H 8400 6500 60  0001 C CNN
@@
 	1    0    0    1
 $EndComp
-Text GLabel 9600 2500 2    50   BiDi ~ 0
+Text GLabel 9550 3950 2    50   BiDi ~ 0
 D53-SS
-Text GLabel 8250 6150 0    50   BiDi ~ 0
+Text GLabel 8400 4050 0    50   BiDi ~ 0
 D49
 Text GLabel 9550 3850 2    50   Input ~ 0
@@
 Must not have external pullups to 5V
 $Comp
-L GND #PWR075
+L GND #PWR076
 U 1 1 5104884C
 P 9950 3850
-F 0 "#PWR075" H 9950 3850 30  0001 C CNN
+F 0 "#PWR076" H 9950 3850 30  0001 C CNN
 F 1 "GND" H 9950 3780 30  0001 C CNN
 F 2 "" H 9950 3850 60  0001 C CNN
@@
 $EndComp
 $Comp
-L GND #PWR076
+L GND #PWR077
 U 1 1 51048839
 P 10200 2350
-F 0 "#PWR076" H 10200 2350 30  0001 C CNN
+F 0 "#PWR077" H 10200 2350 30  0001 C CNN
 F 1 "GND" H 10200 2280 30  0001 C CNN
 F 2 "" H 10200 2350 60  0001 C CNN
@@
 $EndComp
 $Comp
-L GND #PWR077
+L GND #PWR078
 U 1 1 5104861F
 P 1950 2350
-F 0 "#PWR077" H 1950 2350 30  0001 C CNN
+F 0 "#PWR078" H 1950 2350 30  0001 C CNN
 F 1 "GND" H 1950 2280 30  0001 C CNN
 F 2 "" H 1950 2350 60  0001 C CNN
@@
 $EndComp
 $Comp
-L GND #PWR078
+L GND #PWR079
 U 1 1 51047C7E
 P 1550 6850
-F 0 "#PWR078" H 1550 6850 30  0001 C CNN
+F 0 "#PWR079" H 1550 6850 30  0001 C CNN
 F 1 "GND" H 1550 6780 30  0001 C CNN
 F 2 "" H 1550 6850 60  0001 C CNN
@@
 $EndComp
 $Comp
-L +5V #PWR079
+L +5V #PWR080
 U 1 1 51047C7D
 P 1550 6450
-F 0 "#PWR079" H 1550 6540 20  0001 C CNN
+F 0 "#PWR080" H 1550 6540 20  0001 C CNN
 F 1 "+5V" H 1550 6540 30  0000 C CNN
 F 2 "" H 1550 6450 60  0001 C CNN
@@
 SERVO3
 $Comp
-L +5V #PWR080
+L +5V #PWR081
 U 1 1 51047C7B
 P 1550 5700
-F 0 "#PWR080" H 1550 5790 20  0001 C CNN
+F 0 "#PWR081" H 1550 5790 20  0001 C CNN
 F 1 "+5V" H 1550 5790 30  0000 C CNN
 F 2 "" H 1550 5700 60  0001 C CNN
@@
 $EndComp
 $Comp
-L GND #PWR081
+L GND #PWR082
 U 1 1 51047C7A
 P 1550 6100
-F 0 "#PWR081" H 1550 6100 30  0001 C CNN
+F 0 "#PWR082" H 1550 6100 30  0001 C CNN
 F 1 "GND" H 1550 6030 30  0001 C CNN
 F 2 "" H 1550 6100 60  0001 C CNN
@@
 $EndComp
 $Comp
-L GND #PWR082
+L GND #PWR083
 U 1 1 51047C77
 P 1550 5450
-F 0 "#PWR082" H 1550 5450 30  0001 C CNN
+F 0 "#PWR083" H 1550 5450 30  0001 C CNN
 F 1 "GND" H 1550 5380 30  0001 C CNN
 F 2 "" H 1550 5450 60  0001 C CNN
@@
 $EndComp
 $Comp
-L +5V #PWR083
+L +5V #PWR084
 U 1 1 51047C76
 P 1550 5050
-F 0 "#PWR083" H 1550 5140 20  0001 C CNN
+F 0 "#PWR084" H 1550 5140 20  0001 C CNN
 F 1 "+5V" H 1550 5140 30  0000 C CNN
 F 2 "" H 1550 5050 60  0001 C CNN
@@
 SERVO1
 $Comp
-L +5V #PWR084
+L +5V #PWR085
 U 1 1 51047C09
 P 1550 4300
-F 0 "#PWR084" H 1550 4390 20  0001 C CNN
+F 0 "#PWR085" H 1550 4390 20  0001 C CNN
 F 1 "+5V" H 1550 4390 30  0000 C CNN
 F 2 "" H 1550 4300 60  0001 C CNN
@@
 $EndComp
 $Comp
-L GND #PWR085
+L GND #PWR086
 U 1 1 51047C01
 P 1550 4700
-F 0 "#PWR085" H 1550 4700 30  0001 C CNN
+F 0 "#PWR086" H 1550 4700 30  0001 C CNN
 F 1 "GND" H 1550 4630 30  0001 C CNN
 F 2 "" H 1550 4700 60  0001 C CNN
@@
 SDA
 $Comp
-L GND #PWR086
+L GND #PWR087
 U 1 1 51047413
 P 5500 2600
-F 0 "#PWR086" H 5500 2600 30  0001 C CNN
+F 0 "#PWR087" H 5500 2600 30  0001 C CNN
 F 1 "GND" H 5500 2530 30  0001 C CNN
 F 2 "" H 5500 2600 60  0001 C CNN
@@
 Text Notes 550  1600 0    50   ~ 0
 Note: this serial port is shared with\nUSB programming port
-Text GLabel 9550 3950 2    50   Input ~ 0
+Text GLabel 9550 4050 2    50   Input ~ 0
 SPI_CS1
 Wire Wire Line
@@
 Text Notes 6800 5100 0    50   ~ 0
 These are shared with E1 \nand E2 stepper signals
+Wire Notes Line
+	7750 6150 7650 6150
+Wire Notes Line
+	7650 6150 7650 6350
+Wire Notes Line
+	7650 6350 7750 6350
+Wire Notes Line
+	7650 6200 7250 6200
+Text Notes 6100 6200 0    50   ~ 0
+Mega only: same signals as \nMISO, MOSI & SCK on Aux3
 $EndSCHEMATC

Commit message: RAMPS-FD: latest update
Connections:
- net D53-SS is gone; now on net SPI_CS1: P215.6
- net +5V: now also P215.1
- net +V_LOGIC: no longer P215.1
- net D23: now also P213.16 (P16); no longer P213.18 (P18)
- net D25: now also P213.15 (P15); no longer P213.17 (P17)
- net D27: now also P213.14 (P14); no longer P213.16 (P16)
- net D29: now also P213.13 (P13); no longer P213.15 (P15)
- net D31: now also P213.12 (P12); no longer P213.14 (P14)
- net D33: now also P213.11 (P11); no longer P213.13 (P13)
- net D35: now also P213.10 (P10); no longer P213.12 (P12)
- net D37: now also P213.9 (P9); no longer P213.11 (P11)
- net D39: now also P213.8 (P8); no longer P213.10 (P10)
- net D41: now also P213.7 (P7); no longer P213.9 (P9)
- net D43: now also P213.6 (P6); no longer P213.8 (P8)
- net D45: now also P213.5 (P5); no longer P213.7 (P7)
- net D47: now also P213.4 (P4); no longer P213.6 (P6)
- net D49: now also P215.2; no longer P215.7
- net D50-MISO: now also P215.8; no longer P213.5 (P5)
- net D51-MOSI: now also P215.9; no longer P213.4 (P4)
- net D52-SCK: now also P215.10; no longer P213.3 (P3)
- net GND: now also P215.7; no longer P215.2
- net SPI_CS1: no longer P215.8
- net UART2_RX_LV: now also P213.17 (P17); no longer P214.10
- net UART2_TX_LV: now also P213.18 (P18); no longer P214.9
- net UART3_RX_LV: now also P214.10; no longer P215.10
- net UART3_TX_LV: now also P214.9; no longer P215.9
- new net D32: P213.3 (P3)
Other:
- note added: "Aux3 - SPI"
- note added: "Mega: same signals as \nMISO, MOSI & SCK"
- note added: "NB This pin is always 5V"
- note added: "These are free \nfor LCD panel etc"
- note removed: "Aux3"
- note removed: "Mega only: same signals as \nMISO, MOSI & SCK on Aux3"
- moved on the sheet: P213
