File: Decapede/Power.sch (KiCad schematic (older format))
At the start: 25 parts, among them P1 power, Q1 BUK7226-75A,118, Q2 BUK964R8-60E,118, Q3 BC817-25,215, Q4 BC807,215, SW1 Reset, U1 L78M05CDT, U2 L78M12CDT-TR

Commit message: Updates for Decapede project.
Parts:
- removed D4: Diode 10TQ035, ~, symbol DIODESCH
- removed R203: 20 Ohm, ~, symbol R
- removed U1: L78M05CDT, D2PAK, symbol LM7812ACT
- added C18: 47uF, ~, symbol CP1
- added D15: Diode 1N4007, ~, symbol DIODE
- added D26: ES1D, ~, symbol DIODESCH
- added D27: 24V_OK, ~, symbol LED
- added D28: 12V_OK, ~, symbol LED
- added D29: 5V_OK, ~, symbol LED
- added D30: 24V_ERR, ~, symbol LED
- added D4: LED, ~, symbol LED
- added JP1: PWR_SEL, ~, symbol JUMPER
- added P43: Aux, symbol CONN_2
- added R112, R113, R118: 1k8, ~, symbol R
- added R114: 680, ~, symbol R
- added R115: 220, ~, symbol R
- added R116: 330 R, ~, symbol R
- added R117: 1k, ~, symbol R
- added U1: LM317MDT, TO-252, symbol LM317MDT
- D2: value Diode 10TQ035 -> BZV55-B15,115; symbol DIODESCH -> ZENER
- F1: value FUSE -> MAXI FUSE 60A
- P1: value power -> Power; symbol CONN_6 -> CONN_4
- U2: footprint D2PAK -> DPAK
- renumbered R204 to R201, R205 to R203, R202 to R204, R201 to R205
Connections:
- net labels added: +V_LOGIC, AGND, ARDUINO_VIN, AUX_RTN, Aux_output, GND_IN
- net labels removed: +5V, Fan_driver_signal
- wire segments 77 -> 101
Other:
- note added: "Auxiliary/fan output"
- note added: "Fit jumper to provide power to Arduino"
- note added: "For 3.3V (Due) fit 560 R to R117"
- note added: "Reverse polarity protection"
- note added: "Voltage regulators"
- note added: "use 1A part MC7812CDTG\nor\nD2PAK Use 1.5A part e.g. UA7812CKTTR"
- moved on the sheet: C11, C12, C14, C15, C16, C17, D1, D2, D3, F1, Q2, R205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

Commit message: Decapede update: add fuses for each main section; change endstops to use 0V instead of 5V; more space for stepper drivers to allow latching connectors
Parts:
- added F2: AUX/HEATBED, ~, symbol FUSE
- added F3: HEATERS, ~, symbol FUSE
- added F4: MOTORS, ~, symbol FUSE
- F1: value MAXI FUSE 60A -> MAIN 60A MAX
- P43: value Aux -> Aux Out
Connections:
- net labels added: +V_GATE, +V_HEATBED, +V_HEATERS, +V_MOTOR, 24V_IN
- net labels removed: +12V, +24V2
- wire segments 101 -> 113
Other:
- note added: "use 1A part MC7812CDTG"
- note removed: "use 1A part MC7812CDTG\nor\nD2PAK Use 1.5A part e.g. UA7812CKTTR"
- moved on the sheet: C11, C12, C14, C15, C16, C17, C18, D1, D15, D26, D27, D28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
