File: CRAMPS/steppers2.sch (KiCad schematic (older format))
At the start: 15 parts, among them P207 CONN_3X2, P208 CONN_3X2, P209 CONN_3X2, P210 E2-MOT, P212 E1-MOT, P217 E0-MOT, U204 E2, U205 E1, U206 E0

Commit message: Initial placement mostly complete
Signed-off-by: Charles Steinkuehler <charles@steinkuehler.net>
Connections:
- net +V_LOGIC: now also P207.2, P207.4, P207.6, P208.2, P208.4, P208.6, P209.2, P209.4, P209.6; no longer P207.1, P207.3, P207.5, P208.1, P208.3, P208.5, P209.1, P209.3, P209.5
- net at R207.1, U204.2 (MS1): now also P207.1; no longer P207.2
- net at U204.3 (MS2): now also P207.3; no longer P207.4
- net at U204.4 (MS3): now also P207.5; no longer P207.6
- net at R208.1, U205.2 (MS1): now also P209.1; no longer P209.2
- net at R210.1, U206.2 (MS1): now also P208.1; no longer P208.2
- net at U206.3 (MS2): now also P208.3; no longer P208.4
- net at U206.4 (MS3): now also P208.5; no longer P208.6
- net at U205.3 (MS2): now also P209.3; no longer P209.4
- net at U205.4 (MS3): now also P209.5; no longer P209.6
Changed lines of the file:
@@
 Sheet 5 10
 Title "CRAMPS (Cape-RAMPS for BeagleBone)"
-Date "6 feb 2014"
+Date "8 feb 2014"
 Rev "v1.0"
 Comp ""
@@
 F 3 "" H 3000 4400 60  0001 C CNN
 	1    3000 4400
-	1    0    0    -1
+	-1   0    0    -1
 $EndComp
 Text GLabel 3950 4050 0    50   Input ~ 0
@@
 F 3 "" H 3000 2000 60  0001 C CNN
 	1    3000 2000
-	1    0    0    -1
+	-1   0    0    -1
 $EndComp
 $Comp
@@
 F 3 "" H 2900 6850 60  0001 C CNN
 	1    2900 6850
-	1    0    0    -1
-$EndComp
-$Comp
+	-1   0    0    -1
+$EndComp
+$Comp

Commit message: Initial BOM files for PCB version 1.0 Added README and ToDo text files
Signed-off-by: Charles Steinkuehler <charles@steinkuehler.net>
Parts:
- C204, C205, C206: Mfg (none) -> Nichicon; PartNo (none) -> UCD1V101MCL6GS
- P207, P208, P209: Mfg (none) -> Harwin; PartNo (none) -> M20-9980345
- P210, P212, P217: Mfg (none) -> Molex; PartNo (none) -> 22-23-2061
- R207, R208, R210: Mfg (none) -> KOA; PartNo (none) -> RK73H2ATTD1003F
- U204, U205, U206: Mfg (none) -> Sullins; PartNo (none) -> PPTC241LFBN-RC
Changed lines of the file:
@@
 Sheet 5 10
 Title "CRAMPS (Cape-RAMPS for BeagleBone)"
-Date "9 feb 2014"
+Date "11 feb 2014"
 Rev "v1.0"
 Comp ""
@@
 F 2 "" H 3000 4400 60  0001 C CNN
 F 3 "" H 3000 4400 60  0001 C CNN
+F 4 "Harwin" H 6250 6550 60  0001 C CNN "Mfg"
+F 5 "M20-9980345" H 6250 6550 60  0001 C CNN "PartNo"
 	1    3000 4400
 	-1   0    0    -1
@@
 F 2 "" H 5950 4200 60  0001 C CNN
 F 3 "" H 5950 4200 60  0001 C CNN
+F 4 "Molex" H 6250 6550 60  0001 C CNN "Mfg"
+F 5 "22-23-2061" H 6250 6550 60  0001 C CNN "PartNo"
 	1    5950 4200
 	1    0    0    -1
@@
 F 2 "" H 6050 1800 60  0001 C CNN
 F 3 "" H 6050 1800 60  0001 C CNN
+F 4 "Molex" H 6250 6550 60  0001 C CNN "Mfg"
+F 5 "22-23-2061" H 6250 6550 60  0001 C CNN "PartNo"
 	1    6050 1800
 	1    0    0    -1
@@
 F 2 "" H 3000 2000 60  0001 C CNN
 F 3 "" H 3000 2000 60  0001 C CNN
+F 4 "Harwin" H 6250 6550 60  0001 C CNN "Mfg"
+F 5 "M20-9980345" H 6250 6550 60  0001 C CNN "PartNo"
 	1    3000 2000
 	-1   0    0    -1
@@
 F 2 "" H 4650 4250 60  0001 C CNN
 F 3 "" H 4650 4250 60  0001 C CNN
+F 4 "Sullins" H 6250 6550 60  0001 C CNN "Mfg"
+F 5 "PPTC241LFBN-RC" H 6250 6550 60  0001 C CNN "PartNo"
 	1    4650 4250
 	1    0    0    -1
@@
 F 2 "" H 4750 1850 60  0001 C CNN
 F 3 "" H 4750 1850 60  0001 C CNN
+F 4 "Sullins" H 6250 6550 60  0001 C CNN "Mfg"
+F 5 "PPTC241LFBN-RC" H 6250 6550 60  0001 C CNN "PartNo"
 	1    4750 1850
 	1    0    0    -1
@@
 F 2 "" H 6300 1800 60  0001 C CNN
 F 3 "" H 6300 1800 60  0001 C CNN
+F 4 "Nichicon" H 6300 1800 60  0001 C CNN "Mfg"
+F 5 "UCD1V101MCL6GS" H 6300 1800 60  0001 C CNN "PartNo"
 	1    6300 1800
 	1    0    0    -1
@@
 F 2 "" H 6200 4200 60  0001 C CNN
 F 3 "" H 6200 4200 60  0001 C CNN
+F 4 "Nichicon" H 6200 4200 60  0001 C CNN "Mfg"
+F 5 "UCD1V101MCL6GS" H 6200 4200 60  0001 C CNN "PartNo"
 	1    6200 4200
 	1    0    0    -1
@@
 F 2 "" H 3650 2400 60  0001 C CNN
 F 3 "" H 3650 2400 60  0001 C CNN
+F 4 "KOA" H 6250 6550 60  0001 C CNN "Mfg"
+F 5 "RK73H2ATTD1003F" H 6250 6550 60  0001 C CNN "PartNo"
 	1    3650 2400
 	1    0    0    -1
@@
 F 2 "" H 3550 4800 60  0001 C CNN
 F 3 "" H 3550 4800 60  0001 C CNN
+F 4 "KOA" H 6250 6550 60  0001 C CNN "Mfg"
+F 5 "RK73H2ATTD1003F" H 6250 6550 60  0001 C CNN "PartNo"
 	1    3550 4800
 	1    0    0    -1
@@
 F 2 "" H 3450 7250 60  0001 C CNN
 F 3 "" H 3450 7250 60  0001 C CNN
+F 4 "KOA" H 6250 6550 60  0001 C CNN "Mfg"
+F 5 "RK73H2ATTD1003F" H 6250 6550 60  0001 C CNN "PartNo"
 	1    3450 7250
 	1    0    0    -1
@@
 F 2 "" H 6100 6650 60  0001 C CNN
 F 3 "" H 6100 6650 60  0001 C CNN
+F 4 "Nichicon" H 6100 6650 60  0001 C CNN "Mfg"
+F 5 "UCD1V101MCL6GS" H 6100 6650 60  0001 C CNN "PartNo"
 	1    6100 6650
 	1    0    0    -1
@@
 F 2 "" H 4550 6700 60  0001 C CNN
 F 3 "" H 4550 6700 60  0001 C CNN
+F 4 "Sullins" H 6250 6550 60  0001 C CNN "Mfg"
+F 5 "PPTC241LFBN-RC" H 6250 6550 60  0001 C CNN "PartNo"
 	1    4550 6700
 	1    0    0    -1
@@
 F 2 "" H 5850 6650 60  0001 C CNN
 F 3 "" H 5850 6650 60  0001 C CNN
+F 4 "Molex" H 6250 6550 60  0001 C CNN "Mfg"
+F 5 "22-23-2061" H 6250 6550 60  0001 C CNN "PartNo"
 	1    5850 6650
 	1    0    0    -1
@@
 F 2 "" H 2900 6850 60  0001 C CNN
 F 3 "" H 2900 6850 60  0001 C CNN
+F 4 "Harwin" H 6250 6550 60  0001 C CNN "Mfg"
+F 5 "M20-9980345" H 6250 6550 60  0001 C CNN "PartNo"
 	1    2900 6850
 	-1   0    0    -1

Commit message: BOM Updates Fixed incorrect Molex part number Added Stackpole resistor part numbers Switched to value-sorted BOM export from KiCAD Modified some attribute fields to get same-value parts to list on a single BOM line
Signed-off-by: Charles Steinkuehler <charles@steinkuehler.net>
Parts:
- P210, P212, P217: PartNo 22-23-2061 -> 22-23-2041
- R207, R208, R210: AltMfg (none) -> KOA; AltPartNo (none) -> RK73H2ATTD1003F; Mfg KOA -> Stackpole; PartNo RK73H2ATTD1003F -> RMCF0805FT100K
Changed lines of the file:
@@
 Sheet 5 10
 Title "CRAMPS (Cape-RAMPS for BeagleBone)"
-Date "11 feb 2014"
+Date "15 feb 2014"
 Rev "v1.0"
 Comp ""
@@
 F 3 "" H 5950 4200 60  0001 C CNN
 F 4 "Molex" H 6250 6550 60  0001 C CNN "Mfg"
-F 5 "22-23-2061" H 6250 6550 60  0001 C CNN "PartNo"
+F 5 "22-23-2041" H 6250 6550 60  0001 C CNN "PartNo"
 	1    5950 4200
 	1    0    0    -1
@@
 F 3 "" H 6050 1800 60  0001 C CNN
 F 4 "Molex" H 6250 6550 60  0001 C CNN "Mfg"
-F 5 "22-23-2061" H 6250 6550 60  0001 C CNN "PartNo"
+F 5 "22-23-2041" H 6250 6550 60  0001 C CNN "PartNo"
 	1    6050 1800
 	1    0    0    -1
@@
 F 2 "" H 3650 2400 60  0001 C CNN
 F 3 "" H 3650 2400 60  0001 C CNN
-F 4 "KOA" H 6250 6550 60  0001 C CNN "Mfg"
-F 5 "RK73H2ATTD1003F" H 6250 6550 60  0001 C CNN "PartNo"
+F 4 "Stackpole" H 6250 6550 60  0001 C CNN "Mfg"
+F 5 "RMCF0805FT100K" H 6250 6550 60  0001 C CNN "PartNo"
+F 6 "KOA" V 3600 2450 60  0001 C CNN "AltMfg"
+F 7 "RK73H2ATTD1003F" V 3600 2450 60  0001 C CNN "AltPartNo"
 	1    3650 2400
 	1    0    0    -1
@@
 F 2 "" H 3550 4800 60  0001 C CNN
 F 3 "" H 3550 4800 60  0001 C CNN
-F 4 "KOA" H 6250 6550 60  0001 C CNN "Mfg"
-F 5 "RK73H2ATTD1003F" H 6250 6550 60  0001 C CNN "PartNo"
+F 4 "Stackpole" H 6250 6550 60  0001 C CNN "Mfg"
+F 5 "RMCF0805FT100K" H 6250 6550 60  0001 C CNN "PartNo"
+F 6 "KOA" V 3600 2450 60  0001 C CNN "AltMfg"
+F 7 "RK73H2ATTD1003F" V 3600 2450 60  0001 C CNN "AltPartNo"
 	1    3550 4800
 	1    0    0    -1
@@
 F 2 "" H 3450 7250 60  0001 C CNN
 F 3 "" H 3450 7250 60  0001 C CNN
-F 4 "KOA" H 6250 6550 60  0001 C CNN "Mfg"
-F 5 "RK73H2ATTD1003F" H 6250 6550 60  0001 C CNN "PartNo"
+F 4 "Stackpole" H 6250 6550 60  0001 C CNN "Mfg"
+F 5 "RMCF0805FT100K" H 6250 6550 60  0001 C CNN "PartNo"
+F 6 "KOA" V 3600 2450 60  0001 C CNN "AltMfg"
+F 7 "RK73H2ATTD1003F" V 3600 2450 60  0001 C CNN "AltPartNo"
 	1    3450 7250
 	1    0    0    -1
@@
 F 3 "" H 5850 6650 60  0001 C CNN
 F 4 "Molex" H 6250 6550 60  0001 C CNN "Mfg"
-F 5 "22-23-2061" H 6250 6550 60  0001 C CNN "PartNo"
+F 5 "22-23-2041" H 6250 6550 60  0001 C CNN "PartNo"
 	1    5850 6650
 	1    0    0    -1
