File: CRAMPS/con_inputs.sch (KiCad schematic (older format))
At the start: 34 parts, among them P501 HEADER_6X2, P502 HEADER_6, P503 HEADER_4X2, P504 HEADER_4X2, U501 74CBTLV3861

Commit message: General cleanup
Signed-off-by: Charles Steinkuehler <charles@steinkuehler.net>
Connections:
- wire segments 102 -> 150
Other:
- note added: "Endstop inputs are 5V tolerant\nand may also be used as 3.3V \noutput signals if desired"
- note added: "Shunt populated by default\nRemove to support\n4-wire touch-screen\nusing AIN 0-3"
- note removed: "Endstop inputs are 5V tolerant"
- note removed: "Shunt typically populated\nRemove to support\n4-wire touch-screen"
Changed lines of the file:
@@
 	1    0    0    -1
 $EndComp
-Text Notes 2100 1600 0    60   ~ 12
-Endstop inputs are 5V tolerant
-Text Notes 3100 800  2    80   ~ 16
+Text Notes 2100 1600 0    75   ~ 0
+Endstop inputs are 5V tolerant\nand may also be used as 3.3V \noutput signals if desired
+Text Notes 3100 800  2    100  ~ 0
 Endstops
 $Comp
@@
 Text GLabel 4700 4400 2    50   Output ~ 0
 SPI_CS0-5V
-Text GLabel 2800 5000 0    50   Input ~ 0
-MOSI-5V
-Text GLabel 2800 4900 0    50   Input ~ 0
-SCK-5V
-Text GLabel 2800 4800 0    50   Output ~ 0
-MISO-5V
-Text GLabel 2800 5100 0    50   Input ~ 0
-SPI_CS0
 $Comp
 L HEADER_6X2 P501
@@
 Text GLabel 8700 4600 2    50   Output ~ 0
 THERM3
-Text Notes 8200 800  2    80   ~ 16
+Text Notes 8200 800  2    100  ~ 0
 Thermistor Inputs
 Text GLabel 8700 3700 2    50   Output ~ 0
@@
 AIN3
 Text Notes 9200 4600 0    50   ~ 0
-Shunt typically populated\nRemove to support\n4-wire touch-screen
+Shunt populated by default\nRemove to support\n4-wire touch-screen\nusing AIN 0-3
 Text GLabel 8700 2300 2    50   UnSpc ~ 0
 ADC_GND
@@
 	3800 2250 3800 2350
 Wire Wire Line
-	1700 3300 1700 4000
+	1700 3300 1700 3500
+Wire Wire Line
+	1700 3500 1700 3600
+Wire Wire Line
+	1700 3600 1700 3700
+Wire Wire Line
+	1700 3700 1700 3800
+Wire Wire Line
+	1700 3800 1700 3900
+Wire Wire Line
+	1700 3900 1700 4000
 Wire Wire Line
 	3700 4500 3700 4750
@@
 	3700 4750 4200 4750
 Wire Wire Line
-	4200 4700 4200 4800
+	4200 4700 4200 4750
+Wire Wire Line
+	4200 4750 4200 4800
 Connection ~ 4200 4750
 Wire Wire Line
-	1800 3500 1800 4700
+	1800 3500 1800 3600
+Wire Wire Line
+	1800 3600 1800 3700
+Wire Wire Line
+	1800 3700 1800 3800
+Wire Wire Line
+	1800 3800 1800 3900
+Wire Wire Line
+	1800 3900 1800 4000
+Wire Wire Line
+	1800 4000 1800 4700
 Connection ~ 1800 3600
 Connection ~ 1800 3700
@@
 Connection ~ 8000 2800
 Wire Wire Line
-	7800 2800 8700 2800
-Wire Wire Line
-	7800 1900 8700 1900
+	7800 2800 8000 2800
+Wire Wire Line
+	8000 2800 8400 2800
+Wire Wire Line
+	8400 2800 8700 2800
+Wire Wire Line
+	7800 1900 8000 1900
+Wire Wire Line
+	8000 1900 8400 1900
+Wire Wire Line
+	8400 1900 8700 1900
 Wire Wire Line
 	8000 3700 8000 3800
@@
 	8000 4600 8000 4700
 Wire Wire Line
-	7800 4600 8700 4600
-Wire Wire Line
-	7800 3700 8700 3700
+	7800 4600 8000 4600
+Wire Wire Line
+	8000 4600 8400 4600
+Wire Wire Line
+	8400 4600 8700 4600
+Wire Wire Line
+	7800 3700 8000 3700
+Wire Wire Line
+	8000 3700 8400 3700
+Wire Wire Line
+	8400 3700 8700 3700
 Connection ~ 8000 4600
 Connection ~ 8000 3700
@@
 	8950 4400 9100 4400
 Wire Wire Line
-	6800 1500 7400 1500
+	6800 1500 7200 1500
+Wire Wire Line
+	7200 1500 7400 1500
 Wire Wire Line
 	7400 1500 7400 1600
@@
 	8000 2200 8000 2300
 Wire Wire Line
-	8000 2300 8700 2300
+	8000 2300 8400 2300
+Wire Wire Line
+	8400 2300 8700 2300
 Wire Wire Line
 	8400 2300 8400 2200
@@
 	8000 3100 8000 3200
 Wire Wire Line
-	8000 3200 8700 3200
+	8000 3200 8400 3200
+Wire Wire Line
+	8400 3200 8700 3200
 Wire Wire Line
 	8400 3100 8400 3200
@@
 	8000 4000 8000 4100
 Wire Wire Line
-	8000 4100 8700 4100
+	8000 4100 8400 4100
+Wire Wire Line
+	8400 4100 8700 4100
 Wire Wire Line
 	8400 4000 8400 4100
@@
 	8000 4900 8000 5000
 Wire Wire Line
-	8000 5000 8700 5000
+	8000 5000 8400 5000
+Wire Wire Line
+	8400 5000 8700 5000
 Wire Wire Line
 	8400 4900 8400 5000
 Connection ~ 8400 5000
 Wire Wire Line
-	8400 4400 8400 4700
+	8400 4400 8400 4600
+Wire Wire Line
+	8400 4600 8400 4700
 Connection ~ 8400 4600
 Wire Wire Line
 	8700 4400 8400 4400
 Wire Wire Line
-	6850 3700 7600 3700
+	6850 3700 7400 3700
+Wire Wire Line
+	7400 3700 7600 3700
 Wire Wire Line
 	6850 3700 6850 3250
@@
 	6750 3350 6750 4600
 Wire Wire Line
-	6750 4600 7600 4600
+	6750 4600 7400 4600
+Wire Wire Line
+	7400 4600 7600 4600
 Wire Wire Line
 	6850 3150 6850 2800
 Wire Wire Line
-	6850 2800 7600 2800
+	6850 2800 7400 2800
+Wire Wire Line
+	7400 2800 7600 2800
 Wire Wire Line
 	6750 3050 6750 1900
 Wire Wire Line
-	6750 1900 7600 1900
+	6750 1900 7400 1900
+Wire Wire Line
+	7400 1900 7600 1900
 Wire Wire Line
 	6850 3250 6750 3250
@@
 	6450 3350 6350 3350
 Wire Wire Line
-	6450 3050 6450 3350
+	6450 3050 6450 3150
+Wire Wire Line
+	6450 3150 6450 3250
+Wire Wire Line
+	6450 3250 6450 3350
 Connection ~ 6450 3250
 Connection ~ 6450 3150
@@
 	7400 4200 7200 4200
 Wire Wire Line
-	7200 4200 7200 1500
+	7200 4200 7200 3300
+Wire Wire Line
+	7200 3300 7200 2400
+Wire Wire Line
+	7200 2400 7200 1500
 Connection ~ 7200 1500
 Wire Wire Line
@@
 Connection ~ 7200 3300
 Wire Wire Line
-	2100 3500 3700 3500
-Wire Wire Line
-	2100 3600 3700 3600
-Wire Wire Line
-	2100 3700 3700 3700
-Wire Wire Line
-	2100 3800 3700 3800
-Wire Wire Line
-	2100 3900 3700 3900
-Wire Wire Line
-	2100 4000 3700 4000
+	2100 3500 2300 3500
+Wire Wire Line
+	2300 3500 3700 3500
+Wire Wire Line
+	2100 3600 2400 3600
+Wire Wire Line
+	2400 3600 3700 3600
+Wire Wire Line
+	2100 3700 2500 3700
+Wire Wire Line
+	2500 3700 3700 3700
+Wire Wire Line
+	2100 3800 2600 3800
+Wire Wire Line
+	2600 3800 3700 3800
+Wire Wire Line
+	2100 3900 2700 3900
+Wire Wire Line
+	2700 3900 3700 3900
+Wire Wire Line
+	2100 4000 2800 4000
+Wire Wire Line
+	2800 4000 3700 4000
 Wire Wire Line
 	2300 3100 2300 3500
@@
 Connection ~ 2800 4000
 Wire Wire Line
-	2300 2700 2300 2900
-Wire Wire Line
-	2300 2800 3200 2800
+	2300 2700 2300 2800
+Wire Wire Line
+	2300 2800 2300 2900
+Wire Wire Line
+	2300 2800 2400 2800
+Wire Wire Line
+	2400 2800 2500 2800
+Wire Wire Line
+	2500 2800 2600 2800
+Wire Wire Line
+	2600 2800 2700 2800
+Wire Wire Line
+	2700 2800 2800 2800
+Wire Wire Line
+	2800 2800 2900 2800
+Wire Wire Line
+	2900 2800 3000 2800
+Wire Wire Line
+	3000 2800 3100 2800
+Wire Wire Line
+	3100 2800 3200 2800
 Connection ~ 2300 2800
 Wire Wire Line
@@
 $EndComp
 Wire Wire Line
-	2800 4400 2800 4600
-Wire Wire Line
-	2800 4600 2100 4600
-Wire Wire Line
-	3700 4300 2700 4300
-Wire Wire Line
-	2700 4300 2700 4500
-Wire Wire Line
-	2700 4500 2100 4500
-Wire Wire Line
-	3700 4200 2600 4200
-Wire Wire Line
-	2600 4200 2600 4400
-Wire Wire Line
-	2600 4400 2100 4400
-Wire Wire Line
-	3700 4100 2500 4100
-Wire Wire Line
-	2500 4100 2500 4300
-Wire Wire Line
-	2500 4300 2100 4300
-Wire Wire Line
-	2900 3100 2900 4800
+	3100 4400 3100 4600
+Wire Wire Line
+	3100 4600 2100 4600
+Wire Wire Line
+	3700 4300 3100 4300
+Wire Wire Line
+	3100 4300 3000 4300
+Wire Wire Line
+	3000 4300 3000 4500
+Wire Wire Line
+	3000 4500 2100 4500
+Wire Wire Line
+	3700 4200 3000 4200
+Wire Wire Line
+	3000 4200 2900 4200
+Wire Wire Line
+	2900 4200 2900 4400
+Wire Wire Line
+	2900 4400 2100 4400
+Wire Wire Line
+	3700 4100 2900 4100
+Wire Wire Line
+	2900 4100 2800 4100
+Wire Wire Line
+	2800 4100 2800 4300
+Wire Wire Line
+	2800 4300 2100 4300
+Wire Wire Line
+	2900 3100 2900 4100
 Connection ~ 2900 4100
 Wire Wire Line
-	3000 3300 3000 4900
+	3000 3300 3000 4200
 Connection ~ 3000 4200
 Wire Wire Line
-	3100 3100 3100 5000
+	3100 3100 3100 4300
 Connection ~ 3100 4300
 Wire Wire Line
-	3200 3300 3200 5100
-Wire Wire Line
-	2900 4800 2800 4800
-Wire Wire Line
-	3000 4900 2800 4900
-Wire Wire Line
-	3100 5000 2800 5000
-Wire Wire Line
-	3200 5100 2800 5100
+	3200 3300 3200 4400
 Connection ~ 3200 4400
 Wire Wire Line
-	3700 4400 2800 4400
+	3700 4400 3200 4400
+Wire Wire Line
+	3200 4400 3100 4400
 $Comp
 L SHUNT S501
@@
 	1    0    0    -1
 $EndComp
+Text Label 2200 4300 0    60   ~ 0
+MISO-5V
+Text Label 2200 4400 0    60   ~ 0
+SCK-5V
+Text Label 2200 4500 0    60   ~ 0
+MOSI-5V
+Text Label 2200 4600 0    60   ~ 0
+SPI_CS0
 $EndSCHEMATC

Commit message: Reannotate all parts
Signed-off-by: Charles Steinkuehler <charles@steinkuehler.net>
Parts:
- renumbered P502 to P501, P501 to P502, P504 to P503, P503 to P504, R509 to R501, R510 to R502, R511 to R503, R512 to R504, R513 to R505, R514 to R506, R515 to R507, R516 to R508, R517 to R509, R518 to R510, R501 to R511, R502 to R512, R503 to R513, R504 to R514, R505 to R515, R506 to R516, R507 to R517, R508 to R518
Connections:
- wire segments 150 -> 98

Commit message: PCB cleanup Create 20 and 24 pin SOIC footprints
Signed-off-by: Charles Steinkuehler <charles@steinkuehler.net>
Parts:
- U501: value 74CBTLV3861 -> 74CBTD3861
Changed lines of the file:
@@
 P 4200 4000
 F 0 "U501" H 4300 4600 60  0000 L CNN
-F 1 "74CBTLV3861" H 4220 3385 60  0000 L CNN
+F 1 "74CBTD3861" H 4220 3385 60  0000 L CNN
 F 2 "~" H 4200 4100 60  0000 C CNN
 F 3 "~" H 4200 4100 60  0000 C CNN

Commit message: Updated part number attributes BOM generation looks good, pending final review
Signed-off-by: Charles Steinkuehler <charles@steinkuehler.net>
Parts:
- C501, C502, C503, C504, C505: Mfg Taiyo Yuden -> Murata; PartNo GMK212BJ104KGHT -> GRM188R71C104KA01D
- C506, C507, C508, C509: PartNo LMK212F106ZG-T -> JMK107ABJ106MAHT
- JP501: value JUMP_MINI -> HEADER_2; footprint ~ -> (none)
- P501: Mfg (none) -> Harwin; PartNo (none) -> M20-9990645
- P502: Mfg (none) -> Harwin; PartNo (none) -> M20-9980645
- P503, P504: Mfg (none) -> Harwin; PartNo (none) -> M20-9980445
- R501, R502, R503, R504, R505, R506, R507, R508, R509, R510: AltPartNo RK73H2ATTD1002F -> RK73H1JTTD1002F; PartNo RMCF0805FT10K0 -> RMCF0603FT10K0
- R511, R512, R513, R514: AltPartNo RK73H2ATTD4701F -> RK73H1JTTD2001F; PartNo RMCF0805FT4K70 -> RMCF0603FT2K00
- R515, R516, R517, R518: AltPartNo RK73H2ATTD4701F -> RK73H1JTTD4701F; PartNo RMCF0805FT4K70 -> RMCF0603FT4K70
- S501: footprint ~ -> (none); Mfg (none) -> TE; PartNo (none) -> 382811-8
- U501: footprint ~ -> (none); Field5 (none) -> SN74CBTD3861DW; Mfg (none) -> TI

Commit message: Schematic cleanup
Signed-off-by: Charles Steinkuehler <charles@steinkuehler.net>
Other:
- note added: "P503 may be used for:\n* Additional digital I/O\n* CRAMP3 add-on board\n* SPI expansion"
Changed lines of the file:
@@
 $EndDescr
 $Comp
-L GND #PWR505
+L GND #PWR069
 U 1 1 510D87E0
 P 3800 2650
-F 0 "#PWR505" H 3800 2650 30  0001 C CNN
+F 0 "#PWR069" H 3800 2650 30  0001 C CNN
 F 1 "GND" H 3800 2580 30  0001 C CNN
 F 2 "" H 3800 2650 60  0001 C CNN
@@
 $EndComp
 $Comp
-L GND #PWR507
+L GND #PWR070
 U 1 1 50FF1A09
 P 4200 4800
-F 0 "#PWR507" H 4200 4800 30  0001 C CNN
+F 0 "#PWR070" H 4200 4800 30  0001 C CNN
 F 1 "GND" H 4200 4730 30  0001 C CNN
 F 2 "" H 4200 4800 60  0001 C CNN
@@
 Endstops
 $Comp
-L GND #PWR502
+L GND #PWR071
 U 1 1 50FC388F
 P 1800 4700
-F 0 "#PWR502" H 1800 4700 30  0001 C CNN
+F 0 "#PWR071" H 1800 4700 30  0001 C CNN
 F 1 "GND" H 1800 4630 30  0001 C CNN
 F 2 "" H 1800 4700 60  0001 C CNN
@@
 $EndComp
 $Comp
-L +5V #PWR503
+L +5V #PWR072
 U 1 1 524E05B1
 P 2300 2700
-F 0 "#PWR503" H 2300 2790 20  0001 C CNN
+F 0 "#PWR072" H 2300 2790 20  0001 C CNN
 F 1 "+5V" H 2300 2790 30  0000 C CNN
 F 2 "" H 2300 2700 60  0001 C CNN
@@
 X-MIN
 $Comp
-L +5V #PWR506
+L +5V #PWR073
 U 1 1 52EFDB59
 P 4200 3250
-F 0 "#PWR506" H 4200 3340 20  0001 C CNN
+F 0 "#PWR073" H 4200 3340 20  0001 C CNN
 F 1 "+5V" H 4200 3340 30  0000 C CNN
 F 2 "" H 4200 3250 60  0001 C CNN
@@
 $EndComp
 $Comp
-L +5V #PWR504
+L +5V #PWR074
 U 1 1 52EFDB5F
 P 3800 2250
-F 0 "#PWR504" H 3800 2340 20  0001 C CNN
+F 0 "#PWR074" H 3800 2340 20  0001 C CNN
 F 1 "+5V" H 3800 2340 30  0000 C CNN
 F 2 "" H 3800 2250 60  0001 C CNN
@@
 To ADC\nInputs
 $Comp
-L +5V #PWR501
+L +5V #PWR075
 U 1 1 535FDE3E
 P 1700 3300
-F 0 "#PWR501" H 1700 3390 20  0001 C CNN
+F 0 "#PWR075" H 1700 3390 20  0001 C CNN
 F 1 "+5V" H 1700 3390 30  0000 C CNN
 F 2 "" H 1700 3300 60  0001 C CNN
@@
 Text Label 2200 4600 0    60   ~ 0
 SPI_CS0
+Text Notes 1800 5000 0    75   ~ 0
+P503 may be used for:\n* Additional digital I/O\n* CRAMP3 add-on board\n* SPI expansion
 $EndSCHEMATC

Commit message: Switch clamping diodes from ES1F to SS14
Signed-off-by: Charles Steinkuehler <charles@steinkuehler.net>
Changed lines of the file:
@@
 Sheet 5 5
 Title "CRAMPS (Cape-RAMPS for BeagleBone)"
-Date "2 may 2014"
+Date "4 may 2014"
 Rev "v1.0"
 Comp ""
@@
 Text Notes 1800 5000 0    75   ~ 0
 P503 may be used for:\n* Additional digital I/O\n* CRAMP3 add-on board\n* SPI expansion
+Connection ~ 1800 4300
+Connection ~ 1800 4400
+Connection ~ 1800 4500
+Connection ~ 1800 4600
 $EndSCHEMATC
