File: CRAMPS/CRAMPS.routed.kicad_pcb (KiCad board)
At the start: 2 copper layers, 99.1 x 99.1 mm, 192 parts, among them M101 PCB_GREEN_RMC, M102 LOGO_OSHW, P101 SOCKET_6_LONG, P102 HEADER_2, P103 HEADER_2, P201 PT_2,5-2-5,0-H, P202 KK-2.54-4W, P203 KK-2.54-4W, P204 KK-2.54-4W, P205 KK-2.54-4W, P206 KK-2.54-4W, P207 KK-2.54-4W, P208 POLOLU_SOCKET, P209 POLOLU_SOCKET, P210 POLOLU_SOCKET, P211 POLOLU_SOCKET, P301 HEADER_2, P302 KK-2.54-2W, P303 HEADER_4X2, P304 HEADER_3X2, P305 HEADER_6, P401 PT_2,5-2-5,0-H, P402 PT_2,5-2-5,0-H, P403 PT_2,5-2-5,0-H, P404 PT_1,5-3-3,5-H, P405 PT_1,5-2-3,5-H, P406 PT_1,5-2-3,5-H, P407 KK-2.54-2W, P408 PT_1,5-2-3,5-H, P409 KK-2.54-2W, P501 HEADER_6, P502 HEADER_6X2, P503 HEADER_4X2, P504 HEADER_4X2, P8 BB_EXP_CONN, P9 BB_EXP_CONN, Q101 2N7002K, Q301 2N7002K, Q302 2N7002K, Q303 2N7002K, Q304 2N7002K, Q305 2N7002K, Q401 IRLB8743PBF, Q402 IRLB8743PBF, Q403 IRLB8743PBF, Q404 DMN2075U, Q405 IRLB8743PBF, Q406 DMN2075U, SW101 SW_PUSH, SW102 SW_PUSH, U201 Pololu, U202 Pololu, U203 Pololu, U204 Pololu, U205 Pololu, U206 Pololu, U301 24C256, U302 74ACT244, U501 74CBTD3861

Commit message: More post-route cleanup
Signed-off-by: Charles Steinkuehler <charles@steinkuehler.net>
Parts:
- moved Q305 6.35 mm to (100.3, 97.8)
- moved Q302 3.81 mm to (100.3, 101.6)
- turned JP301 to 90 degrees
Routing:
- net DGND: track 710.7 -> 719.6 mm, vias 8 -> 9
- net D3.3V: track 335.4 -> 326.9 mm
- net N-00000185: track 2.94 -> 9.55 mm
- net Y_STEP: track 20.9 -> 26.2 mm
- net FET5: track 57.8 -> 62.9 mm, vias 1 -> 2
- net N-00000180: track 14.4 -> 9.84 mm, vias 2 -> 0
- net FET1: track 36.3 -> 32.0 mm
- net Z_DIR: track 45.4 -> 41.8 mm
- net E0_EN_BUFn: track 165.4 -> 163.2 mm
- net AXIS_ENAn: track 34.0 -> 36.1 mm
- net N-00000184: track 115.4 -> 117.2 mm
- net FET6_BUF: track 44.9 -> 43.4 mm
- net ADC_VDD: track 45.4 -> 43.9 mm
- net Y_DIR: track 25.8 -> 24.4 mm
- net /Emergency Stop/MACHINE_PWRn: track 54.0 -> 52.7 mm
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Other:
- board text added: "A0"
- board text added: "PWR ON"
- board text added: "WP"

Commit message: Cleanup mostly complete, ready for final check plots
Signed-off-by: Charles Steinkuehler <charles@steinkuehler.net>
Routing:
- net E0_EN_BUFn: track 163.2 -> 163.9 mm
Changed lines of the file:
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@@
     (links 451)
     (no_connects 0)
-    (area 23.6982 8.84428 158.9278 149.3012)
+    (area 50.609499 34.099499 150.050501 133.540501)
     (thickness 1.6002)
     (drawings 297)
-    (tracks 1949)
+    (tracks 1953)
     (zones 0)
     (modules 192)
@@
     (pcbplotparams
       (layerselection 284721153)
-      (usegerberextensions false)
+      (usegerberextensions true)
       (excludeedgelayer true)
       (linewidth 0.150000)
@@
       (viasonmask false)
       (mode 1)
-      (useauxorigin false)
+      (useauxorigin true)
       (hpglpennumber 1)
       (hpglpenspeed 20)
@@
       (plotinvisibletext false)
       (padsonsilk false)
-      (subtractmaskfromsilk false)
-      (outputformat 2)
+      (subtractmaskfromsilk true)
+      (outputformat 1)
       (mirror false)
       (drillshape 0)
@@
   (segment (start 93.98 107.95) (end 95.25 106.68) (width 0.2032) (layer Front) (net 53))
   (segment (start 93.98 107.95) (end 95.25 106.68) (width 0.2032) (layer Front) (net 53))
+  (segment (start 88.9 60.325) (end 88.9 62.23) (width 0.2032) (layer Back) (net 54))
+  (segment (start 100.711 72.771) (end 100.711 73.66) (width 0.2032) (layer Back) (net 54))
+  (segment (start 90.805 62.865) (end 100.711 72.771) (width 0.2032) (layer Back) (net 54))
+  (segment (start 89.535 62.865) (end 90.805 62.865) (width 0.2032) (layer Back) (net 54))
+  (segment (start 88.9 62.23) (end 89.535 62.865) (width 0.2032) (layer Back) (net 54))
   (segment (start 125.73 113.03) (end 124.587 111.887) (width 0.2032) (layer Front) (net 54))
   (segment (start 106.553 111.887) (end 105.41 113.03) (width 0.2032) (layer Front) (net 54))
@@
   (segment (start 84.455 56.515) (end 88.9 56.515) (width 0.2032) (layer Back) (net 54))
   (segment (start 100.711 74.168) (end 100.7116 74.168) (width 0.2032) (layer Back) (net 54))
-  (segment (start 100.711 73.406) (end 100.711 74.168) (width 0.2032) (layer Back) (net 54))
-  (segment (start 88.9 61.595) (end 100.711 73.406) (width 0.2032) (layer Back) (net 54))
-  (segment (start 88.9 56.515) (end 88.9 61.595) (width 0.2032) (layer Back) (net 54))
+  (segment (start 100.711 73.66) (end 100.711 74.168) (width 0.2032) (layer Back) (net 54))
+  (segment (start 88.9 56.515) (end 88.9 60.325) (width 0.2032) (layer Back) (net 54))
   (segment (start 100.7116 79.5003) (end 100.7116 74.168) (width 0.2032) (layer Back) (net 54))
   (via (at 100.7116 79.5003) (size 0.635) (layers Front Back) (net 54))
@@
     (polygon
       (pts
-        (xy 51.435 50.8) (xy 60.325 50.8) (xy 65.405 45.72) (xy 74.93 45.72) (xy 75.565 45.085)
-        (xy 78.74 45.085) (xy 79.375 45.72) (xy 79.375 53.34) (xy 78.105 54.61) (xy 74.93 54.61)
-        (xy 73.66 55.88) (xy 66.04 55.88) (xy 63.5 58.42) (xy 60.96 58.42) (xy 60.325 59.055)
-        (xy 60.325 71.755) (xy 51.435 71.755) (xy 51.435 67.945)
+        (xy 51.435 50.8) (xy 60.325 50.8) (xy 66.04 45.085) (xy 78.74 45.085) (xy 79.375 45.72)
+        (xy 79.375 53.34) (xy 78.105 54.61) (xy 74.93 54.61) (xy 73.66 55.88) (xy 66.04 55.88)
+        (xy 63.5 58.42) (xy 60.96 58.42) (xy 60.325 59.055) (xy 60.325 71.755) (xy 51.435 71.755)
+        (xy 51.435 67.945)
       )
     )
@@
         (xy 80.645 90.805) (xy 83.82 90.805) (xy 83.82 71.755) (xy 60.96 71.755) (xy 60.96 59.69)
         (xy 61.595 59.055) (xy 64.135 59.055) (xy 66.675 56.515) (xy 74.295 56.515) (xy 75.565 55.245)
-        (xy 78.74 55.245) (xy 80.01 53.975) (xy 80.01 45.085) (xy 79.375 44.45) (xy 74.93 44.45)
-        (xy 74.295 45.085) (xy 64.77 45.085) (xy 59.69 50.165) (xy 51.435 50.165) (xy 51.435 34.925)
-        (xy 149.225 34.925)
+        (xy 78.74 55.245) (xy 80.01 53.975) (xy 80.01 45.085) (xy 79.375 44.45) (xy 65.405 44.45)
+        (xy 59.69 50.165) (xy 51.435 50.165) (xy 51.435 34.925) (xy 149.225 34.925)
       )
     )

Commit message: Continued PCB Cleanup
Signed-off-by: Charles Steinkuehler <charles@steinkuehler.net>
Routing:
- net SPI_CS1: track 71.8 -> 73.0 mm
- net FET6_BUF: track 43.4 -> 42.9 mm
Changed lines of the file:
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@@
     (links 451)
     (no_connects 0)
-    (area 50.609499 34.099499 150.050501 133.540501)
+    (area 23.6982 8.84428 158.9278 149.3012)
     (thickness 1.6002)
-    (drawings 297)
-    (tracks 1953)
+    (drawings 303)
+    (tracks 1958)
     (zones 0)
     (modules 192)
@@
     (descr "Pin strip 4x2pin")
     (tags "CONN DEV")
-    (fp_text reference P503 (at -6.35 0 270) (layer F.SilkS)
+    (fp_text reference P503 (at 6.35 0 270) (layer F.SilkS)
       (effects (font (size 1.016 1.016) (thickness 0.2032)))
     )
@@
     )
   )
+  (gr_text S (at 66.04 109.22 90) (layer F.SilkS)
+    (effects (font (size 1.27 1.27) (thickness 0.3048)))
+  )
+  (gr_line (start 138.43 69.215) (end 138.43 67.945) (angle 90) (layer F.SilkS) (width 0.3048))
+  (gr_text S (at 138.43 71.12 90) (layer F.SilkS)
+    (effects (font (size 1.27 1.27) (thickness 0.3048)))
+  )
+  (gr_line (start 145.415 88.9) (end 146.685 88.9) (angle 90) (layer F.SilkS) (width 0.3048))
+  (gr_line (start 146.05 89.535) (end 146.05 88.265) (angle 90) (layer F.SilkS) (width 0.3048))
+  (gr_line (start 143.51 89.535) (end 143.51 88.265) (angle 90) (layer F.SilkS) (width 0.3048))
+  (gr_line (start 139.7 67.31) (end 139.7 72.39) (angle 90) (layer F.SilkS) (width 0.3048))
+  (gr_line (start 137.16 67.31) (end 139.7 67.31) (angle 90) (layer F.SilkS) (width 0.3048))
   (gr_line (start 67.31 110.49) (end 67.31 107.95) (angle 90) (layer F.SilkS) (width 0.3048))
   (gr_line (start 62.23 110.49) (end 67.31 110.49) (angle 90) (layer F.SilkS) (width 0.3048))
@@
     (effects (font (size 1.27 1.27) (thickness 0.3048)))
   )
-  (gr_line (start 65.405 109.22) (end 66.675 109.22) (angle 90) (layer F.SilkS) (width 0.3048))
-  (gr_line (start 66.04 108.585) (end 66.04 109.855) (angle 90) (layer F.SilkS) (width 0.3048))
   (gr_line (start 63.5 108.585) (end 63.5 109.855) (angle 90) (layer F.SilkS) (width 0.3048))
   (gr_text "LIMIT SW" (at 138.43 80.01 90) (layer F.SilkS)
@@
   (segment (start 94.3434 80.645) (end 94.4451 80.645) (width 0.2032) (layer Front) (net 50))
   (segment (start 94.4451 80.645) (end 94.615 80.645) (width 0.2032) (layer Front) (net 50))
+  (segment (start 114.3 48.26) (end 114.3 45.72) (width 0.4064) (layer Back) (net 51))
+  (segment (start 114.3 50.8) (end 114.3 48.26) (width 0.4064) (layer Front) (net 51))
   (segment (start 84.455 104.775) (end 83.185 103.505) (width 0.2032) (layer Back) (net 51))
   (segment (start 83.185 100.33) (end 83.82 99.695) (width 0.2032) (layer Back) (net 51))
@@
   (segment (start 95.25 45.72) (end 97.79 43.18) (width 0.4064) (layer Back) (net 51))
   (segment (start 114.3 45.72) (end 115.57 45.72) (width 0.4064) (layer Back) (net 51))
-  (segment (start 118.11 43.18) (end 118.11 41.91) (width 0.4064) (layer Back) (net 51))
   (segment (start 115.57 45.72) (end 118.11 43.18) (width 0.4064) (layer Back) (net 51))
-  (segment (start 114.3 50.8) (end 114.3 48.26) (width 0.4064) (layer Back) (net 51))
-  (segment (start 114.3 48.26) (end 114.3 45.72) (width 0.4064) (layer Front) (net 51))
+  (segment (start 118.11 43.18) (end 118.11 41.91) (width 0.4064) (layer Back) (net 51))
   (segment (start 133.35 54.61) (end 133.35 53.34) (width 0.4064) (layer Front) (net 51))
   (segment (start 134.62 52.07) (end 134.62 50.8) (width 0.4064) (layer Front) (net 51))
@@
   (segment (start 100.5411 91.821) (end 103.5813 91.821) (width 0.2032) (layer Front) (net 73))
   (segment (start 94.4451 85.725) (end 100.5411 91.821) (width 0.2032) (layer Front) (net 73))
+  (segment (start 83.508 115.824) (end 83.508 115.247) (width 0.2032) (layer Front) (net 74))
+  (segment (start 83.508 115.247) (end 83.82 114.935) (width 0.2032) (layer Front) (net 74))
+  (segment (start 83.82 114.935) (end 84.455 114.935) (width 0.2032) (layer Front) (net 74))
+  (segment (start 84.455 114.935) (end 85.725 113.665) (width 0.2032) (layer Front) (net 74))
+  (segment (start 85.725 113.665) (end 85.725 112.395) (width 0.2032) (layer Front) (net 74))
+  (segment (start 85.725 112.395) (end 86.36 111.76) (width 0.2032) (layer Front) (net 74))
   (segment (start 88.9 111.125) (end 90.805 111.125) (width 0.2032) (layer Back) (net 74))
   (segment (start 91.44 100.965) (end 97.8235 94.5815) (width 0.2032) (layer Back) (net 74))
   (segment (start 91.44 110.49) (end 91.44 100.965) (width 0.2032) (layer Back) (net 74))
   (segment (start 90.805 111.125) (end 91.44 110.49) (width 0.2032) (layer Back) (net 74))
-  (segment (start 83.508 115.824) (end 83.508 115.247) (width 0.2032) (layer Front) (net 74))
-  (segment (start 83.508 115.247) (end 84.455 114.3) (width 0.2032) (layer Front) (net 74))
   (segment (start 88.9 111.125) (end 86.995 111.125) (width 0.2032) (layer Back) (net 74))
   (segment (start 86.995 111.125) (end 86.36 111.76) (width 0.2032) (layer Back) (net 74))
   (via (at 86.36 111.76) (size 0.635) (layers Front Back) (net 74))
-  (segment (start 86.36 111.76) (end 86.36 112.2019) (width 0.2032) (layer Front) (net 74))
-  (segment (start 86.36 112.2019) (end 86.36 112.395) (width 0.2032) (layer Front) (net 74))
-  (segment (start 86.36 112.395) (end 84.455 114.3) (width 0.2032) (layer Front) (net 74))
-  (segment (start 84.455 114.3) (end 83.82 114.935) (width 0.2032) (layer Front) (net 74))
   (via (at 97.8235 87.6431) (size 0.635) (layers Front Back) (net 74))
   (segment (start 83.508 117.348) (end 83.508 115.824) (width 0.2032) (layer Front) (net 74))
@@
   (segment (start 120.015 74.295) (end 118.0626 74.295) (width 0.2032) (layer Front) (net 135))
   (segment (start 118.0626 74.295) (end 116.8099 75.5477) (width 0.2032) (layer Front) (net 135))
-  (segment (start 121.8639 88.3211) (end 121.1728 87.63) (width 0.2032) (layer Front) (net 136))
-  (segment (start 113.5365 85.5965) (end 113.5365 84.1772) (width 0.2032) (layer Front) (net 136))
-  (segment (start 115.57 87.63) (end 113.5365 85.5965) (width 0.2032) (layer Front) (net 136))
-  (segment (start 121.1728 87.63) (end 115.57 87.63) (width 0.2032) (layer Front) (net 136))
-  (segment (start 113.03 71.12) (end 113.03 72.39) (width 0.2032) (layer Back) (net 136))
-  (via (at 113.5365 84.1772) (size 0.635) (layers Front Back) (net 136))
-  (segment (start 113.03 72.39) (end 114.3 73.66) (width 0.2032) (layer Back) (net 136))
-  (segment (start 114.3 73.66) (end 114.3 83.4137) (width 0.2032) (layer Back) (net 136))
-  (segment (start 114.3 83.4137) (end 113.5365 84.1772) (width 0.2032) (layer Back) (net 136))
+  (segment (start 139.065 104.775) (end 140.335 103.505) (width 0.2032) (layer Front) (net 136))
+  (segment (start 140.335 103.505) (end 140.335 102.235) (width 0.2032) (layer Front) (net 136))
+  (segment (start 137.795 105.41) (end 138.43 105.41) (width 0.2032) (layer Front) (net 136))
+  (segment (start 142.8451 88.8701) (end 144.78 90.805) (width 0.2032) (layer Front) (net 136))
+  (segment (start 137.795 88.8701) (end 122.4129 88.8701) (width 0.2032) (layer Front) (net 136))
   (segment (start 122.4129 88.8701) (end 121.8639 88.3211) (width 0.2032) (layer Front) (net 136))
-  (segment (start 142.5648 88.8701) (end 122.4129 88.8701) (width 0.2032) (layer Front) (net 136))
-  (segment (start 144.6407 90.946) (end 142.5648 88.8701) (width 0.2032) (layer Front) (net 136))
-  (segment (start 144.6407 100.0124) (end 144.6407 90.946) (width 0.2032) (layer Front) (net 136))
-  (segment (start 143.8147 100.8384) (end 144.6407 100.0124) (width 0.2032) (layer Front) (net 136))
-  (segment (start 142.6726 100.8384) (end 143.8147 100.8384) (width 0.2032) (layer Front) (net 136))
-  (segment (start 138.101 105.41) (end 142.6726 100.8384) (width 0.2032) (layer Front) (net 136))
-  (segment (start 134.62 105.41) (end 138.101 105.41) (width 0.2032) (layer Front) (net 136))
+  (segment (start 114.3 83.4137) (end 113.5365 84.1772) (width 0.2032) (layer Back) (net 136))
+  (segment (start 114.3 73.66) (end 114.3 83.4137) (width 0.2032) (layer Back) (net 136))
+  (segment (start 113.03 72.39) (end 114.3 73.66) (width 0.2032) (layer Back) (net 136))
+  (via (at 113.5365 84.1772) (size 0.635) (layers Front Back) (net 136))
+  (segment (start 113.03 71.12) (end 113.03 72.39) (width 0.2032) (layer Back) (net 136))
+  (segment (start 121.1728 87.63) (end 115.57 87.63) (width 0.2032) (layer Front) (net 136))
+  (segment (start 115.57 87.63) (end 113.5365 85.5965) (width 0.2032) (layer Front) (net 136))
+  (segment (start 113.5365 85.5965) (end 113.5365 84.1772) (width 0.2032) (layer Front) (net 136))
+  (segment (start 121.8639 88.3211) (end 121.1728 87.63) (width 0.2032) (layer Front) (net 136))
+  (segment (start 142.8451 88.8701) (end 137.795 88.8701) (width 0.2032) (layer Front) (net 136))
+  (segment (start 141.605 100.965) (end 140.335 102.235) (width 0.2032) (layer Front) (net 136))
+  (segment (start 144.145 100.965) (end 141.605 100.965) (width 0.2032) (layer Front) (net 136))
+  (segment (start 144.78 100.33) (end 144.145 100.965) (width 0.2032) (layer Front) (net 136))
+  (segment (start 144.78 90.805) (end 144.78 100.33) (width 0.2032) (layer Front) (net 136))
+  (segment (start 139.065 104.775) (end 138.43 105.41) (width 0.2032) (layer Front) (net 136))
+  (segment (start 134.62 105.41) (end 137.795 105.41) (width 0.2032) (layer Front) (net 136))
   (segment (start 133.35 106.68) (end 134.62 105.41) (width 0.2032) (layer Front) (net 136))
   (segment (start 110.49 71.12) (end 109.22 69.85) (width 0.2032) (layer Back) (net 137))
