File: R2C2_cp_shield/R2C2_shield_template.sch (KiCad schematic (older format))
At the start: 28 parts, among them J1 R2C2_CONNECTOR, P1 LCD, P2 Gen4 Interface Board, P3 UART, P4 ENC28J60, P5 RRW_PANEL, Q1 BC337, Q2 BC337, Q3 BC337, U1 74HCT165, U2 74HCT164, U3 CONN_CORTEX_DEBUG, U4 LPC11XX_HVQFN33, X1 12 MHz

Commit message: R2C2_cp_shield: add some notes to schematic
Connections:
- wire segments 156 -> 165
Other:
- note added: "??"
- note added: "For standalone variant"
- note added: "For standalone variant:\nconnect VCC, 3.3V, GND, \nEX_TXD and EX_RXD only"
- note added: "XX"
