File: RAMPS-FD-EXT/Mosfets2.sch (KiCad schematic (older format))
At the start: 14 parts, among them P601 FET_5, P602 FET_4, Q601 DMN2075U, Q602 DMN2075U, Q603 IRLB8743PBF, Q604 IRLB8743PBF

Commit message: RAMPS-FD V2.A
Connections:
- net +V_POWER: now also R603.1, R604.1
- net V_GATE: no longer R603.1, R604.1
Changed lines of the file:
@@
 Sheet 6 6
 Title ""
-Date "10 oct 2013"
+Date "8 feb 2014"
 Rev ""
 Comp ""
@@
 	3650 6200 2800 6200
 Wire Wire Line
-	4350 5550 4350 4700
+	4350 4700 4350 5550
 Wire Wire Line
 	4350 5550 4950 5550
 Wire Wire Line
 	4250 1100 4250 1700
-Wire Wire Line
-	2100 1250 3300 1250
 Wire Wire Line
 	3300 2400 3300 2450
@@
 	3300 2000 3300 1900
 Wire Wire Line
-	4700 2250 4700 1250
+	4700 1250 4700 2250
 Wire Wire Line
 	4700 2250 5100 2250
@@
 	3450 5750 4950 5750
 Wire Wire Line
-	2150 4700 3450 4700
-Wire Wire Line
 	3950 6950 3950 6350
 Wire Wire Line
@@
 	1600 3150 2450 3150
 Wire Wire Line
-	4700 1250 4250 1250
-Wire Wire Line
-	4350 4700 3950 4700
+	3300 1250 4700 1250
+Wire Wire Line
+	3450 4700 4350 4700
 Connection ~ 3950 4700
 Text Label 4500 5750 0    50   ~ 0
@@
 Text Label 4600 2450 0    50   ~ 0
 P_FET4
+Wire Wire Line
+	2750 1250 2100 1250
+Wire Wire Line
+	2800 4700 2150 4700
 $EndSCHEMATC
