File: CRAMP3/CRAMP3.kicad_pcb (KiCad board)
At the start: 2 copper layers, 20 parts, among them M101 POLOLU_SOCKET, M102 POLOLU_SOCKET, P101 HEADER_3X2, P102 HEADER_3X2, P103 HEADER_3X2, P104 X-MOT, P105 Y-MOT, P106 Z-MOT, P107 HEADER_4X2, P108 Aux-3, P109 HEADER_3X2, U101 SM_DRIVER, U102 SM_DRIVER, U103 SM_DRIVER

Commit message: CRAMP3 updates, PCB mostly complete
Signed-off-by: Charles Steinkuehler <charles@steinkuehler.net>
Parts:
- removed P103: HEADER_3X2, pin_strip_3x2
- added M1: 4-40, MTH_4-40, F.Cu at (77.5, 59.7)
- added M2: 4-40, MTH_4-40, F.Cu at (143.5, 62.9)
- added P3: HEADER_3X2, pin_strip_3x2, F.Cu at (123.2, 82.5)
- moved R3 44.0 mm to (121.9, 74.3), turned to 0 degrees
- moved P4 41.9 mm to (86.4, 60.3)
- moved U1 41.9 mm to (86.4, 77.5)
- moved C3 41.9 mm to (121.9, 69.8)
- moved P1 41.9 mm to (82.5, 82.5)
- moved C1 40.6 mm to (81.3, 69.8)
- moved P6 39.4 mm to (127.0, 60.3)
- moved U3 39.4 mm to (127.0, 77.5)
- moved R1 39.0 mm to (81.3, 74.3), turned to 0 degrees
- moved R2 8.64 mm to (101.6, 74.3), turned to 0 degrees
- moved C2 1.27 mm to (100.3, 69.8)
- moved P10 1.27 mm to (77.5, 77.5)
- moved P11 1.27 mm to (77.5, 64.8)
- moved P2 1.27 mm to (102.9, 82.5)
- moved P5 1.27 mm to (106.7, 60.3)
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- renumbered C101 to C1, C102 to C2, C103 to C3, P101 to P1, M101 to P10, M102 to P11, P102 to P2, P104 to P4, P105 to P5, P106 to P6, P107 to P7, P108 to P8, P109 to P9, R101 to R1, R102 to R2, R103 to R3, U101 to U1, U102 to U2, U103 to U3
Connections:
- P7 pad 2: (no net) -> STEP_1
- P7 pad 4: (no net) -> STEP_2
- P7 pad 6: (no net) -> DIR_1
- P7 pad 8: (no net) -> DIR_2
- P8 pad 3: (no net) -> STEP_0
- P8 pad 5: (no net) -> DIR_0
- U1 pad 7: (no net) -> STEP_0
- U1 pad 8: (no net) -> DIR_0
- U2 pad 7: (no net) -> STEP_1
- U2 pad 8: (no net) -> DIR_1
- U3 pad 7: (no net) -> STEP_2
- U3 pad 8: (no net) -> DIR_2
Routing:
- net +3.3V: track 0.00 -> 135.7 mm
- net +V_MOTOR: track 0.00 -> 68.1 mm
- net ENAn: track 0.00 -> 61.8 mm
- net STEP_0: track 0.00 -> 25.8 mm
- net DIR_1: track 0.00 -> 24.2 mm
- net GND: track 0.00 -> 22.3 mm
- net STEP_1: track 0.00 -> 21.1 mm
- net DIR_0: track 0.00 -> 19.7 mm
- net STEP_2: track 0.00 -> 9.94 mm
- net DIR_2: track 0.00 -> 9.94 mm
- net N-0000040: track 0.00 -> 7.17 mm
- net N-0000043: track 0.00 -> 7.17 mm
- net N-0000042: track 0.00 -> 7.17 mm
- net N-000009: track 0.00 -> 4.44 mm
- net N-0000041: track 0.00 -> 4.44 mm
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- added copper zone on B.Cu, net GND
- added copper zone on F.Cu, net GND
Other:
- board outline added: 72.4 x 31.1 mm

Commit message: More progress on CRAMP3
Signed-off-by: Charles Steinkuehler <charles@steinkuehler.net>
Parts:
- added Logo: OSHW_LOGO, OSHW_Logo_5, F.Cu at (132.1, 81.9)
- added S1: SHUNT, Shunt, F.Cu at (80.0, 82.5)
- added S2: SHUNT, Shunt, F.Cu at (82.5, 82.5)
- added S3: SHUNT, Shunt, F.Cu at (85.1, 82.5)
- added S4: SHUNT, Shunt, F.Cu at (100.3, 82.5)
- added S5: SHUNT, Shunt, F.Cu at (102.9, 82.5)
- added S6: SHUNT, Shunt, F.Cu at (105.4, 82.5)
- added S7: SHUNT, Shunt, F.Cu at (120.7, 82.5)
- added S8: SHUNT, Shunt, F.Cu at (123.2, 82.5)
- added S9: SHUNT, Shunt, F.Cu at (125.7, 82.5)
- P4: value X-MOT -> KK-2.54-4W
- P5: value Y-MOT -> KK-2.54-4W
- P6: value Z-MOT -> KK-2.54-4W
- P7: value HEADER_4X2 -> SOCKET_4X2; footprint pin_strip_4x2 -> Pin_Socket_4x2; moved to B.Cu
- P8: value Aux-3 -> SOCKET_4X2; footprint pin_strip_4x2 -> Pin_Socket_4x2; moved to B.Cu
- P9: value HEADER_3X2 -> SOCKET_3X2; footprint pin_strip_3x2 -> Pin_Socket_3x2; moved to B.Cu
- U1, U2, U3: value SM_DRIVER -> Pololu
- turned P7 to 180 degrees
Connections:
- net DIR_0 renamed DIR_U
- net N-000001 renamed /W2B
- net N-0000012 renamed /U1A
- net N-0000013 renamed /V2B
- net N-0000014 renamed /V2A
- net N-0000015 renamed /V1A
- net N-0000016 renamed /V1B
- net N-0000019 renamed /U2B
- net N-000002 renamed /W2A
- net N-0000020 renamed /U2A
- net N-000003 renamed /W1A
- net N-0000041 renamed /W1B
- net N-000009 renamed /U1B
- net STEP_0 renamed STEP_U
- P7 pad 2: STEP_1 -> STEP_W
- P7 pad 3: (no net) -> GND
- P7 pad 4: STEP_2 -> STEP_V
- P7 pad 5: (no net) -> GND
- P7 pad 6: DIR_1 -> DIR_W
- P7 pad 7: (no net) -> GND
- P7 pad 8: DIR_2 -> DIR_V
- P9 pad 1: GND -> +V_MOTOR
- P9 pad 2: +V_MOTOR -> GND
- P9 pad 3: GND -> +V_MOTOR
- P9 pad 4: +V_MOTOR -> GND
- P9 pad 5: GND -> +V_MOTOR
- P9 pad 6: +V_MOTOR -> GND
- U2 pad 7: STEP_1 -> STEP_V
- U2 pad 8: DIR_1 -> DIR_V
- U3 pad 7: STEP_2 -> STEP_W
- U3 pad 8: DIR_2 -> DIR_W
Routing:
- net STEP_V: track 0.00 -> 24.7 mm
- net DIR_1: track 24.2 -> 0.00 mm
- net STEP_1: track 21.1 -> 0.00 mm
- net DIR_V: track 0.00 -> 16.1 mm
- net DIR_W: track 0.00 -> 12.1 mm
- net STEP_2: track 9.94 -> 0.00 mm
- net DIR_2: track 9.94 -> 0.00 mm
- net STEP_W: track 0.00 -> 7.40 mm
- net +V_MOTOR: track 68.1 -> 75.2 mm
- net +3.3V: track 135.7 -> 138.8 mm
Other:
- board text added: "1"
- board text added: "2"
- board text added: "3"
- board text added: "CRAMP3 V1.0"
- board text added: "U"
- board text added: "V"
- board text added: "W"
- board text added: "©2014 GPL v3"

Commit message: More CRAMP3 updates
Signed-off-by: Charles Steinkuehler <charles@steinkuehler.net>
Connections:
- P8 pad 3: STEP_U -> (no net)
- P8 pad 4: (no net) -> STEP_U
- P8 pad 5: DIR_U -> (no net)
- P8 pad 6: (no net) -> DIR_U
Routing:
- net STEP_U: track 25.8 -> 24.7 mm
Changed lines of the file:
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@@
     (thickness 1.6)
     (drawings 32)
-    (tracks 145)
+    (tracks 148)
     (zones 0)
     (modules 32)
@@
     (pad 3 thru_hole circle (at -1.27 1.27 180) (size 1.651 1.651) (drill 1.016)
       (layers *.Cu *.Mask B.SilkS)
+    )
+    (pad 4 thru_hole circle (at -1.27 -1.27 180) (size 1.651 1.651) (drill 1.016)
+      (layers *.Cu *.Mask B.SilkS)
       (net 29 STEP_U)
     )
-    (pad 4 thru_hole circle (at -1.27 -1.27 180) (size 1.651 1.651) (drill 1.016)
-      (layers *.Cu *.Mask B.SilkS)
-    )
     (pad 5 thru_hole circle (at 1.27 1.27 180) (size 1.651 1.651) (drill 1.016)
       (layers *.Cu *.Mask B.SilkS)
+    )
+    (pad 6 thru_hole circle (at 1.27 -1.27 180) (size 1.651 1.651) (drill 1.016)
+      (layers *.Cu *.Mask B.SilkS)
       (net 15 DIR_U)
-    )
-    (pad 6 thru_hole circle (at 1.27 -1.27 180) (size 1.651 1.651) (drill 1.016)
-      (layers *.Cu *.Mask B.SilkS)
     )
     (pad 7 thru_hole circle (at 3.81 1.27 180) (size 1.651 1.651) (drill 1.016)
@@
   (segment (start 125.73 64.77) (end 125.73 60.325) (width 0.762) (layer B.Cu) (net 13))
   (segment (start 123.19 64.77) (end 123.19 60.325) (width 0.762) (layer B.Cu) (net 14))
-  (segment (start 110.49 68.58) (end 109.22 69.85) (width 0.254) (layer B.Cu) (net 15))
-  (segment (start 95.25 76.2) (end 95.25 77.47) (width 0.254) (layer B.Cu) (net 15))
-  (segment (start 101.6 69.85) (end 95.25 76.2) (width 0.254) (layer B.Cu) (net 15))
-  (segment (start 109.22 69.85) (end 101.6 69.85) (width 0.254) (layer B.Cu) (net 15))
+  (segment (start 110.49 71.12) (end 109.22 72.39) (width 0.254) (layer B.Cu) (net 15))
+  (segment (start 96.52 78.74) (end 95.25 77.47) (width 0.254) (layer B.Cu) (net 15))
+  (segment (start 98.425 78.74) (end 96.52 78.74) (width 0.254) (layer B.Cu) (net 15))
+  (segment (start 99.06 78.105) (end 98.425 78.74) (width 0.254) (layer B.Cu) (net 15))
+  (segment (start 99.06 76.2) (end 99.06 78.105) (width 0.254) (layer B.Cu) (net 15))
+  (segment (start 102.87 72.39) (end 99.06 76.2) (width 0.254) (layer B.Cu) (net 15))
+  (segment (start 109.22 72.39) (end 102.87 72.39) (width 0.254) (layer B.Cu) (net 15))
   (segment (start 115.57 76.2) (end 115.57 77.47) (width 0.254) (layer B.Cu) (net 16))
   (segment (start 128.27 71.12) (end 120.65 71.12) (width 0.254) (layer B.Cu) (net 16))
@@
   (segment (start 121.1 75.75) (end 120.65 76.2) (width 0.254) (layer F.Cu) (net 28))
   (segment (start 120.65 81.28) (end 120.65 77.47) (width 0.254) (layer B.Cu) (net 28))
-  (segment (start 113.03 68.58) (end 111.76 67.31) (width 0.254) (layer B.Cu) (net 29))
+  (segment (start 111.76 69.85) (end 99.06 69.85) (width 0.254) (layer B.Cu) (net 29))
+  (segment (start 99.06 69.85) (end 92.71 76.2) (width 0.254) (layer B.Cu) (net 29))
+  (segment (start 113.03 71.12) (end 111.76 69.85) (width 0.254) (layer B.Cu) (net 29))
   (segment (start 92.71 76.2) (end 92.71 77.47) (width 0.254) (layer B.Cu) (net 29))
-  (segment (start 101.6 67.31) (end 92.71 76.2) (width 0.254) (layer B.Cu) (net 29))
-  (segment (start 111.76 67.31) (end 101.6 67.31) (width 0.254) (layer B.Cu) (net 29))
   (segment (start 133.35 71.12) (end 132.08 69.85) (width 0.254) (layer B.Cu) (net 30))
   (segment (start 132.08 69.85) (end 119.38 69.85) (width 0.254) (layer B.Cu) (net 30))

Commit message: Initial CRAMP3 Gerbers
Signed-off-by: Charles Steinkuehler <charles@steinkuehler.net>
Routing:
- net GND: track 22.3 -> 54.4 mm
Changed lines of the file:
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@@
     (area 73.676934 53.898799 147.303066 88.8238)
     (thickness 1.6)
-    (drawings 32)
-    (tracks 148)
+    (drawings 35)
+    (tracks 162)
     (zones 0)
     (modules 32)
     (nets 32)
   )
-  (page A3)
+  (page A)
+  (title_block
+    (title "CRAMP3 (3-axis add-on for CRAMPS)")
+    (rev 1.0)
+    (comment 2 "Derived from CRAMPS by Charles Steinkuehler and Murray Lindeblom")
+    (comment 3 "Copyright 2014 GPL v3")
+    (comment 4 "CRAMP3 by Charles Steinkuehler")
+  )
   (layers
     (15 F.Cu signal)
@@
     (user_trace_width 0.508)
     (user_trace_width 0.762)
+    (user_trace_width 2.54)
     (trace_clearance 0.254)
     (zone_clearance 0.254)
@@
     (visible_elements 7FFF7FFF)
     (pcbplotparams
-      (layerselection 3178497)
+      (layerselection 284721153)
       (usegerberextensions true)
       (excludeedgelayer true)
-      (linewidth 0.150000)
+      (linewidth 0.203200)
       (plotframeref false)
       (viasonmask false)
       (mode 1)
-      (useauxorigin false)
+      (useauxorigin true)
       (hpglpennumber 1)
       (hpglpenspeed 20)
@@
       (psa4output false)
       (plotreference true)
-      (plotvalue true)
+      (plotvalue false)
       (plotothertext true)
       (plotinvisibletext false)
       (padsonsilk false)
-      (subtractmaskfromsilk false)
+      (subtractmaskfromsilk true)
       (outputformat 1)
       (mirror false)
-      (drillshape 1)
+      (drillshape 0)
       (scaleselection 1)
-      (outputdirectory ""))
+      (outputdirectory gerbers/))
   )
   (net 0 "")
@@
     (descr "Pin strip 4x2pin")
     (tags "CONN DEV")
-    (fp_text reference P7 (at 0 3.81 180) (layer B.SilkS)
-      (effects (font (size 1.016 1.016) (thickness 0.2032)) (justify mirror))
+    (fp_text reference P7 (at -3.81 -4.445 180) (layer B.SilkS)
+      (effects (font (size 1.778 1.778) (thickness 0.381)) (justify mirror))
     )
     (fp_text value SOCKET_4X2 (at 0 0 180) (layer B.SilkS) hide
@@
     (descr "Pin strip 4x2pin")
     (tags "CONN DEV")
-    (fp_text reference P8 (at 0 3.81 180) (layer B.SilkS)
-      (effects (font (size 1.016 1.016) (thickness 0.2032)) (justify mirror))
+    (fp_text reference P8 (at -3.81 -4.445 180) (layer B.SilkS)
+      (effects (font (size 1.778 1.778) (thickness 0.381)) (justify mirror))
     )
     (fp_text value SOCKET_4X2 (at 0 0 180) (layer B.SilkS) hide
@@
     (descr "Pin strip 4x2pin")
     (tags "CONN DEV")
-    (fp_text reference P9 (at 0 3.81 180) (layer B.SilkS)
-      (effects (font (size 1.016 1.016) (thickness 0.2032)) (justify mirror))
+    (fp_text reference P9 (at -2.54 -4.445 180) (layer B.SilkS)
+      (effects (font (size 1.778 1.778) (thickness 0.381)) (justify mirror))
     )
     (fp_text value SOCKET_3X2 (at 0 0 180) (layer B.SilkS) hide
@@
       (xy -1.68656 2.49936)) (layer F.SilkS) (width 0.00254))
   )
+  (gr_circle (center 77.47 59.69) (end 77.47 62.865) (layer F.SilkS) (width 0.3048))
+  (gr_circle (center 143.51 62.865) (end 143.51 66.04) (layer B.SilkS) (width 0.3048))
+  (gr_circle (center 77.47 59.69) (end 77.47 62.865) (layer B.SilkS) (width 0.3048))
+  (gr_arc (start 80.2379 53.975) (end 80.2379 57.15) (angle 25.8) (layer Edge.Cuts) (width 0.1524))
   (gr_text W (at 134.62 60.325 90) (layer F.SilkS)
     (effects (font (size 2.54 2.54) (thickness 0.508)))
@@
     (effects (font (size 1.778 1.524) (thickness 0.3048)) (justify left))
   )
-  (gr_arc (start 80.2379 53.975) (end 80.2379 57.15) (angle 25.8) (layer Edge.Cuts) (width 0.1524))
   (gr_arc (start 77.47 59.69) (end 77.47 56.515) (angle 25.8) (layer Edge.Cuts) (width 0.1524))
   (gr_line (start 137.16 57.15) (end 80.2379 57.15) (angle 90) (layer Edge.Cuts) (width 0.1524))
@@
   (segment (start 107.95 71.12) (end 102.87 71.12) (width 0.254) (layer B.Cu) (net 18))
   (segment (start 102.87 71.12) (end 97.79 76.2) (width 0.254) (layer B.Cu) (net 18))
+  (segment (start 77.47 59.69) (end 78.105 59.055) (width 2.54) (layer B.Cu) (net 19))
+  (segment (start 76.2 60.96) (end 77.47 59.69) (width 2.54) (layer B.Cu) (net 19))
+  (segment (start 76.2 62.23) (end 76.2 60.96) (width 2.54) (layer B.Cu) (net 19))
+  (segment (start 80.01 62.23) (end 76.2 62.23) (width 2.54) (layer B.Cu) (net 19))
+  (segment (start 80.01 59.055) (end 80.01 62.23) (width 2.54) (layer B.Cu) (net 19))
+  (segment (start 78.105 59.055) (end 80.01 59.055) (width 2.54) (layer B.Cu) (net 19))
+  (segment (start 77.47 59.69) (end 78.105 59.055) (width 2.54) (layer F.Cu) (net 19))
+  (segment (start 76.2 60.96) (end 77.47 59.69) (width 2.54) (layer F.Cu) (net 19))
+  (segment (start 76.2 62.23) (end 76.2 60.96) (width 2.54) (layer F.Cu) (net 19))
+  (segment (start 80.01 62.23) (end 76.2 62.23) (width 2.54) (layer F.Cu) (net 19))
+  (segment (start 80.01 59.055) (end 80.01 62.23) (width 2.54) (layer F.Cu) (net 19))
+  (segment (start 78.105 59.055) (end 80.01 59.055) (width 2.54) (layer F.Cu) (net 19))
+  (segment (start 143.51 62.865) (end 140.335 62.865) (width 5.08) (layer B.Cu) (net 19))
+  (segment (start 143.51 62.865) (end 140.335 62.865) (width 5.08) (layer F.Cu) (net 19))
   (segment (start 84.03082 69.85) (end 84.03082 68.15582) (width 0.762) (layer F.Cu) (net 19))
   (segment (start 80.01 66.04) (end 80.01 64.77) (width 0.762) (layer F.Cu) (net 19))
