File: CRAMP3/CRAMP3.sch (KiCad schematic (older format))
At the start: 20 parts, among them M201 POLOLU_SOCKET, M202 POLOLU_SOCKET, P201 HEADER_3X2, P202 HEADER_3X2, P203 HEADER_3X2, P205 X-MOT, P206 Y-MOT, P207 Z-MOT, U201 SM_DRIVER, U202 SM_DRIVER, U203 SM_DRIVER

Commit message: PCB placement in-progress CRAMP3 initial design and placement complete
Signed-off-by: Charles Steinkuehler <charles@steinkuehler.net>
Parts:
- gave numbers to parts that had none: 3
- renumbered C201 to C101, C202 to C102, C203 to C103, M201 to M101, M202 to M102, P201 to P101, P202 to P102, P203 to P103, P205 to P104, P206 to P105, P207 to P106, R201 to R101, R202 to R102, R203 to R103, U201 to U101, U202 to U102, U203 to U103
Connections:
- wire segments 123 -> 95

Commit message: CRAMP3 updates, PCB mostly complete
Signed-off-by: Charles Steinkuehler <charles@steinkuehler.net>
Parts:
- added M1, M2: 4-40, ~, symbol TEST_POINT_RMC
- renumbered M101 to P110, M102 to P120
Connections:
- wire segments 95 -> 98
Changed lines of the file:
@@
 Sheet 1 1
 Title "CRAMP3 (3-channel add-on for CRAMPS)"
-Date "1 may 2014"
+Date "10 may 2014"
 Rev "v1.0"
 Comp "Derived from RAMPS 1.4 reprap.org/wiki/RAMPS1.4"
@@
 Connection ~ 4650 2200
 $Comp
-L POLOLU_SOCKET M101
+L POLOLU_SOCKET P110
 U 1 1 535FFA9B
 P 9200 5250
-F 0 "M101" H 9200 5550 60  0000 C CNN
+F 0 "P110" H 9200 5550 60  0000 C CNN
 F 1 "POLOLU_SOCKET" H 9200 4950 60  0000 C CNN
 F 2 "~" H 9200 5250 60  0000 C CNN
@@
 $EndComp
 $Comp
-L POLOLU_SOCKET M102
+L POLOLU_SOCKET P120
 U 1 1 535FFAAA
 P 10100 5250
-F 0 "M102" H 10100 5550 60  0000 C CNN
+F 0 "P120" H 10100 5550 60  0000 C CNN
 F 1 "POLOLU_SOCKET" H 10100 4950 60  0000 C CNN
 F 2 "~" H 10100 5250 60  0000 C CNN
@@
 	1    0    0    -1
 $EndComp
-Text GLabel 6750 1800 0    50   BiDi ~ 0
+Text GLabel 6350 1800 0    50   BiDi ~ 0
 SPI_CS1
 $Comp
@@
 	1    0    0    -1
 $EndComp
-Text GLabel 6750 1900 0    50   BiDi ~ 0
+Text GLabel 6350 1900 0    50   BiDi ~ 0
 SPI_SPARE
 Text GLabel 7450 2000 2    50   Input ~ 0
@@
 	1    0    0    -1
 $EndComp
-Text GLabel 7050 3200 2    50   Input ~ 0
+Text GLabel 7450 3200 2    50   Input ~ 0
 MOSI-5V
-Text GLabel 7050 3100 2    50   Input ~ 0
+Text GLabel 7450 3100 2    50   Input ~ 0
 SCK-5V
-Text GLabel 7050 3000 2    50   Output ~ 0
+Text GLabel 7450 3000 2    50   Output ~ 0
 MISO-5V
-Text GLabel 7050 3300 2    50   Input ~ 0
+Text GLabel 7450 3300 2    50   Input ~ 0
 SPI_CS0
 $Comp
@@
 	1    0    0    -1
 $EndComp
-Text GLabel 6200 1900 0    50   Input ~ 0
+Text GLabel 6750 1900 0    50   Input ~ 0
 DIR_0
-Text GLabel 6200 1800 0    50   Input ~ 0
+Text GLabel 6750 1800 0    50   Input ~ 0
 STEP_0
-Text GLabel 7950 3100 0    50   Input ~ 0
+Text GLabel 7050 3200 2    50   Input ~ 0
 DIR_1
-Text GLabel 7950 3000 0    50   Input ~ 0
+Text GLabel 7050 3000 2    50   Input ~ 0
 STEP_1
-Text GLabel 8000 3450 0    50   Input ~ 0
+Text GLabel 7050 3300 2    50   Input ~ 0
 DIR_2
-Text GLabel 8000 3350 0    50   Input ~ 0
+Text GLabel 7050 3100 2    50   Input ~ 0
 STEP_2
 Wire Wire Line
 	6750 3000 6750 3400
+$Comp
+L TEST_POINT_RMC M1
+U 1 1 536D47EF
+P 8850 2200
+F 0 "M1" H 9050 2200 60  0000 C CNN
+F 1 "4-40" H 8850 2350 60  0000 C CNN
+F 2 "~" H 8850 2200 60  0000 C CNN
+F 3 "~" H 8850 2200 60  0000 C CNN
+	1    8850 2200
+	1    0    0    -1
+$EndComp
+$Comp
+L TEST_POINT_RMC M2
+U 1 1 536D47FE
+P 8850 2500
+F 0 "M2" H 9050 2500 60  0000 C CNN
+F 1 "4-40" H 8850 2650 60  0000 C CNN
+F 2 "~" H 8850 2500 60  0000 C CNN
+F 3 "~" H 8850 2500 60  0000 C CNN
+	1    8850 2500
+	1    0    0    -1
+$EndComp
+Wire Wire Line
+	8700 2200 8600 2200
+Wire Wire Line
+	8600 2200 8600 2600
+Wire Wire Line
+	8700 2500 8600 2500
+Connection ~ 8600 2500
+$Comp
+L GND #PWR019
+U 1 1 536D493E
+P 8600 2600
+F 0 "#PWR019" H 8600 2600 30  0001 C CNN
+F 1 "GND" H 8600 2530 30  0001 C CNN
+F 2 "" H 8600 2600 60  0001 C CNN
+F 3 "" H 8600 2600 60  0001 C CNN
+	1    8600 2600
+	1    0    0    -1
+$EndComp
 $EndSCHEMATC

Commit message: More progress on CRAMP3
Signed-off-by: Charles Steinkuehler <charles@steinkuehler.net>
Parts:
- removed P101, P102, P103: HEADER_3X2, symbol HEADER_3X2
- removed P104: X-MOT, symbol HEADER_4
- removed P105: Y-MOT, symbol HEADER_4
- removed P106: Z-MOT, symbol HEADER_4
- removed R101, R102, R103: 100k, symbol R
- removed U101, U102, U103: SM_DRIVER, ~, symbol SM_DRIVER
- added P1, P2, P3: HEADER_3X2, pin_strip_3x2, symbol HEADER_3X2
- added P4, P5, P6: KK-2.54-4W, CONN_KK_2.54_4W, symbol HEADER_4
- added R1, R2, R3: 100k, RESC1608x55N, symbol R
- added S1, S2, S3, S4, S5, S6, S7, S8, S9: SHUNT, Shunt, symbol SHUNT
- added U1, U2, U3: Pololu, POLOLU, symbol SM_DRIVER
- C1: renamed from C101; footprint (none) -> c_elec_6.3x7.7
- C2: renamed from C102; footprint (none) -> c_elec_6.3x7.7
- C3: renamed from C103; footprint (none) -> c_elec_6.3x7.7
- M1, M2: footprint ~ -> MTH_4-40
- P10: renamed from P110; footprint ~ -> Pololu_Socket
- P11: renamed from P120; footprint ~ -> Pololu_Socket
- P7: renamed from P107; value HEADER_4X2 -> SOCKET_4X2; footprint (none) -> Pin_Socket_4x2
- P8: renamed from P108; value Aux-3 -> SOCKET_4X2; footprint (none) -> Pin_Socket_4x2
- P9: renamed from P109; value HEADER_3X2 -> SOCKET_3X2; footprint (none) -> Pin_Socket_3x2
Connections:
- net labels added: DIR_U, DIR_V, DIR_W, STEP_U, STEP_V, STEP_W, U1A, U1B, U2A, U2B, V1A, V1B, V2A, V2B, W1A, W1B, W2A, W2B
- net labels removed: DIR_0, DIR_1, DIR_2, STEP_0, STEP_1, STEP_2
- wire segments 98 -> 100
Other:
- moved on the sheet: C1, C2, C3

Commit message: More CRAMP3 updates
Signed-off-by: Charles Steinkuehler <charles@steinkuehler.net>
Connections:
- net labels added: SPI_CS0-5V
- net labels removed: SPI_CS0
Changed lines of the file:
@@
 Sheet 1 2
 Title "CRAMP3 (3-channel add-on for CRAMPS)"
-Date "11 may 2014"
+Date "12 may 2014"
 Rev "v1.0"
 Comp "Derived from RAMPS 1.4 reprap.org/wiki/RAMPS1.4"
@@
 	1    0    0    -1
 $EndComp
-Text GLabel 6400 1700 0    50   BiDi ~ 0
+Text GLabel 7900 1700 2    50   BiDi ~ 0
 SPI_CS1
 $Comp
@@
 	1    0    0    -1
 $EndComp
-Text GLabel 6400 1800 0    50   BiDi ~ 0
+Text GLabel 7900 1800 2    50   BiDi ~ 0
 SPI_SPARE
 Text GLabel 7500 1900 2    50   Input ~ 0
 ENAn
-Text GLabel 7500 1700 2    50   BiDi ~ 0
+Text GLabel 6800 1700 0    50   BiDi ~ 0
 SCL
-Text GLabel 7500 1800 2    50   BiDi ~ 0
+Text GLabel 6800 1800 0    50   BiDi ~ 0
 SDA
 Wire Wire Line
@@
 	7400 1600 7400 1500
 Wire Wire Line
+	7000 1700 6800 1700
+Wire Wire Line
+	7000 1800 6800 1800
+Wire Wire Line
+	7300 1900 7500 1900
+Wire Wire Line
+	7300 1800 7500 1800
+Wire Wire Line
 	7300 1700 7500 1700
-Wire Wire Line
-	7300 1800 7500 1800
-Wire Wire Line
-	7300 1900 7500 1900
-Wire Wire Line
-	7000 1800 6800 1800
-Wire Wire Line
-	7000 1700 6800 1700
 $Comp
 L HEADER_3X2 P9
@@
 MISO-5V
 Text GLabel 7900 3300 2    50   Input ~ 0
-SPI_CS0
+SPI_CS0-5V
 $Comp
 L HEADER_4X2 P7
@@
 Text Label 4200 5500 0    60   ~ 0
 W1B
-Text GLabel 6800 1800 0    50   Input ~ 0
+Text GLabel 7500 1800 2    50   Input ~ 0
 DIR_U
-Text GLabel 6800 1700 0    50   Input ~ 0
+Text GLabel 7500 1700 2    50   Input ~ 0
 STEP_U
 Text GLabel 7500 3300 2    50   Input ~ 0

Commit message: Update CRAMP3 manufacturer part numbers
Signed-off-by: Charles Steinkuehler <charles@steinkuehler.net>
Parts:
- M1, M2: Mfg (none) -> None; PartNo (none) -> Part of PCB
- P10: Mfg (none) -> Sullins; PartNo (none) -> PPTC241LFBN-RC
- P11: Field4 (none) -> Sullins; PartNo (none) -> PPTC241LFBN-RC
- P7, P8: Mfg (none) -> Sullins; PartNo (none) -> PPPC042LFBN-RC
- P9: Mfg (none) -> Sullins; PartNo (none) -> PPPC032LFBN-RC
Changed lines of the file:
@@
 $Descr A 11000 8500
 encoding utf-8
-Sheet 1 2
+Sheet 1 1
 Title "CRAMP3 (3-channel add-on for CRAMPS)"
-Date "12 may 2014"
+Date "13 may 2014"
 Rev "v1.0"
 Comp "Derived from RAMPS 1.4 reprap.org/wiki/RAMPS1.4"
@@
 F 2 "Pololu_Socket" H 9200 5250 60  0001 C CNN
 F 3 "~" H 9200 5250 60  0000 C CNN
+F 4 "Sullins" H 9200 5250 60  0001 C CNN "Mfg"
+F 5 "PPTC241LFBN-RC" H 9200 5250 60  0001 C CNN "PartNo"
 	1    9200 5250
 	1    0    0    -1
@@
 F 2 "Pololu_Socket" H 10100 5250 60  0001 C CNN
 F 3 "~" H 10100 5250 60  0000 C CNN
+F 4 "Sullins" H 10100 5250 60  0001 C CNN "Field4"
+F 5 "PPTC241LFBN-RC" H 10100 5250 60  0001 C CNN "PartNo"
 	1    10100 5250
 	1    0    0    -1
@@
 F 2 "Pin_Socket_4x2" H 7150 1750 60  0001 C CNN
 F 3 "" H 7150 1750 60  0000 C CNN
+F 4 "Sullins" H 7150 1750 60  0001 C CNN "Mfg"
+F 5 "PPPC042LFBN-RC" H 7150 1750 60  0001 C CNN "PartNo"
 	1    7150 1750
 	1    0    0    -1
@@
 F 2 "Pin_Socket_3x2" H 7150 2500 60  0001 C CNN
 F 3 "" H 7150 2500 60  0000 C CNN
+F 4 "Sullins" H 7150 2500 60  0001 C CNN "Mfg"
+F 5 "PPPC032LFBN-RC" H 7150 2500 60  0001 C CNN "PartNo"
 	1    7150 2500
 	1    0    0    -1
@@
 F 2 "Pin_Socket_4x2" H 7150 3150 60  0001 C CNN
 F 3 "" H 7150 3150 60  0000 C CNN
+F 4 "Sullins" H 7150 3150 60  0001 C CNN "Mfg"
+F 5 "PPPC042LFBN-RC" H 7150 3150 60  0001 C CNN "PartNo"
 	1    7150 3150
 	1    0    0    -1
@@
 F 2 "MTH_4-40" H 8850 2200 60  0001 C CNN
 F 3 "~" H 8850 2200 60  0000 C CNN
+F 4 "None" H 8850 2200 60  0001 C CNN "Mfg"
+F 5 "Part of PCB" H 8850 2200 60  0001 C CNN "PartNo"
 	1    8850 2200
 	1    0    0    -1
@@
 F 2 "MTH_4-40" H 8850 2500 60  0001 C CNN
 F 3 "~" H 8850 2500 60  0000 C CNN
+F 4 "None" H 8850 2500 60  0001 C CNN "Mfg"
+F 5 "Part of PCB" H 8850 2500 60  0001 C CNN "PartNo"
 	1    8850 2500
 	1    0    0    -1
