File: MS-F1/MS-F100.kicad_pcb (KiCad board)
At the start: 2 copper layers, 50.8 x 17.8 mm, 32 parts, among them M1 LOGO_OSHW, M2 PCB_GREEN_RMC, P1 USBCONN, P2 CONN_20, P3 CONN_20, P4 SWD, Q1 BSS84, SW1 RST, SW2 BUT, U1 MCP1703_SOT23, U2 STM32F1xx, U3 MCP1703_SOT23, U4 NUF2042, X1 8MHz

Commit message: MS-F1 : update
Parts:
- added R7: 10k, SM0603_Resistor, B.Cu at (40.0, 42.1)
- X1: footprint XTAL-3.2x2.5mm -> crystal_smd_5x3.2mm
- moved C6 1.28 mm to (57.1, 45.4)
- moved R3 1.27 mm to (33.6, 42.1)
- moved Q1 1.27 mm to (36.8, 42.1)
- moved X1 0.19 mm to (41.2, 35.9)
- turned R1 to 180 degrees
Connections:
- C2 pad 1: N-0000035 -> N-0000032
- U2 pad 6: N-0000035 -> N-0000032
- X1 pad 2: GND -> N-0000032
Routing:
- net GND: track 135.9 -> 124.8 mm, vias 7 -> 8
- net N-0000032: track 0.00 -> 9.82 mm
- net N-0000035: track 8.79 -> 0.00 mm
- net VDD: track 97.0 -> 103.9 mm
- net /D24_USBDM: track 28.7 -> 31.8 mm
- net /D22_SWIO: track 30.8 -> 33.8 mm
- net /D26: track 8.23 -> 10.2 mm
- net /D27: track 10.5 -> 12.1 mm
- net /nRESET: track 40.5 -> 38.8 mm
- net /DISC: track 12.5 -> 13.8 mm
- net /D25: track 7.13 -> 8.29 mm
- net /D23_USBDP: track 30.1 -> 30.9 mm
- net N-0000031: track 10.2 -> 9.39 mm
- net /D14: track 19.3 -> 19.9 mm
- net /D13: track 18.1 -> 18.7 mm
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