File: Lyre_reboot/User.sch (KiCad schematic (older format))
At the start: 14 parts, among them SW1 USER, SW2 RESET

Commit message: Lyre_reboot: Update
Parts:
- removed C17: 100n, ~, symbol C
- removed R14: 100, ~, symbol R
- removed R16: 100k, NF, symbol R
- removed SB2, SB3: SOLDER_BRIDGE, ~, symbol SOLDER_BRIDGE
- added R16: 100k, NF, symbol RES
Connections:
- net BTN_USER: now also R13.1
- net NRST: now also C18.1, SW2.1, R16.2
- net VDD: now also R16.1
Other:
- moved on the sheet: C18, R13, R15, SW1, SW2
