File: Lyre_reboot/audio.sch (KiCad schematic (older format))
At the start: 24 parts, among them U5 WM8731, U6 STEREO-AUDIO-JACK

Commit message: Lyre_reboot: Update
Parts:
- removed U6: STEREO-AUDIO-JACK, ~, symbol STEREO-AUDIO-JACK
- added P11: STEREO-AUDIO-JACK_SJ1-3524-SMT, ~, symbol STEREO-AUDIO-JACK_SJ1-3524-SMT
- added R36, R37: 0R, ~, symbol RES
- L2, L3: symbol INDUCTOR_SMALL -> IND
Connections:
- net AGND_AUDIO: now also P11.1 (GND), R37.2
- net AVDD: now also R36.2
- net GND: now also R37.1
- net VDD: now also R36.1
- net at C27.2, R26.1: now also L2.2; no longer L2.1
- net at C28.2, R27.1: now also L3.2; no longer L3.1
- net at C31.1: now also L2.1, P11.3; no longer L2.2
- net at C32.1: now also L3.1, P11.2, P11.4; no longer L3.2
Changed lines of the file:
@@
 LIBS:STM32F429 LQFP144
 LIBS:RMC_connectors
+LIBS:w_connectors
+LIBS:FE
 LIBS:lyre-cache
 EELAYER 27 0
@@
 $Descr A4 11693 8268
 encoding utf-8
-Sheet 7 8
+Sheet 7 9
 Title ""
-Date "1 dec 2014"
+Date "4 feb 2015"
 Rev ""
 Comp ""
@@
 $EndComp
 $Comp
-L VDD #PWR52
+L VDD #PWR071
 U 1 1 5477A216
 P 3000 2500
-F 0 "#PWR52" H 3000 2600 30  0001 C CNN
+F 0 "#PWR071" H 3000 2600 30  0001 C CNN
 F 1 "VDD" H 3000 2610 30  0000 C CNN
 F 2 "" H 3000 2500 60  0000 C CNN
@@
 Connection ~ 3450 3700
 $Comp
-L GND #PWR53
+L GND #PWR072
 U 1 1 5477A38D
 P 3000 3300
-F 0 "#PWR53" H 3000 3300 30  0001 C CNN
+F 0 "#PWR072" H 3000 3300 30  0001 C CNN
 F 1 "GND" H 3000 3230 30  0001 C CNN
 F 2 "" H 3000 3300 60  0000 C CNN
@@
 $EndComp
 $Comp
-L VDD #PWR51
+L VDD #PWR073
 U 1 1 5477A3EA
 P 2350 3850
-F 0 "#PWR51" H 2350 3950 30  0001 C CNN
+F 0 "#PWR073" H 2350 3950 30  0001 C CNN
 F 1 "VDD" H 2350 3960 30  0000 C CNN
 F 2 "" H 2350 3850 60  0000 C CNN
@@
 $EndComp
 $Comp
-L GND #PWR55
+L GND #PWR074
 U 1 1 5477A509
 P 3250 6300
-F 0 "#PWR55" H 3250 6300 30  0001 C CNN
+F 0 "#PWR074" H 3250 6300 30  0001 C CNN
 F 1 "GND" H 3250 6230 30  0001 C CNN
 F 2 "" H 3250 6300 60  0000 C CNN
@@
 	3250 5600 3250 5650
 $Comp
-L AGND_AUDIO #PWR54
+L AGND_AUDIO #PWR075
 U 1 1 5477A5A9
 P 3000 4250
-F 0 "#PWR54" H 3000 4250 40  0001 C CNN
+F 0 "#PWR075" H 3000 4250 40  0001 C CNN
 F 1 "AGND_AUDIO" H 3000 4180 40  0000 C CNN
 F 2 "" H 3000 4250 60  0000 C CNN
@@
 $EndComp
 $Comp
-L AGND_AUDIO #PWR59
+L AGND_AUDIO #PWR076
 U 1 1 5477A5B6
 P 7000 3300
-F 0 "#PWR59" H 7000 3300 40  0001 C CNN
+F 0 "#PWR076" H 7000 3300 40  0001 C CNN
 F 1 "AGND_AUDIO" H 7000 3230 40  0000 C CNN
 F 2 "" H 7000 3300 60  0000 C CNN
@@
 $EndComp
 $Comp
-L AVDD #PWR58
+L AVDD #PWR077
 U 1 1 5477A5BE
 P 7000 2400
-F 0 "#PWR58" H 7000 2370 30  0001 C CNN
+F 0 "#PWR077" H 7000 2370 30  0001 C CNN
 F 1 "AVDD" H 7000 2500 30  0000 C CNN
 F 2 "~" H 7000 2400 60  0000 C CNN
@@
 $EndComp
 $Comp
-L INDUCTOR_SMALL L2
+L IND L2
 U 1 1 5477A8D9
 P 7600 3600
-F 0 "L2" H 7600 3700 50  0000 C CNN
-F 1 "INDUCTOR_SMALL" H 7600 3550 50  0000 C CNN
+F 0 "L2" H 7650 3625 40  0000 L CNN
+F 1 "INDUCTOR_SMALL" H 7650 3550 40  0000 L CNN
 F 2 "~" H 7600 3600 60  0000 C CNN
 F 3 "~" H 7600 3600 60  0000 C CNN
 	1    7600 3600
-	1    0    0    -1
-$EndComp
-$Comp
-L INDUCTOR_SMALL L3
+	0    1    1    0
+$EndComp
+$Comp
+L IND L3
 U 1 1 5477A8E6
 P 7600 3950
-F 0 "L3" H 7600 4050 50  0000 C CNN
-F 1 "INDUCTOR_SMALL" H 7600 3900 50  0000 C CNN
+F 0 "L3" H 7650 3975 40  0000 L CNN
+F 1 "INDUCTOR_SMALL" H 7650 3900 40  0000 L CNN
 F 2 "~" H 7600 3950 60  0000 C CNN
 F 3 "~" H 7600 3950 60  0000 C CNN
 	1    7600 3950
-	1    0    0    -1
+	0    1    1    0
 $EndComp
 $Comp
@@
 	5800 4200 6100 4200
 $Comp
-L AGND_AUDIO #PWR56
+L AGND_AUDIO #PWR078
 U 1 1 5477A9A6
 P 6100 5100
-F 0 "#PWR56" H 6100 5100 40  0001 C CNN
+F 0 "#PWR078" H 6100 5100 40  0001 C CNN
 F 1 "AGND_AUDIO" H 6100 5030 40  0000 C CNN
 F 2 "" H 6100 5100 60  0000 C CNN
@@
 	5800 3600 6100 3600
 Wire Wire Line
-	6500 3600 7350 3600
+	6500 3600 7400 3600
 $Comp
 L C C31
@@
 	1    0    0    -1
 $EndComp
-$Comp
-L STEREO-AUDIO-JACK U6
-U 1 1 5477AAB7
-P 9150 3700
-F 0 "U6" H 8900 3350 40  0000 C CNN
-F 1 "STEREO-AUDIO-JACK" H 9075 4025 30  0000 C CNN
-F 2 "~" H 9150 3700 60  0000 C CNN
-F 3 "~" H 9150 3700 60  0000 C CNN
-	1    9150 3700
-	-1   0    0    -1
-$EndComp
-Wire Wire Line
-	7850 3600 8850 3600
-Wire Wire Line
-	8850 3700 8700 3700
-Wire Wire Line
-	8700 3700 8700 3600
-Connection ~ 8700 3600
-Wire Wire Line
-	7850 3950 8850 3950
-Wire Wire Line
-	8850 3850 8700 3850
-Wire Wire Line
-	8700 3850 8700 3950
-Connection ~ 8700 3950
-Wire Wire Line
-	6500 3950 7350 3950
+Wire Wire Line
+	7800 3600 8850 3600
+Wire Wire Line
+	7800 3950 8850 3950
+Wire Wire Line
+	6500 3950 7400 3950
 Wire Wire Line
 	6100 3950 5950 3950
@@
 Connection ~ 6800 3600
 $Comp
-L AGND_AUDIO #PWR60
+L AGND_AUDIO #PWR079
 U 1 1 5477AE0D
 P 8350 4700
-F 0 "#PWR60" H 8350 4700 40  0001 C CNN
+F 0 "#PWR079" H 8350 4700 40  0001 C CNN
 F 1 "AGND_AUDIO" H 8350 4630 40  0000 C CNN
 F 2 "" H 8350 4700 60  0000 C CNN
@@
 Connection ~ 8350 4600
 $Comp
-L AGND_AUDIO #PWR57
+L AGND_AUDIO #PWR080
 U 1 1 5477B067
 P 6950 4800
-F 0 "#PWR57" H 6950 4800 40  0001 C CNN
+F 0 "#PWR080" H 6950 4800 40  0001 C CNN
 F 1 "AGND_AUDIO" H 6950 4730 40  0000 C CNN
 F 2 "" H 6950 4800 60  0000 C CNN
@@
 NoConn ~ 3900 5300
 NoConn ~ 3900 5400
+$Comp
+L VDD #PWR081
+U 1 1 54862D10
+P 7900 1100
+F 0 "#PWR081" H 7900 1200 30  0001 C CNN
+F 1 "VDD" H 7900 1210 30  0000 C CNN
+F 2 "" H 7900 1100 60  0000 C CNN
+F 3 "" H 7900 1100 60  0000 C CNN
+	1    7900 1100
+	1    0    0    -1
+$EndComp
+$Comp
+L AVDD #PWR082
+U 1 1 54862D16
+P 8350 1100
+F 0 "#PWR082" H 8350 1070 30  0001 C CNN
+F 1 "AVDD" H 8350 1200 30  0000 C CNN
+F 2 "~" H 8350 1100 60  0000 C CNN
+F 3 "~" H 8350 1100 60  0000 C CNN
+	1    8350 1100
+	1    0    0    -1
+$EndComp
+$Comp
+L AGND_AUDIO #PWR083
+U 1 1 54862D1C
+P 8350 1600
+F 0 "#PWR083" H 8350 1600 40  0001 C CNN
+F 1 "AGND_AUDIO" H 8350 1530 40  0000 C CNN
+F 2 "" H 8350 1600 60  0000 C CNN
+F 3 "" H 8350 1600 60  0000 C CNN
+	1    8350 1600
+	1    0    0    -1
+$EndComp
+$Comp
+L GND #PWR084
+U 1 1 54862D22
+P 7900 1600
+F 0 "#PWR084" H 7900 1600 30  0001 C CNN
+F 1 "GND" H 7900 1530 30  0001 C CNN
+F 2 "" H 7900 1600 60  0000 C CNN
+F 3 "" H 7900 1600 60  0000 C CNN
+	1    7900 1600
+	1    0    0    -1
+$EndComp
+Wire Wire Line
+	7900 1600 7900 1500
+Wire Wire Line
+	8350 1500 8350 1600
+Wire Wire Line
+	7900 1100 7900 1200
+Wire Wire Line
+	8350 1200 8350 1100
+$Comp
+L STEREO-AUDIO-JACK_SJ1-3524-SMT P11
+U 1 1 548A1756
+P 9150 3700
+F 0 "P11" H 8900 3350 40  0000 C CNN
+F 1 "STEREO-AUDIO-JACK_SJ1-3524-SMT" H 9075 4025 30  0000 C CNN
+F 2 "~" H 9150 3700 60  0000 C CNN
+F 3 "~" H 9150 3700 60  0000 C CNN
+	1    9150 3700
+	-1   0    0    -1
+$EndComp
+Connection ~ 8700 3950
+Wire Wire Line
+	8700 3850 8700 3950
+Wire Wire Line
+	8850 3850 8700 3850
+$Comp
+L RES R36
+U 1 1 548B810E
+P 8100 1200
+F 0 "R36" H 8175 1250 40  0000 L CNN
+F 1 "0R" H 8175 1175 40  0000 L CNN
+F 2 "~" H 8175 1100 40  0000 L CNN
+F 3 "~" H 8175 1025 40  0000 L CNN
+	1    8100 1200
+	0    -1   -1   0
+$EndComp
+$Comp
+L RES R37
+U 1 1 548B8125
+P 8100 1500
+F 0 "R37" H 8175 1550 40  0000 L CNN
+F 1 "0R" H 8175 1475 40  0000 L CNN
+F 2 "~" H 8175 1400 40  0000 L CNN
+F 3 "~" H 8175 1325 40  0000 L CNN
+	1    8100 1500
+	0    -1   -1   0
+$EndComp
+$Comp
+L PWR_FLAG #FLG085
+U 1 1 548E0449
+P 8700 1200
+F 0 "#FLG085" H 8700 1295 30  0001 C CNN
+F 1 "PWR_FLAG" H 8700 1380 30  0000 C CNN
+F 2 "" H 8700 1200 60  0000 C CNN
+F 3 "" H 8700 1200 60  0000 C CNN
+	1    8700 1200
+	1    0    0    -1
+$EndComp
+$Comp
+L PWR_FLAG #FLG086
+U 1 1 548E0456
+P 8700 1500
+F 0 "#FLG086" H 8700 1595 30  0001 C CNN
+F 1 "PWR_FLAG" H 8700 1680 30  0000 C CNN
+F 2 "" H 8700 1500 60  0000 C CNN
+F 3 "" H 8700 1500 60  0000 C CNN
+	1    8700 1500
+	1    0    0    -1
+$EndComp
+Wire Wire Line
+	8300 1500 8700 1500
+Wire Wire Line
+	8300 1200 8700 1200
+Connection ~ 8350 1500
+Connection ~ 8350 1200
 $EndSCHEMATC
