File: Lyre_reboot/cpu.sch (KiCad schematic (older format))
At the start: 32 parts, among them P1 SWD, U1 STM32F407_LQFP100, U2 CONN_CORTEX_DEBUG, X1 8MHz

Commit message: Lyre_reboot: Update
Parts:
- removed R8: NF, ~, symbol R
- removed SB1: SOLDER_BRIDGE, symbol SOLDER_BRIDGE
- removed X1: 8MHz, ~, symbol CRYSTAL
- added R38: 10k, ~, symbol R
- added U8: FRAM 2KB, symbol EEPROM_SPI
- added X1: 8MHz, ~, symbol CRYSTAL_4PIN_GND
- R2: footprint ~ -> NF
- R3, R9: symbol R -> RES
- R4, R5: footprint ~ -> NF; symbol R -> RES
- renumbered U2 to P8
Connections:
- net PD0 is gone; now on net D2: U1.81 (PD0)
- net PD1 is gone; now on net D3: U1.82 (PD1)
- net PD10 is gone; now on net D15: U1.57 (PD10)
- net PD14 is gone; now on net D0: U1.61 (PD14)
- net PD15 is gone; now on net D1: U1.62 (PD15)
- net PD8 is gone; now on net D13: U1.55 (PD8)
- net PD9 is gone; now on net D14: U1.56 (PD9)
- net D0: no longer U1.97 (PE0)
- net D1: no longer U1.98 (PE1)
- net D10: now also U1.44 (PE13); no longer U1.41 (PE10)
- net D11: now also U1.45 (PE14); no longer U1.42 (PE11)
- net D12: now also U1.46 (PE15); no longer U1.43 (PE12)
- net D13: no longer U1.44 (PE13)
- net D14: no longer U1.45 (PE14)
- net D15: no longer U1.46 (PE15)
- net D2: no longer U1.1 (PE2-TRACECLK)
- net D3: no longer U1.2 (PE3-TRACED0)
- net D4: now also U1.38 (PE7); no longer U1.3 (PE4-TRACED1)
- net D5: now also U1.39 (PE8); no longer U1.4 (PE5-TRACED2)
- net D6: now also U1.40 (PE9); no longer U1.5 (PE6-TRACED3)
- net D7: now also U1.41 (PE10); no longer U1.38 (PE7)
- net D8: now also U1.42 (PE11); no longer U1.39 (PE8)
- net D9: now also U1.43 (PE12); no longer U1.40 (PE9)
- net GND: now also R3.2, R5.2, R9.2, R38.1, U8.4 (VSS), X1.2 (GND), X1.4 (GND); no longer R3.1, R5.1
- net PB2: now also R38.2
- net SWO: no longer P8.6 (TDO), U1.89 (PB3-JTDO-SWTRACE)
- net UART2_RX: no longer U1.26 (PA3)
- net UART2_TX: no longer U1.25 (PA2)
- net VDD: now also R4.2, U8.3 (~WP), U8.7 (~HOLD), U8.8 (VDD); no longer R4.1
- net at C4.1, R7.2: now also X1.3 (B)
- net at C3.1, R6.2: now also X1.1 (A)
- net at C1.1, U1.49 (VCAP1): now also R5.1; no longer R5.2
- net PA1 renamed LED_PWM
- net PA15 renamed SPI3_SS
- net SPI3_SS: now also U8.1 (~CS)
- net PB0 renamed LED1
- net PB1 renamed LED2
- net PB4 renamed SPI3_MISO
- net SPI3_MISO: now also U8.2 (SO)
- net PB5 renamed SPI3_MOSI
- net SPI3_MOSI: now also U8.5 (SI)
- net PB8 renamed AUDIO_SCL
- net PB9 renamed AUDIO_SDA
- net PC13 renamed LCD_RST
- net PC14 renamed TP_INT
- net PC15 renamed SD_SS
- net PD11 renamed LCD_RS
- net PD3 renamed SD_CARD_DET
- net PD4 renamed LCD_RD
- net PD5 renamed LCD_WR
- net PD7 renamed LCD_CS
- new net: R3.1, R4.1, U1.99 (VSS)
- new net BUCK_ON: U1.2 (PE3-TRACED0)
- new net HPWR: U1.97 (PE0)
- new net LDO_ON: U1.1 (PE2-TRACECLK)
- new net PA2: U1.25 (PA2)
- new net PA3: U1.26 (PA3)
- new net PBSTAT: U1.4 (PE5-TRACED2)
- new net SPI3_SCK: U1.89 (PB3-JTDO-SWTRACE), U8.6 (SCK)
- new net STBY: U1.3 (PE4-TRACED1)
- new net SUSP: U1.98 (PE1)
- new net nCHRG: U1.5 (PE6-TRACED3)
- no-connect marks 2 -> 3
Other:
- note added: "Boot0 \n0 = user Flash\n1 = ROM bootloader"
- note added: "Compatible with F429, F103 in 100 pin package"
- note added: "FRAM"
- note added: "PB2-Boot1 must be \nlow at startup\nto invoke ROM \nbootloader"
- note added: "TODO:\n\nroute boot0 to pin or test pad?\n\n"
- moved on the sheet: C3, C4, R9
