File: Lyre_reboot/lcd.sch (KiCad schematic (older format))
At the start: 4 parts, among them P2 LCD 2.4, P3 LCD 2.4 SD, P4 LCD_2.8_INCH, P5 LCD 2.2

Commit message: Lyre_reboot: Update
Parts:
- added P10: LCD_2.4_INCH, ~, symbol CONN_2X20
- added Q1: BSS84, ~, symbol MOSFET_P
Connections:
- net labels added: F_CS, LED_A, LED_PWM, SPI1_MISO, SPI1_MOSI, SPI1_SCK, SPI1_SS, SPI3_MISO, SPI3_MOSI, SPI3_SCK, VDD
- net labels removed: +3.3V
- wire segments 67 -> 105
- no-connect marks 0 -> 7
Other:
- note added: "2.4" LCD with 16 bit i/f and \nSPI Touch panel, SD card socket"
- note added: "Option"
- note added: "SD card only"
- note added: "also 2.8" TFT\nhttp://imall.iteadstudio.com/im120419010.html"
- note added: "http://www.ebay.co.uk/itm/171551006462?_trksid=p2055119.m1438.l2649&ssPageName=STRK%3AMEBIDX%3AIT"
- note added: "http://www.elabpeers.com/2-4-tft-lcd-touch.html"
- moved on the sheet: P5
