File: Lyre_reboot/power.sch (KiCad schematic (older format))
At the start: 11 parts, among them P6 EXT_5V, P7 Battery, SW3 SWITCH_INV, U4 1117

Commit message: Lyre updates
Parts:
- removed SW3: SWITCH_INV, ~, symbol SWITCH_INV
- added C34, C38: 10u, ~, symbol C
- added C35: 10p, ~, symbol C
- added C36: 4u7, ~, symbol CAP
- added C37: 2u2, ~, symbol C
- added L4: 10uH, ~, symbol IND
- added R28: 100k, ~, symbol R
- added R29: 1.87k, ~, symbol R
- added R30: 2.05M, ~, symbol RES
- added R31, R33: 649k, ~, symbol R
- added R32: 332k, ~, symbol R
- added SW3: SW_ON, ~, symbol SW_PUSH
- added U7: LTC3553, symbol LTC3553
- added VR1: 100k, ~, symbol VR
- C19: value 1u -> 10u
- D3: symbol DIODE -> DIOD
Connections:
- net +5V: now also R28.1, U7.20 (VBUS); no longer U4.3 (VI)
- net GND: now also C34.2, C36.2, C37.2, C38.2, R29.2, R31.2, R33.2, SW3.1, U7.2 (SEQ), U7.21 (GND), VR1.2
- net at P7.1 (P1): now also U7.17 (BAT)
- new net: C34.1, C37.1, U4.3 (VI), U7.11 (VINLDO), U7.12 (BVIN), U7.18 (VOUT)
- new net: C36.1, R30.1, U7.10 (LDO)
- new net: L4.2, U7.13 (SW)
- new net: R28.2, U7.15 (NTC), VR1.1
- new net: R29.1, U7.16 (PROG)
- new net: SW3.2, U7.4 (~ON)
- new net: C35.2, R32.2, R33.1, U7.8 (BUCK_FB)
- new net: R30.2, R31.1, U7.9 (LDO_FB)
- new net: C35.1, C38.1, L4.1, R32.1
- no-connect marks 1 -> 0
Other:
- moved on the sheet: C20, D3, D4, D5, D6, P6, P7, R19, U4

Commit message: Lyre_reboot: Update
Parts:
- removed U4: 1117, symbol 1117
- added D7: DIODE, ~, symbol DIOD
- added D8: CHRG, ~, symbol LED_RMC
- added P14: 12V_IN, symbol CONN_2
- added R14: 470, ~, symbol RES
- added R34, R35: 0, ~, symbol RES
- added R8: 100k, ~, symbol RES
- added U2: Traco TSR 1-2450, ~, symbol 78XX_RMC
- added U4: MCP1703_SOT23, SOT23, symbol MCP1703_SOT23
- C19, C20, C34, C35, C37, C38: symbol C -> CAP
- D4, D6: symbol DIODE -> DIOD
- D5: symbol LED -> LED_RMC
- L4: value 10uH -> 4.7uH
- P7: symbol CONN_2 -> CONN_3
- R19, R29, R31, R33: symbol R -> RES
- R28: value 100k -> 10k; symbol R -> RES
- R32: value 332k -> 2.05M; symbol R -> RES
- VR1: value 100k -> 10k; symbol VR -> VR_RMC
Connections:
- net +5V: now also D7.2 (K)
- net GND: now also P14.2 (PM), U2.2 (GND), U4.1 (GND); no longer U7.2 (SEQ)
- net VDD: now also R19.1, R34.2, R35.2, R8.1; no longer D6.2 (K)
- net at C20.1, D6.1 (A): now also U4.2 (VO); no longer R19.1
- net V_OUT: now reaches C34.1, C37.1, U7.11 (VINLDO), U7.12 (BVIN), U7.18 (VOUT)
- net V_OUT: now also U7.2 (SEQ), R14.1, U4.3 (VI)
- net BAT_THERMISTOR: now reaches P7.1 (P1)
- net BAT_THERMISTOR: now also R28.2, U7.15 (NTC), VR1.1; no longer U7.17 (BAT)
- net HPWR: now reaches U7.1 (HPWR)
- net at C36.1, R30.1, U7.10 (LDO): now also R35.1
- net at U7.13 (SW): now also L4.1; no longer L4.2
- net nCHRG: now reaches U7.14 (~CHRG)
- net nCHRG: now also D8.2 (K)
- net SUSP: now reaches U7.19 (SUSP)
- net PBSTAT: now reaches U7.3 (PBSTAT)
- net PBSTAT: now also R8.2
- net LDO_ON: now reaches U7.5 (LDO_ON)
- net STBY: now reaches U7.6 (STBY)
- net BUCK_ON: now reaches U7.7 (BUCK_ON)
- net at C35.1, C38.1, R32.1: now also L4.2; no longer L4.1
- new net: D6.2 (K), R34.1
- new net: D7.1 (A), U2.3 (VO)
- new net: D8.1 (A), R14.2
- new net +12V: P14.1 (P1), U2.1 (VI)
- new net V_BAT: P7.3 (P3), U7.17 (BAT)
Other:
- note added: "3.3V, Max 150mA"
- note added: "3.3V, Max 200mA"
- note added: "Aux 5V input for testing"
- note added: "May not be required?"
- note added: "NTC\nthermistor"
- note added: "Nominal 12V"
- note added: "Note\n\n1. R29 determines charging current\nwhere I = 750 / R\n1.87k = 400mA\n\n2. SEQ = high turn on LDO first"
- note added: "Optionals"
- note added: "Probably not required"
- note added: "TSR 1-2450 has input range\n6.5 - 32V input"
- moved on the sheet: D6, R19, R28
