File: Lyre_reboot/sdcard.sch (KiCad schematic (older format))
At the start: 2 parts, among them K1 SDCARD

Commit message: Lyre_reboot: Update
Parts:
- removed K1: SDCARD, ~, symbol SDCARD
- added P12: CONN_MICROSD, ~, symbol CONN_MICROSD
- added P13: CONN_SD, ~, symbol CONN_SD
- C33: symbol C -> CAP
Connections:
- wire segments 16 -> 32
Other:
- note added: "SD Card"
- note added: "SD_CS"
- note added: "SD_MISO"
- note added: "SD_MOSI"
- note added: "SD_SCLK"
