File: Lyre_reboot/usb.sch (KiCad schematic (older format))
At the start: 3 parts, among them U3 USBCONN-HOSTCAPABLE

Commit message: Lyre_reboot: Update
Parts:
- renumbered U3 to P9
Changed lines of the file:
@@
 LIBS:STM32F429 LQFP144
 LIBS:RMC_connectors
+LIBS:w_connectors
+LIBS:FE
 LIBS:lyre-cache
 EELAYER 27 0
@@
 $Descr A4 11693 8268
 encoding utf-8
-Sheet 3 8
+Sheet 3 9
 Title ""
-Date "1 dec 2014"
+Date "4 feb 2015"
 Rev ""
 Comp ""
@@
 $EndDescr
 $Comp
-L USBCONN-HOSTCAPABLE U3
+L USBCONN-HOSTCAPABLE P9
 U 1 1 5477BD71
 P 6700 4550
-F 0 "U3" H 6700 4200 60  0000 C CNN
+F 0 "P9" H 6700 4200 60  0000 C CNN
 F 1 "USBCONN-HOSTCAPABLE" H 6850 4875 20  0000 C CNN
 F 2 "~" H 6700 4550 60  0000 C CNN
@@
 	6400 4400 5900 4400
 $Comp
-L GND #PWR21
+L GND #PWR025
 U 1 1 5477C49E
 P 6100 5150
-F 0 "#PWR21" H 6100 5150 30  0001 C CNN
+F 0 "#PWR025" H 6100 5150 30  0001 C CNN
 F 1 "GND" H 6100 5080 30  0001 C CNN
 F 2 "" H 6100 5150 60  0000 C CNN
